File: audio.kicad_sch (KiCad schematic)
At the start: 25 parts, among them IC1 ES9218PQ, Y2 ECS-2520SMV-500-GP-TR

Commit message: finishing up schematic
Parts:
- added J5: SJ2-35954B-SMT-TR, SJ2-35954B-SMT-TR:CUI_SJ2-35954B-SMT-TR, symbol Connector_Audio:AudioJack4_SwitchT1
- added JP9: SolderJumper_2_Bridged, Jumper:SolderJumper-2_P1.3mm_Bridged_RoundedPad1.0x1.5mm, symbol Jumper:SolderJumper_2_Bridged
- R13: now not fitted
- R5, R6: now fitted
Connections:
- net +3V3MCLK: now also JP9.1 (A)
- net MCLK_EN: now also JP9.2 (B)
- new net: J5.R1, J5.R2, J5.S, J5.T, J5.TN

Commit message: esd, jack, io expander, led, power swquence
Parts:
- removed C28: 2.2nF, symbol Device:C
- removed JP9: SolderJumper_2_Bridged, Jumper:SolderJumper-2_P1.3mm_Bridged_RoundedPad1.0x1.5mm, symbol Jumper:SolderJumper_2_Bridged
- added C50: 2.2nF, symbol Device:C
- added D10, D11, D8, D9: D_TVS, Diode_SMD:D_0201_0603Metric, symbol Device:D_TVS
- added JP4: SolderJumper_2_Open, Jumper:SolderJumper-2_P1.3mm_Open_RoundedPad1.0x1.5mm, symbol Jumper:SolderJumper_2_Open
- added R27: 1.8k, symbol Device:R
- added R29: 47k, symbol Device:R
- R13: now fitted
Connections:
- net +3V3MCLK: now also JP4.1 (A)
- net GND: now also C27.1, J5.R2, C50.1, D10.1 (A1), D11.1 (A1), D8.1 (A1), D9.1 (A1); no longer C27.2
- net MCLK_EN: now also JP4.2 (B)
- net OUT_L: now reaches C29.2, IC1.22 (OUT_L)
- net OUT_L: now also J5.T, D9.2 (A2)
- net at IC1.8 (IN_R): now also C27.2; no longer C27.1
- net at IC1.23 (IN_L): now also C50.2
- net OUT_R: now reaches C30.1, IC1.9 (OUT_R)
- net OUT_R: now also J5.R1, D10.2 (A2)
- new net +1V8MIC: R27.1
- new net +3V3: R29.2
- new net MIC: D11.2 (A2), J5.S, R27.2
- new net TN: D8.2 (A2), J5.TN, R29.1
Other:
- moved on the sheet: C27, C29, J5
