File: audio.kicad_sch (KiCad schematic)
At the start: 33 parts, among them IC1 ES9218PQ, J5 SJ2-35954B-SMT-TR, Y2 ECS-2520SMV-500-GP-TR

Commit message: reannotated schematic
Parts:
- renumbered C5 to C41, C26 to C42, C25 to C43, C24 to C44, C23 to C45, C22 to C46, C14 to C47, C17 to C48, C20 to C49, C21 to C50, C15 to C51, C19 to C52, C30 to C53, C29 to C54, C27 to C55, C50 to C56, D9 to D11, D8 to D12, D11 to D9, IC1 to IC4, J5 to J4, JP4 to JP9, R4 to R27, R1 to R28, R6 to R29, R2 to R30, R3 to R31, R5 to R32, R13 to R33, R27 to R34, R29 to R35, Y2 to Y1

Commit message: added titles to sheets
Other:
- title: (none) -> AUDIO
Changed lines of the file:
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@@
 	(generator_version "9.0")
 	(paper "A4")
+	(title_block
+		(title "AUDIO")
+	)
 	(rectangle
 		(start 12.7 12.7)

Commit message: small fixes
Parts:
- removed R29, R32: 47k, symbol Device:R
- R27, R35: value 47k -> 10k
- R28, R30, R31: value 47k -> 1.2k
Connections:
- no-connect marks 1 -> 3
Other:
- moved on the sheet: C41, R27, R35

Commit message: added 3d models
Parts:
- D10, D11, D12, D9: footprint Diode_SMD:D_0201_0603Metric -> CD0201-T2.0LC:CD0201T20LC
Changed lines of the file:
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@@
 	(wire
 		(pts
+			(xy 165.1 85.09) (xy 165.1 86.36)
+		)
+		(stroke
+			(width 0)
+			(type default)
+		)
+	)
+	(wire
+		(pts
 			(xy 153.67 106.68) (xy 154.94 106.68)
 		)
@@
 	(wire
 		(pts
+			(xy 154.94 83.82) (xy 153.67 83.82)
+		)
+		(stroke
+			(width 0)
+			(type default)
+		)
+	)
+	(wire
+		(pts
 			(xy 166.37 110.49) (xy 166.37 111.76)
 		)
@@
 	(wire
 		(pts
-			(xy 106.68 91.44) (xy 113.03 91.44)
-		)
-		(stroke
-			(width 0)
-			(type default)
-		)
-	)
-	(wire
-		(pts
 			(xy 172.72 68.58) (xy 176.53 68.58)
 		)
@@
 	(wire
 		(pts
-			(xy 154.94 83.82) (xy 153.67 83.82)
-		)
-		(stroke
-			(width 0)
-			(type default)
-		)
-	)
-	(wire
-		(pts
 			(xy 153.67 52.07) (xy 153.67 45.72)
 		)
@@
 	(wire
 		(pts
+			(xy 154.94 82.55) (xy 157.48 82.55)
+		)
+		(stroke
+			(width 0)
+			(type default)
+		)
+	)
+	(wire
+		(pts
 			(xy 120.65 62.23) (xy 116.84 62.23)
 		)
@@
 	(wire
 		(pts
+			(xy 96.52 90.17) (xy 96.52 91.44)
+		)
+		(stroke
+			(width 0)
+			(type default)
+		)
+	)
+	(wire
+		(pts
 			(xy 143.51 128.27) (xy 147.32 128.27)
 		)
@@
 	(wire
 		(pts
-			(xy 160.02 86.36) (xy 153.67 86.36)
+			(xy 138.43 39.37) (xy 138.43 63.5)
 		)
 		(stroke
@@
 	(wire
 		(pts
-			(xy 138.43 39.37) (xy 138.43 63.5)
+			(xy 34.29 76.2) (xy 34.29 85.09)
 		)
 		(stroke
@@
 	(wire
 		(pts
-			(xy 34.29 76.2) (xy 34.29 85.09)
+			(xy 46.99 153.67) (xy 46.99 152.4)
 		)
 		(stroke
@@
 	(wire
 		(pts
-			(xy 46.99 153.67) (xy 46.99 152.4)
+			(xy 21.59 30.48) (xy 21.59 31.75)
 		)
 		(stroke
@@
 	(wire
 		(pts
-			(xy 21.59 30.48) (xy 21.59 31.75)
+			(xy 149.86 45.72) (xy 153.67 45.72)
 		)
 		(stroke
@@
 	(wire
 		(pts
-			(xy 149.86 45.72) (xy 153.67 45.72)
+			(xy 165.1 86.36) (xy 153.67 86.36)
 		)
 		(stroke
@@
 	(wire
 		(pts
+			(xy 154.94 82.55) (xy 154.94 83.82)
+		)
+		(stroke
+			(width 0)
+			(type default)
+		)
+	)
+	(wire
+		(pts
 			(xy 54.61 137.16) (xy 54.61 143.51)
 		)
@@
 	(wire
 		(pts
+			(xy 96.52 91.44) (xy 113.03 91.44)
+		)
+		(stroke
+			(width 0)
+			(type default)
+		)
+	)
+	(wire
+		(pts
 			(xy 104.14 110.49) (xy 104.14 111.76)
 		)
@@
 			)
 		)
-		(property "Footprint" "Diode_SMD:D_0201_0603Metric"
+		(property "Footprint" "CD0201-T2.0LC:CD0201T20LC"
 			(at 39.37 147.32 0)
 			(effects
@@
 			)
 		)
-		(property "Footprint" "Diode_SMD:D_0201_0603Metric"
+		(property "Footprint" "CD0201-T2.0LC:CD0201T20LC"
 			(at 44.45 147.32 0)
 			(effects
@@
 			)
 		)
-		(property "Footprint" "Diode_SMD:D_0201_0603Metric"
+		(property "Footprint" "CD0201-T2.0LC:CD0201T20LC"
 			(at 49.53 147.32 0)
 			(effects
@@
 	(symbol
 		(lib_id "power:+1V8")
-		(at 160.02 86.36 270)
+		(at 165.1 85.09 0)
 		(unit 1)
 		(exclude_from_sim no)
@@
 		(on_board yes)
 		(dnp no)
-		(fields_autoplaced yes)
 		(property "Reference" "#PWR088"
-			(at 156.21 86.36 0)
+			(at 165.1 88.9 0)
 			(effects
 				(font
@@
 		)
 		(property "Value" "+3V3AVDD"
-			(at 163.83 86.3599 90)
+			(at 166.116 83.566 0)
 			(effects
 				(font
@@
 		)
 		(property "Footprint" ""
-			(at 160.02 86.36 0)
+			(at 165.1 85.09 0)
 			(effects
 				(font
@@
 		)
 		(property "Datasheet" ""
-			(at 160.02 86.36 0)
+			(at 165.1 85.09 0)
 			(effects
 				(font
@@
 		)
 		(property "Description" "Power symbol creates a global label with name \"+1V8\""
-			(at 160.02 86.36 0)
+			(at 165.1 85.09 0)
 			(effects
 				(font
@@
 	(symbol
 		(lib_id "power:+3V3")
-		(at 106.68 91.44 90)
+		(at 96.52 90.17 0)
 		(unit 1)
 		(exclude_from_sim no)
@@
 		(dnp no)
 		(property "Reference" "#PWR090"
-			(at 110.49 91.44 0)
+			(at 96.52 93.98 0)
 			(effects
 				(font
@@
 		)
 		(property "Value" "+3V3VCCA"
-			(at 103.632 91.44 90)
+			(at 85.598 88.646 0)
 			(effects
 				(font
@@
 		)
 		(property "Footprint" ""
-			(at 106.68 91.44 0)
+			(at 96.52 90.17 0)
 			(effects
 				(font
@@
 		)
 		(property "Datasheet" ""
-			(at 106.68 91.44 0)
+			(at 96.52 90.17 0)
 			(effects
 				(font
@@
 		)
 		(property "Description" "Power symbol creates a global label with name \"+3V3\""
-			(at 106.68 91.44 0)
+			(at 96.52 90.17 0)
 			(effects
 				(font
@@
 	(symbol
 		(lib_id "power:GND")
-		(at 154.94 83.82 90)
+		(at 157.48 82.55 0)
 		(unit 1)
 		(exclude_from_sim no)
@@
 		(dnp no)
 		(property "Reference" "#PWR087"
-			(at 161.29 83.82 0)
+			(at 157.48 88.9 0)
 			(effects
 				(font
@@
 		)
 		(property "Value" "GND"
-			(at 160.02 83.82 90)
+			(at 160.782 84.328 0)
 			(effects
 				(font
@@
 		)
 		(property "Footprint" ""
-			(at 154.94 83.82 0)
+			(at 157.48 82.55 0)
 			(effects
 				(font
@@
 		)
 		(property "Datasheet" ""
-			(at 154.94 83.82 0)
+			(at 157.48 82.55 0)
 			(effects
 				(font
@@
 		)
 		(property "Description" "Power symbol creates a global label with name \"GND\" , ground"
-			(at 154.94 83.82 0)
+			(at 157.48 82.55 0)
 			(effects
 				(font
@@
 			)
 		)
-		(property "Footprint" "Diode_SMD:D_0201_0603Metric"
+		(property "Footprint" "CD0201-T2.0LC:CD0201T20LC"
 			(at 54.61 147.32 0)
 			(effects

Commit message: fuel gauge ic
Parts:
- removed R31: 1.2k, symbol Device:R
- added R29: 47k, Resistor_SMD:R_0402_1005Metric, symbol Device:R
- C41, C42, C43, C44, C45, C46, C47, C48, C49, C50, C51, C52, C53, C54, C55, C56: footprint (none) -> Capacitor_SMD:C_0402_1005Metric
- R27, R33, R34, R35: footprint (none) -> Resistor_SMD:R_0402_1005Metric
- R28, R30: value 1.2k -> 47k; footprint (none) -> Resistor_SMD:R_0402_1005Metric
- Y1: footprint ECS2520SMV500GPTR -> ECS-2520SMV-500-GP-TR:ECS2520SMV500GPTR
Connections:
- net DATA1: now also R29.1; no longer R30.1
- net DATA_CLK: now also R30.1
- net GND: now also R29.2
Other:
- note added: "addr(dec.):54"

Commit message: layout
Parts:
- C42: footprint Capacitor_SMD:C_0402_1005Metric -> Capacitor_SMD:C_0603_1608Metric
Other:
- moved on the sheet: C42, C43

Commit message: almost finished with the layout
Parts:
- removed R30: 47k, Resistor_SMD:R_0402_1005Metric, symbol Device:R
Connections:
- net +3V3: now also R27.1
- net +3V3AVDD: no longer R27.1
Changed lines of the file:
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@@
 	)
 	(junction
-		(at 133.35 52.07)
-		(diameter 0)
-		(color 0 0 0 0)
-	)
-	(junction
 		(at 44.45 129.54)
 		(diameter 0)
@@
 	)
 	(junction
-		(at 153.67 52.07)
-		(diameter 0)
-		(color 0 0 0 0)
-	)
-	(junction
 		(at 121.92 147.32)
 		(diameter 0)
@@
 	(wire
 		(pts
-			(xy 133.35 50.8) (xy 133.35 52.07)
+			(xy 133.35 50.8) (xy 133.35 63.5)
 		)
 		(stroke
@@
 	(wire
 		(pts
-			(xy 153.67 53.34) (xy 153.67 52.07)
+			(xy 153.67 45.72) (xy 153.67 49.53)
 		)
 		(stroke
@@
 	(wire
 		(pts
-			(xy 149.86 52.07) (xy 153.67 52.07)
-		)
-		(stroke
-			(width 0)
-			(type default)
-		)
-	)
-	(wire
-		(pts
 			(xy 161.29 111.76) (xy 154.94 111.76)
 		)
@@
 	(wire
 		(pts
-			(xy 133.35 52.07) (xy 133.35 63.5)
-		)
-		(stroke
-			(width 0)
-			(type default)
-		)
-	)
-	(wire
-		(pts
 			(xy 21.59 135.89) (xy 21.59 137.16)
 		)
@@
 	(wire
 		(pts
-			(xy 153.67 52.07) (xy 153.67 45.72)
-		)
-		(stroke
-			(width 0)
-			(type default)
-		)
-	)
-	(wire
-		(pts
 			(xy 166.37 111.76) (xy 161.29 111.76)
 		)
@@
 	(wire
 		(pts
-			(xy 133.35 52.07) (xy 142.24 52.07)
-		)
-		(stroke
-			(width 0)
-			(type default)
-		)
-	)
-	(wire
-		(pts
 			(xy 138.43 130.81) (xy 138.43 127)
 		)
@@
 	)
 	(symbol
-		(lib_id "Device:R")
-		(at 146.05 52.07 90)
-		(unit 1)
-		(exclude_from_sim no)
-		(in_bom yes)
-		(on_board yes)
-		(dnp no)
-		(property "Reference" "R30"
-			(at 146.05 48.006 90)
-			(effects
-				(font
-					(size 1.27 1.27)
-				)
-			)
-		)
-		(property "Value" "47k"
-			(at 146.05 49.784 90)
-			(effects
-				(font
-					(size 1.27 1.27)
-				)
-			)
-		)
-		(property "Footprint" "Resistor_SMD:R_0402_1005Metric"
-			(at 146.05 53.848 90)
-			(effects
-				(font
-					(size 1.27 1.27)
-				)
-				(hide yes)
-			)
-		)
-		(property "Datasheet" "~"
-			(at 146.05 52.07 0)
-			(effects
-				(font
-					(size 1.27 1.27)
-				)
-				(hide yes)
-			)
-		)
-		(property "Description" "Resistor"
-			(at 146.05 52.07 0)
-			(effects
-				(font
-					(size 1.27 1.27)
-				)
-				(hide yes)
-			)
-		)
-		(pin "2"
-		)
-		(pin "1"
-		)
-		(instances
-			(project "meko-pcb"
-				(path "/bdd43acd-23c1-472b-909a-8e24eb60d56d/dd2be10c-708f-4995-b13e-6fc09628a9ce"
-					(reference "R30")
-					(unit 1)
-				)
-			)
-		)
-	)
-	(symbol
 		(lib_id "Device:C")
 		(at 57.15 52.07 0)
@@
 			)
 		)
-		(property "Value" "+3V3AVDD"
+		(property "Value" "+3V3"
 			(at 113.538 34.29 0)
 			(effects
@@
 	(symbol
 		(lib_id "power:GND")
-		(at 153.67 53.34 0)
+		(at 153.67 49.53 0)
 		(unit 1)
 		(exclude_from_sim no)
@@
 		(dnp no)
 		(property "Reference" "#PWR079"
-			(at 153.67 59.69 0)
+			(at 153.67 55.88 0)
 			(effects
 				(font
@@
 		)
 		(property "Value" "GND"
-			(at 153.67 57.15 0)
+			(at 153.67 53.34 0)
 			(effects
 				(font
@@
 		)
 		(property "Footprint" ""
-			(at 153.67 53.34 0)
+			(at 153.67 49.53 0)
 			(effects
 				(font
@@
 		)
 		(property "Datasheet" ""
-			(at 153.67 53.34 0)
+			(at 153.67 49.53 0)
 			(effects
 				(font
@@
 		)
 		(property "Description" "Power symbol creates a global label with name \"GND\" , ground"
-			(at 153.67 53.34 0)
+			(at 153.67 49.53 0)
 			(effects
 				(font

Commit message: finished routing
Parts:
- removed R34: 1.8k, Resistor_SMD:R_0402_1005Metric, symbol Device:R
Connections:
- net MIC: no longer names the net of D9.2 (A2), J4.S
Changed lines of the file:
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@@
 	)
 	(junction
-		(at 39.37 124.46)
-		(diameter 0)
-		(color 0 0 0 0)
-	)
-	(junction
 		(at 46.99 152.4)
 		(diameter 0)
@@
 	)
 	(junction
-		(at 50.8 124.46)
-		(diameter 0)
-		(color 0 0 0 0)
-	)
-	(junction
 		(at 44.45 152.4)
 		(diameter 0)
@@
 	(wire
 		(pts
-			(xy 34.29 124.46) (xy 39.37 124.46)
-		)
-		(stroke
-			(width 0)
-			(type default)
-		)
-	)
-	(wire
-		(pts
 			(xy 45.72 46.99) (xy 45.72 48.26)
 		)
@@
 	(wire
 		(pts
-			(xy 50.8 114.3) (xy 50.8 115.57)
-		)
-		(stroke
-			(width 0)
-			(type default)
-		)
-	)
-	(wire
-		(pts
 			(xy 143.51 25.4) (xy 130.81 25.4)
 		)
@@
 	(wire
 		(pts
-			(xy 50.8 123.19) (xy 50.8 124.46)
-		)
-		(stroke
-			(width 0)
-			(type default)
-		)
-	)
-	(wire
-		(pts
 			(xy 135.89 133.35) (xy 135.89 127)
 		)
@@
 	(wire
 		(pts
-			(xy 50.8 124.46) (xy 55.88 124.46)
+			(xy 39.37 124.46) (xy 55.88 124.46)
 		)
 		(stroke
@@
 	(wire
 		(pts
-			(xy 39.37 124.46) (xy 50.8 124.46)
-		)
-		(stroke
-			(width 0)
-			(type default)
-		)
-	)
-	(wire
-		(pts
 			(xy 138.43 39.37) (xy 142.24 39.37)
 		)
@@
 		)
 	)
-	(hierarchical_label "MIC"
-		(shape output)
-		(at 34.29 124.46 180)
-		(effects
-			(font
-				(size 1.27 1.27)
-			)
-			(justify right)
-		)
-	)
 	(hierarchical_label "RESETB"
 		(shape input)
@@
 	)
 	(symbol
-		(lib_id "Device:R")
-		(at 50.8 119.38 0)
-		(mirror y)
-		(unit 1)
-		(exclude_from_sim no)
-		(in_bom yes)
-		(on_board yes)
-		(dnp no)
-		(property "Reference" "R34"
-			(at 48.26 118.1099 0)
-			(effects
-				(font
-					(size 1.27 1.27)
-				)
-				(justify left)
-			)
-		)
-		(property "Value" "1.8k"
-			(at 48.26 120.6499 0)
-			(effects
-				(font
-					(size 1.27 1.27)
-				)
-				(justify left)
-			)
-		)
-		(property "Footprint" "Resistor_SMD:R_0402_1005Metric"
-			(at 52.578 119.38 90)
-			(effects
-				(font
-					(size 1.27 1.27)
-				)
-				(hide yes)
-			)
-		)
-		(property "Datasheet" "~"
-			(at 50.8 119.38 0)
-			(effects
-				(font
-					(size 1.27 1.27)
-				)
-				(hide yes)
-			)
-		)
-		(property "Description" "Resistor"
-			(at 50.8 119.38 0)
-			(effects
-				(font
-					(size 1.27 1.27)
-				)
-				(hide yes)
-			)
-		)
-		(pin "2"
-		)
-		(pin "1"
-		)
-		(instances
-			(project ""
-				(path "/bdd43acd-23c1-472b-909a-8e24eb60d56d/dd2be10c-708f-4995-b13e-6fc09628a9ce"
-					(reference "R34")
-					(unit 1)
-				)
-			)
-		)
-	)
-	(symbol
 		(lib_id "Device:C")
 		(at 21.59 52.07 0)
@@
 					(unit 1)
 				)
-			)
-		)
-	)
-	(symbol
-		(lib_id "power:+1V8")
-		(at 50.8 114.3 0)
-		(unit 1)
-		(exclude_from_sim no)
-		(in_bom yes)
-		(on_board yes)
-		(dnp no)
-		(fields_autoplaced yes)
-		(property "Reference" "#PWR096"
-			(at 50.8 118.11 0)
-			(effects
-				(font
-					(size 1.27 1.27)
-				)
-				(hide yes)
-			)
-		)
-		(property "Value" "+1V8MIC"
-			(at 50.8 109.22 0)
-			(effects
-				(font
-					(size 1.27 1.27)
-				)
-			)
-		)
-		(property "Footprint" ""
-			(at 50.8 114.3 0)
-			(effects
-				(font
-					(size 1.27 1.27)
-				)
-				(hide yes)
-			)
-		)
-		(property "Datasheet" ""
-			(at 50.8 114.3 0)
-			(effects
-				(font
-					(size 1.27 1.27)
-				)
-				(hide yes)
-			)
-		)
-		(property "Description" "Power symbol creates a global label with name \"+1V8\""
-			(at 50.8 114.3 0)
-			(effects
-				(font
-					(size 1.27 1.27)
-				)
-				(hide yes)
-			)
-		)
-		(pin "1"
-		)
-		(instances
-			(project "meko-pcb"
-				(path "/bdd43acd-23c1-472b-909a-8e24eb60d56d/dd2be10c-708f-4995-b13e-6fc09628a9ce"
-					(reference "#PWR096")
-					(unit 1)
-				)
