File: meko-pcb.kicad_pcb (KiCad board)
At the start: 2 copper layers, 225.5 x 158 mm, 170 parts, among them IC1 AS5600-ASOM, IC2 TCAL9538RSVR, IC3 LP5912-3.3DRVR, IC4 ES9218PQ, IC5 BQ27427YZFR, J1 GDEY0154D67, J2 MEM2090-00-145-00-A, J3 USB_C_Receptacle_USB2.0_16P, J4 SJ2-35954B-SMT-TR, M1 HD-EMB1204-SM, Q1 SS8050, Q2 SS8050, Q3 SS8050, Q4 Si1308EDL, SW1 SW_Push, SW2 SW_Push, SW3 SW_Push, SW4 SW_Push, SW5 SW_Push, SW6 SW_Push, SW7 SW_Push, U1 ESP32-PICO-MINI-02, U10 LP5907SNX-1.8/NOPB, U2 BQ24075RGT, U3 LP5907SNX-3.3/NOPB, U4 LP5907SNX-3.3/NOPB, U5 LP5907SNX-1.8/NOPB, U6 LP5907SNX-3.3/NOPB, U7 LP5907SNX-1.8/NOPB, U8 USBLC6-2SC6, U9 CP2102N-Axx-xQFN24, Y1 ECS-2520SMV-500-GP-TR

Commit message: added models
Parts:
- added BT1: Battery_Cell, S2B-PH-SM4-TB_LF__SN_:JST_S2B-PH-SM4-TB_LF__SN_, F.Cu at (86.5, 108.5)
- D2: footprint LED_SMD:LED_SK6805_PLCC4_2.4x2.7mm_P1.3mm -> sk6805-ec14:sk6805ec14

Commit message: started layout
Parts:
- BT1, C1, C10, C11, C12, C13, C14, C15, C16, C17, C18, C19, C2, C20, C21, C22, C23, C24, C25, C26, C27, C28, C29, C3, C30, C31, C32, C33, C34, C35, C36, C37, C38, C39, C4, C40, C41, C42, C43, C44, C45, C46, C47, C48, C49, C5, C50, C51, C52, C53, C54, C55, C56, C57, C58, C59, C6, C7, C8, C9, D1, D10, D11, D12, D13, D2, D3, D4, D5, D9, F1, IC2, IC3, IC4, IC5, J3, J4, JP1, JP10, JP2, JP3, JP4, JP5, JP6, JP7, JP8, JP9, L1, M1, Q1, Q2, Q3, R1, R10, R11, R12, R14, R15, R16, R17, R18, R19, R2, R20, R21, R22, R23, R24, R25, R26, R27, R28, R29, R3, R30, R31, R33, R34, R35, R4, R5, R6, R7, R8, R9, TP1, TP10, TP11, TP12, TP13, TP14, TP15, TP16, TP17, TP18, TP19, TP2, TP20, TP3, TP4, TP5, TP6, TP7, TP8, TP9, U1, U10, U2, U3, U4, U5, U6, U7, U8, U9, Y1: moved to B.Cu
- IC1: moved to F.Cu
- J1: footprint FH34SRJ-24S-0.5SH(99):FH34SRJ24S05SH99 -> FH34SRJ-24S-0.5SH(99):FH34SRJ24S05SH99-disp; moved to F.Cu
- moved D3 426.4 mm to (-246.3, 65.3), turned to 180 degrees
- moved D4 426.4 mm to (-246.3, 61.9), turned to 180 degrees
- moved Q4 425.0 mm to (-245.6, 69.0)
- moved JP2 416.2 mm to (-241.2, 65.6), turned to 180 degrees
- moved L1 415.5 mm to (-240.8, 68.8), turned to 180 degrees
- moved JP10 393.9 mm to (-230.0, 73.3), turned to 180 degrees
- moved D5 380.4 mm to (-223.2, 41.2), turned to 180 degrees
- moved D1 377.5 mm to (-221.8, 73.8), turned to 180 degrees
- moved D13 375.2 mm to (-220.6, 77.7), turned to 180 degrees
- moved C26 364.5 mm to (-191.0, 14.5), turned to 180 degrees
- moved R16 303.8 mm to (-184.9, 32.2), turned to 180 degrees
- moved JP9 298.1 mm to (-182.0, 20.4), turned to 180 degrees
- moved TP7 290.8 mm to (-178.3, 13.8), turned to 180 degrees
- moved D7 284.4 mm to (-175.1, 9.96)
- moved JP6 279.3 mm to (-172.6, 27.4), turned to 180 degrees
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Connections:
- C31 pad 1: +3V3AVCC -> +3V3
- C38 pad 1: +3V3AVCC -> +3V3
- JP10 pad 1: +3V3AVCC -> +3V3
- U1 pad 26: /AUDIO_DATA_2 -> /AUDIO_DATA1
- U1 pad 27: /LED -> /AUDIO_DATA_2
- U1 pad 33: /AUDIO_DATA1 -> /LED
- U10 pad 4: +3V3AVCC -> +3V3
- U5 pad 3: +3V3AVCC -> +3V3
- U5 pad 4: +3V3AVCC -> +3V3
Routing:
- added copper zone on In1.Cu, net GND
- added copper zone on In2.Cu, net GND
Other:
- board size 225.5 x 158 mm -> 40 x 85 mm
- copper layers 2 -> 4
