File: power.kicad_sch (KiCad schematic)
At the start: 51 parts, among them IC3 LP5912-3.3DRVR, IC5 BQ27427YZFR, U10 LP5907SNX-1.8/NOPB, U2 BQ24075RGT, U3 LP5907SNX-3.3/NOPB, U4 LP5907SNX-3.3/NOPB, U5 LP5907SNX-1.8/NOPB, U6 LP5907SNX-3.3/NOPB, U7 LP5907SNX-1.8/NOPB

Commit message: layout
Parts:
- removed JP4, JP5: SolderJumper_2_Bridged, Jumper:SolderJumper-2_P1.3mm_Bridged_RoundedPad1.0x1.5mm, symbol Jumper:SolderJumper_2_Bridged
- removed TP11: TestPoint, TestPoint:TestPoint_Pad_D1.5mm, symbol Connector:TestPoint
- added D14: LED, LED_SMD:LED_0201_0603Metric, symbol Device:LED
- added R32: 1.5k, Resistor_SMD:R_0402_1005Metric, symbol Device:R
Connections:
- net EN3V3MCLK is gone; now on net REG-OUT: U3.3 (EN)
- net +5V: now also U2.6 (EN1)
- net GND: now also D14.1 (K)
- net at U2.9 (~{CHG}): now also R32.1
- new net: D14.2 (A), R32.2
Other:
- moved on the sheet: C23, C24, C25, C26, R16, R17, R18, R19, R20, TP10, U2

Commit message: more layout
Parts:
- removed C30, C35, C37, C39: 1uF, Capacitor_SMD:C_0402_1005Metric, symbol Device:C

Commit message: more layout
Parts:
- removed C59: 1uF, Capacitor_SMD:C_0402_1005Metric, symbol Device:C
- C33: value 1uF -> 4.7uF
- D14: footprint LED_SMD:LED_0201_0603Metric -> LED_SMD:LED_0603_1608Metric
Other:
- moved on the sheet: C24, C25, C26

Commit message: more routing
Connections:
- net +3V3: no longer C31.1, C38.1, JP10.1 (A), U10.4 (VIN), U5.3 (EN), U5.4 (VIN)
- net REG-OUT: now also C31.1, C38.1, JP10.1 (A), U10.4 (VIN), U5.3 (EN), U5.4 (VIN)
Other:
- moved on the sheet: TP18

Commit message: finished routing
Parts:
- removed C31, C32: 1uF, Capacitor_SMD:C_0402_1005Metric, symbol Device:C
- removed TP12, TP14, TP15: TestPoint, TestPoint:TestPoint_Pad_D1.5mm, symbol Connector:TestPoint
- removed U5: LP5907SNX-1.8/NOPB, Package_SON:Texas_X2SON-4_1x1mm_P0.65mm, symbol LP5907SNX-1-8-NOPB:LP5907SNX-1.8_NOPB
- TP10, TP13, TP16, TP17, TP18: footprint TestPoint:TestPoint_Pad_D1.5mm -> TestPoint:TestPoint_Pad_D1.0mm

Commit message: minor stuff
Connections:
- net +BATT: no longer U2.2 (BAT), U2.3 (BAT)
- net REG-OUT: no longer IC5.C2 (SRX)
- new net SRX: IC5.C2 (SRX), U2.2 (BAT), U2.3 (BAT)
Changed lines of the file:
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@@
 	(wire
 		(pts
-			(xy 207.01 59.69) (xy 213.36 59.69)
-		)
-		(stroke
-			(width 0)
-			(type default)
-		)
-	)
-	(wire
-		(pts
 			(xy 38.1 142.24) (xy 36.83 142.24)
 		)
@@
 	(wire
 		(pts
-			(xy 92.71 33.02) (xy 95.25 33.02)
+			(xy 92.71 33.02) (xy 99.06 33.02)
 		)
 		(stroke
@@
 	(wire
 		(pts
-			(xy 207.01 57.15) (xy 204.47 57.15)
+			(xy 204.47 57.15) (xy 213.36 57.15)
 		)
 		(stroke
@@
 	(wire
 		(pts
-			(xy 207.01 59.69) (xy 207.01 57.15)
-		)
-		(stroke
-			(width 0)
-			(type default)
-		)
-	)
-	(wire
-		(pts
 			(xy 154.94 90.17) (xy 157.48 90.17)
 		)
@@
 	(wire
 		(pts
-			(xy 95.25 31.75) (xy 95.25 33.02)
-		)
-		(stroke
-			(width 0)
-			(type default)
-		)
-	)
-	(wire
-		(pts
 			(xy 157.48 152.4) (xy 157.48 154.94)
 		)
@@
 		)
 	)
+	(label "SRX"
+		(at 99.06 33.02 180)
+		(effects
+			(font
+				(size 1.27 1.27)
+			)
+			(justify right bottom)
+		)
+	)
 	(label "ILIM"
 		(at 54.61 43.18 0)
@@
 		)
 	)
+	(label "SRX"
+		(at 213.36 57.15 180)
+		(effects
+			(font
+				(size 1.27 1.27)
+			)
+			(justify right bottom)
+		)
+	)
 	(label "TMR"
 		(at 39.37 31.75 0)
@@
 	)
 	(symbol
-		(lib_id "power:+BATT")
-		(at 95.25 31.75 0)
-		(unit 1)
-		(exclude_from_sim no)
-		(in_bom yes)
-		(on_board yes)
-		(dnp no)
-		(property "Reference" "#PWR0108"
-			(at 95.25 35.56 0)
-			(effects
-				(font
-					(size 1.27 1.27)
-				)
-				(hide yes)
-			)
-		)
-		(property "Value" "+BATT"
-			(at 94.488 28.194 0)
-			(effects
-				(font
-					(size 1.27 1.27)
-				)
-			)
-		)
-		(property "Footprint" ""
-			(at 95.25 31.75 0)
-			(effects
-				(font
-					(size 1.27 1.27)
-				)
-				(hide yes)
-			)
-		)
-		(property "Datasheet" ""
-			(at 95.25 31.75 0)
-			(effects
-				(font
-					(size 1.27 1.27)
-				)
-				(hide yes)
-			)
-		)
-		(property "Description" "Power symbol creates a global label with name \"+BATT\""
-			(at 95.25 31.75 0)
-			(effects
-				(font
-					(size 1.27 1.27)
-				)
-				(hide yes)
-			)
-		)
-		(pin "1"
-		)
-		(instances
-			(project "meko-pcb"
-				(path "/bdd43acd-23c1-472b-909a-8e24eb60d56d/8a6dc5b3-4f2f-4276-a496-11a08be250c4"
-					(reference "#PWR0108")
-					(unit 1)
-				)
-			)
-		)
-	)
-	(symbol
 		(lib_id "power:GND")
 		(at 110.49 140.97 0)
@@
 					(unit 1)
 				)
-			)
-		)
-	)
-	(symbol
-		(lib_id "power:+BATT")
-		(at 213.36 59.69 0)
-		(unit 1)
-		(exclude_from_sim no)
-		(in_bom yes)
-		(on_board yes)
-		(dnp no)
-		(property "Reference" "#PWR0117"
-			(at 213.36 63.5 0)
-			(effects
-				(font
-					(size 1.27 1.27)
-				)
-				(hide yes)
-			)
-		)
-		(property "Value" "REG-OUT"
-			(at 213.614 56.388 0)
-			(effects
-				(font
-					(size 1.27 1.27)
-				)
-			)
-		)
-		(property "Footprint" ""
-			(at 213.36 59.69 0)
-			(effects
-				(font
-					(size 1.27 1.27)
-				)
-				(hide yes)
-			)
-		)
-		(property "Datasheet" ""
-			(at 213.36 59.69 0)
-			(effects
-				(font
-					(size 1.27 1.27)
-				)
-				(hide yes)
-			)
-		)
-		(property "Description" "Power symbol creates a global label with name \"+BATT\""
-			(at 213.36 59.69 0)
-			(effects
-				(font
-					(size 1.27 1.27)
-				)
-				(hide yes)
-			)
-		)
-		(pin "1"
-		)
-		(instances
-			(project "meko-pcb"
-				(path "/bdd43acd-23c1-472b-909a-8e24eb60d56d/8a6dc5b3-4f2f-4276-a496-11a08be250c4"
-					(reference "#PWR0117")
-					(unit 1)
-				)
