File: meko-pcb/usb.kicad_sch (KiCad schematic)
At the start: 13 parts, among them J3 USB_C_Receptacle_USB2.0_16P, U8 USBLC6-2SC6, U9 CP2102N-Axx-xQFN24

Commit message: component selection
Parts:
- F1: Mfr. No. (none) -> MF-FSMF050X-2
- J3: Mfr. No. (none) -> USB4105-GF-A
- R21, R22, R23, R24: Mfr. No. (none) -> CRCW040210K0FKED
- R25, R26: Mfr. No. (none) -> RC0402FR-075K1L
- TP5, TP7: now left out of the parts list
- U8: Mfr. No. (none) -> USBLC6-2SC6
- U9: Mfr. No. (none) -> CP2102N-A02-GQFN24R
Changed lines of the file:
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@@
+			)
+		)
+		(property "Mfr. No." "RC0402FR-075K1L"
+			(at 52.07 73.66 0)
+			(effects
+				(font
+					(size 1.27 1.27)
+				)
+				(hide yes)
 			)
 		)
@@
 			)
 		)
+		(property "Mfr. No." "CRCW040210K0FKED"
+			(at 128.27 21.59 0)
+			(effects
+				(font
+					(size 1.27 1.27)
+				)
+				(hide yes)
+			)
+		)
 		(pin "2"
 		)
@@
 		)
 		(property "LCSC" "C25905"
+			(at 41.91 73.66 0)
+			(effects
+				(font
+					(size 1.27 1.27)
+				)
+				(hide yes)
+			)
+		)
+		(property "Mfr. No." "RC0402FR-075K1L"
 			(at 41.91 73.66 0)
 			(effects
@@
 			)
 		)
+		(property "Mfr. No." "CRCW040210K0FKED"
+			(at 167.64 31.75 0)
+			(effects
+				(font
+					(size 1.27 1.27)
+				)
+				(hide yes)
+			)
+		)
 		(pin "2"
 		)
@@
 			)
 		)
+		(property "Mfr. No." "CRCW040210K0FKED"
+			(at 163.83 57.15 0)
+			(effects
+				(font
+					(size 1.27 1.27)
+				)
+				(hide yes)
+			)
+		)
 		(pin "2"
 		)
@@
 			)
 		)
+		(property "Mfr. No." "MF-FSMF050X-2"
+			(at 50.8 30.48 90)
+			(effects
+				(font
+					(size 1.27 1.27)
+				)
+				(hide yes)
+			)
+		)
 		(pin "1"
 		)
@@
 		(unit 1)
 		(exclude_from_sim no)
-		(in_bom yes)
+		(in_bom no)
 		(on_board yes)
 		(dnp no)
@@
 			)
 		)
+		(property "Mfr. No." "CP2102N-A02-GQFN24R "
+			(at 142.24 49.53 0)
+			(effects
+				(font
+					(size 1.27 1.27)
+				)
+				(hide yes)
+			)
+		)
 		(pin "8"
 		)
@@
 		)
 		(property "LCSC" "C7519"
+			(at 86.36 30.48 0)
+			(effects
+				(font
+					(size 1.27 1.27)
+				)
+				(hide yes)
+			)
+		)
+		(property "Mfr. No." "USBLC6-2SC6"
 			(at 86.36 30.48 0)
 			(effects
@@
 			)
 		)
+		(property "Mfr. No." "USB4105-GF-A"
+			(at 30.48 45.72 0)
+			(effects
+				(font
+					(size 1.27 1.27)
+				)
+				(hide yes)
+			)
+		)
 		(pin "B1"
 		)
@@
 			)
 		)
+		(property "Mfr. No." "CRCW040210K0FKED"
+			(at 176.53 57.15 0)
+			(effects
+				(font
+					(size 1.27 1.27)
+				)
+				(hide yes)
+			)
+		)
 		(pin "2"
 		)
@@
 		(unit 1)
 		(exclude_from_sim no)
-		(in_bom yes)
-		(on_board yes)
-		(dnp no)
+		(in_bom no)
+		(on_board yes)
+		(dnp no)

Commit message: picked MPNs
Parts:
- C40: MPN (none) -> CL05A106MQ5NUNC
- F1: MPN (none) -> MF-FSMF050X-2; Mfr. No. MF-FSMF050X-2 -> (none)
- J3: MPN (none) -> USB4105-GF-A; Mfr. No. USB4105-GF-A -> (none)
- R21, R22, R23, R24: MPN (none) -> CRCW040210K0FKED; Mfr. No. CRCW040210K0FKED -> (none)
- R25, R26: MPN (none) -> RC0402FR-075K1L; Mfr. No. RC0402FR-075K1L -> (none)
- U8: MPN (none) -> USBLC6-2SC6; Mfr. No. USBLC6-2SC6 -> (none)
- U9: MPN (none) -> CP2102N-A02-GQFN24R; Mfr. No. CP2102N-A02-GQFN24R -> (none)
Changed lines of the file:
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@@
 			)
 		)
-		(property "Mfr. No." "RC0402FR-075K1L"
+		(property "MPN" "RC0402FR-075K1L"
 			(at 52.07 73.66 0)
 			(effects
@@
 			)
 		)
-		(property "Mfr. No." "CRCW040210K0FKED"
+		(property "MPN" "CRCW040210K0FKED"
 			(at 128.27 21.59 0)
 			(effects
@@
 			)
 		)
-		(property "Mfr. No." "RC0402FR-075K1L"
+		(property "MPN" "RC0402FR-075K1L"
 			(at 41.91 73.66 0)
 			(effects
@@
 			)
 		)
-		(property "Mfr. No." "CRCW040210K0FKED"
+		(property "MPN" "CRCW040210K0FKED"
 			(at 167.64 31.75 0)
 			(effects
@@
 			)
 		)
-		(property "Mfr. No." "CRCW040210K0FKED"
+		(property "MPN" "CRCW040210K0FKED"
 			(at 163.83 57.15 0)
 			(effects
@@
 			)
 		)
-		(property "Mfr. No." "MF-FSMF050X-2"
+		(property "MPN" "MF-FSMF050X-2"
 			(at 50.8 30.48 90)
 			(effects
@@
 			)
 		)
+		(property "MPN" "CL05A106MQ5NUNC"
+			(at 64.77 35.56 0)
+			(effects
+				(font
+					(size 1.27 1.27)
+				)
+				(hide yes)
+			)
+		)
 		(pin "1"
 		)
@@
 			)
 		)
-		(property "Mfr. No." "CP2102N-A02-GQFN24R "
+		(property "MPN" "CP2102N-A02-GQFN24R "
 			(at 142.24 49.53 0)
 			(effects
@@
 			)
 		)
-		(property "Mfr. No." "USBLC6-2SC6"
+		(property "MPN" "USBLC6-2SC6"
 			(at 86.36 30.48 0)
 			(effects
@@
 			)
 		)
-		(property "Mfr. No." "USB4105-GF-A"
+		(property "MPN" "USB4105-GF-A"
 			(at 30.48 45.72 0)
 			(effects
@@
 			)
 		)
-		(property "Mfr. No." "CRCW040210K0FKED"
+		(property "MPN" "CRCW040210K0FKED"
 			(at 176.53 57.15 0)
 			(effects

Commit message: readme updates, removed unused fileds form kicad
Parts:
- F1: LCSC C210357 -> (none)
- R25, R26: LCSC C25905 -> (none)
- U8: LCSC C7519 -> (none)
Changed lines of the file:
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@@
-			)
-		)
-		(property "LCSC" "C25905"
-			(at 52.07 73.66 0)
-			(effects
-				(font
-					(size 1.27 1.27)
-				)
-				(hide yes)
 			)
 		)
@@
 			)
 		)
-		(property "LCSC" "C25905"
-			(at 41.91 73.66 0)
-			(effects
-				(font
-					(size 1.27 1.27)
-				)
-				(hide yes)
-			)
-		)
 		(property "MPN" "RC0402FR-075K1L"
 			(at 41.91 73.66 0)
@@
 			)
 		)
-		(property "LCSC" "C210357"
-			(at 50.8 30.48 90)
-			(effects
-				(font
-					(size 1.27 1.27)
-				)
-				(hide yes)
-			)
-		)
 		(property "MPN" "MF-FSMF050X-2"
 			(at 50.8 30.48 90)
@@
 			(at 86.36 30.48 0)
 			(effects
-				(font
-					(size 1.27 1.27)
-				)
-				(hide yes)
-			)
-		)
-		(property "LCSC" "C7519"
-			(at 86.36 30.48 0)
-			(effects
