File: meko-pcb/meko-pcb.kicad_sch (KiCad schematic)
At the start: 83 parts, among them IC1 AS5600-ASOM, IC2 TCAL9538RSVR, J1 GDEY0154D67, J2 MEM2090-00-145-00-A, M1 HD-EMB1204-SM, Q1 SS8050, Q2 SS8050, Q3 SS8050, Q4 Si1308EDL, SW1 SW_Push, SW2 SW_Push, SW3 SW_Push, SW4 SW_Push, SW5 SW_Push, SW6 SW_Push, SW7 SW_Push, U1 ESP32-PICO-MINI-02

Commit message: component selection
Parts:
- IC1: Manufacturer_Part_Number AS5600-ASOM -> (none); Mfr. No. (none) -> AS5600-ASOM
- IC2: Manufacturer_Part_Number TCAL9538RSVR -> (none); Mfr. No. (none) -> TCAL9538RSVR
- J1: Manufacturer_Part_Number FH34SRJ-24S-0.5SH(99) -> (none); Mfr. No. (none) -> FH34SRJ-24S-0.5SH(99)
- J2: Manufacturer_Part_Number MEM2090-00-145-00-A -> (none); Mfr. No. (none) -> MEM2090-00-145-00-A
- L1: Mfr. No. (none) -> MLZ2012M470WT000
- M1: Mfr. No. (none) -> HD-EMB1204-SM
- Q1, Q2, Q3: Mfr. No. (none) -> SS8050-HF
- Q4: Mfr. No. (none) -> SI1308EDL-T1-GE3
- R1, R10, R11, R14, R15, R2, R3, R4, R5, R6, R7, R8: Mfr. No. (none) -> CRCW040210K0FKED
- R12: Mfr. No. (none) -> RC0402FR-071ML
- R13: Mfr. No. (none) -> RC0402FR-072R2L
- R30: Mfr. No. (none) -> RC0402FR-07100KL
- R9: Mfr. No. (none) -> RC0402FR-071KL
- SW1, SW2, SW3, SW4, SW5: Mfr. No. (none) -> SKRTLAE010
- SW6, SW7: Mfr. No. (none) -> SKRKAGE020
- TP1, TP19, TP2, TP20, TP21, TP22, TP3, TP4, TP6: now left out of the parts list
- U1: Mfr. No. (none) -> ESP32-PICO-MINI-02-N8R2

Commit message: picked MPNs
Parts:
- C1, C2, C3, C30, C4, C5, C6, C61, C7, C8: MPN (none) -> CL05B104KO5NNNC
- C10, C11, C12, C13, C14, C15, C16, C17, C18, C19, C20, C21, C22, C9: MPN (none) -> CL05A105KO5NNNC
- C60: MPN (none) -> CL05A475KP5NRNC
- D1: MPN (none) -> US1B
- D2: MPN (none) -> SK6805-EC14
- D3, D4, D5: MPN (none) -> MBR0530T1G
- D6, D7, D8: MPN (none) -> D3V3F8U9LP3810-7; Mfr. No. D3V3F8U9LP3810-7 -> (none)
- IC1: MPN (none) -> AS5600-ASOM; Mfr. No. AS5600-ASOM -> (none); Mouser Part Number 985-AS5600-ASOM -> (none); Mouser Price/Stock https://www.mouser.co.uk/ProductDetail/ams-OSRAM/AS5600-ASO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 -> (none)
- IC2: MPN (none) -> TCAL9538RSVR; Mfr. No. TCAL9538RSVR -> (none); Mouser Part Number 595-TCAL9538RSVR -> (none); Mouser Price/Stock https://www.mouser.co.uk/ProductDetail/Texas-Instruments/TC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 -> (none)
- J1: MPN (none) -> FH34SRJ-24S-0.5SH(99); Mfr. No. FH34SRJ-24S-0.5SH(99) -> (none); Mouser Part Number 798-FH34SRJ24S05SH99 -> (none); Mouser Price/Stock https://www.mouser.co.uk/ProductDetail/Hirose-Connector/FH3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 -> (none)
- J2: MPN (none) -> MEM2090-00-145-00-A; Mfr. No. MEM2090-00-145-00-A -> (none); Mouser Part Number 640-MEM20900014500A -> (none); Mouser Price/Stock https://www.mouser.co.uk/ProductDetail/GCT/MEM2090-00-145-0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 -> (none)
- L1: MPN (none) -> MLZ2012M470WT000; Mfr. No. MLZ2012M470WT000 -> (none)
- M1: DigiKey_Part_Number 668-HD-EMB1204-SMTR-ND -> (none); MANUFACTURER PUI Audio -> (none); MF PUI Audio -> (none); MP HD-EMB1204-SM -> (none); MPN (none) -> HD-EMB1204-SM; Mfr. No. HD-EMB1204-SM -> (none)
- Q1, Q2, Q3: MPN (none) -> SS8050-HF; Mfr. No. SS8050-HF -> (none)
- Q4: MPN (none) -> SI1308EDL-T1-GE3; Mfr. No. SI1308EDL-T1-GE3 -> (none)
- R1, R10, R11, R14, R15, R2, R3, R4, R5, R6, R7, R8: MPN (none) -> CRCW040210K0FKED; Mfr. No. CRCW040210K0FKED -> (none)
- R12: MPN (none) -> RC0402FR-071ML; Mfr. No. RC0402FR-071ML -> (none)
- R13: MPN (none) -> RC0402FR-072R2L; Mfr. No. RC0402FR-072R2L -> (none)
- R30: MPN (none) -> RC0402FR-07100KL; Mfr. No. RC0402FR-07100KL -> (none)
- R9: MPN (none) -> RC0402FR-071KL; Mfr. No. RC0402FR-071KL -> (none)
- SW1, SW2, SW3, SW4, SW5: MPN (none) -> SKRTLAE010; Mfr. No. SKRTLAE010 -> (none)
- SW6, SW7: MPN (none) -> SKRKAGE020; Mfr. No. SKRKAGE020 -> (none)
- U1: MPN (none) -> ESP32-PICO-MINI-02-N8R2; Mfr. No. ESP32-PICO-MINI-02-N8R2 -> (none)

Commit message: 3d stuff, fixes
Parts:
- added H5: MountingHole, Library:MountingHole_1.8mm_M1.6, symbol Mechanical:MountingHole
- H1, H2, H3, H4: footprint MountingHole:MountingHole_2.2mm_M2 -> Library:MountingHole_1.8mm_M1.6
Changed lines of the file:
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@@
 	(rectangle
 		(start 50.8 130.81)
-		(end 85.09 140.335)
+		(end 95.885 140.335)
 		(stroke
 			(width 0)
@@
 	(text "HOLES"
 		(exclude_from_sim no)
-		(at 78.232 134.366 0)
+		(at 84.836 134.366 0)
 		(effects
 			(font
@@
 	)
 	(symbol
+		(lib_id "Mechanical:MountingHole")
+		(at 74.93 134.62 0)
+		(unit 1)
+		(exclude_from_sim no)
+		(in_bom no)
+		(on_board yes)
+		(dnp no)
+		(property "Reference" "H5"
+			(at 73.66 138.176 0)
+			(effects
+				(font
+					(size 1.27 1.27)
+				)
+				(justify left)
+			)
+		)
+		(property "Value" "MountingHole"
+			(at 77.47 135.8899 0)
+			(effects
+				(font
+					(size 1.27 1.27)
+				)
+				(justify left)
+				(hide yes)
+			)
+		)
+		(property "Footprint" "Library:MountingHole_1.8mm_M1.6"
+			(at 74.93 134.62 0)
+			(effects
+				(font
+					(size 1.27 1.27)
+				)
+				(hide yes)
+			)
+		)
+		(property "Datasheet" "~"
+			(at 74.93 134.62 0)
+			(effects
+				(font
+					(size 1.27 1.27)
+				)
+				(hide yes)
+			)
+		)
+		(property "Description" "Mounting Hole without connection"
+			(at 74.93 134.62 0)
+			(effects
+				(font
+					(size 1.27 1.27)
+				)
+				(hide yes)
+			)
+		)
+		(instances
+			(project "meko-pcb"
+				(path "/bdd43acd-23c1-472b-909a-8e24eb60d56d"
+					(reference "H5")
+					(unit 1)
+				)
+			)
+		)
+	)
+	(symbol
 		(lib_id "power:+3V3")
 		(at 196.85 111.76 0)
@@
 			)
 		)
-		(property "Footprint" "MountingHole:MountingHole_2.2mm_M2"
+		(property "Footprint" "Library:MountingHole_1.8mm_M1.6"
 			(at 59.69 134.62 0)
 			(effects
@@
 			)
 		)
-		(property "Footprint" "MountingHole:MountingHole_2.2mm_M2"
+		(property "Footprint" "Library:MountingHole_1.8mm_M1.6"
 			(at 69.85 134.62 0)
 			(effects
@@
 			)
 		)
-		(property "Footprint" "MountingHole:MountingHole_2.2mm_M2"
+		(property "Footprint" "Library:MountingHole_1.8mm_M1.6"
 			(at 64.77 134.62 0)
 			(effects
@@
 			)
 		)
-		(property "Footprint" "MountingHole:MountingHole_2.2mm_M2"
+		(property "Footprint" "Library:MountingHole_1.8mm_M1.6"
 			(at 54.61 134.62 0)
 			(effects

Commit message: readme updates, removed unused fileds form kicad
Parts:
- C60: LCSC C307423 -> (none)
- IC1: Arrow Part Number AS5600-ASOM -> (none); Arrow Price/Stock https://www.arrow.com/en/products/as5600-asom/ams-osram?utm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 -> (none); Height 1.75 -> (none); Manufacturer_Name ams OSRAM -> (none)
- IC2: Height 0.55 -> (none); Manufacturer_Name Texas Instruments -> (none)
- J1: Height 1.1 -> (none); Manufacturer_Name Hirose -> (none)
- J2: Height 1.6 -> (none); Manufacturer_Name GCT (GLOBAL CONNECTOR TECHNOLOGY) -> (none)
- M1: Check_prices https://www.snapeda.com/parts/HD-EMB1204-SM/PUI+Audio/view-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 -> (none); Description_1 12X4MM ERM HAPTIC 12000RPM -> (none); MAXIMUM_PACKAGE_HEIGHT 3.4 mm -> (none); PARTREV A -> (none); Package None -> (none); STANDARD Manufacturer Recommendations -> (none); SnapEDA_Link https://www.snapeda.com/parts/HD-EMB1204-SM/PUI+Audio/view-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 -> (none)
Changed lines of the file:
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@@
 			)
 		)
-		(property "LCSC" "C307423"
-			(at 118.11 24.13 0)
-			(effects
-				(font
-					(size 1.27 1.27)
-				)
-				(hide yes)
-			)
-		)
 		(property "MPN" "CL05A475KP5NRNC"
 			(at 118.11 24.13 0)
@@
 			)
 		)
-		(property "Height" "0.55"
-			(at 156.21 542.24 0)
-			(effects
-				(font
-					(size 1.27 1.27)
-				)
-				(justify left top)
-				(hide yes)
-			)
-		)
-		(property "Manufacturer_Name" "Texas Instruments"
-			(at 156.21 642.24 0)
-			(effects
-				(font
-					(size 1.27 1.27)
-				)
-				(justify left top)
-				(hide yes)
-			)
-		)
-		(property "Arrow Part Number" ""
-			(at 156.21 1042.24 0)
-			(effects
-				(font
-					(size 1.27 1.27)
-				)
-				(justify left top)
-				(hide yes)
-			)
-		)
-		(property "Arrow Price/Stock" ""
-			(at 156.21 1142.24 0)
-			(effects
-				(font
-					(size 1.27 1.27)
-				)
-				(justify left top)
-				(hide yes)
-			)
-		)
 		(property "MPN" "TCAL9538RSVR"
 			(at 129.54 154.94 0)
@@
 			)
 		)
-		(property "Height" "1.6"
-			(at 69.85 549.86 0)
-			(effects
-				(font
-					(size 1.27 1.27)
-				)
-				(justify left top)
-				(hide yes)
-			)
-		)
-		(property "Manufacturer_Name" "GCT (GLOBAL CONNECTOR TECHNOLOGY)"
-			(at 69.85 649.86 0)
-			(effects
-				(font
-					(size 1.27 1.27)
-				)
-				(justify left top)
-				(hide yes)
-			)
-		)
-		(property "Arrow Part Number" ""
-			(at 69.85 1049.86 0)
-			(effects
-				(font
-					(size 1.27 1.27)
-				)
-				(justify left top)
-				(hide yes)
-			)
-		)
-		(property "Arrow Price/Stock" ""
-			(at 69.85 1149.86 0)
-			(effects
-				(font
-					(size 1.27 1.27)
-				)
-				(justify left top)
-				(hide yes)
-			)
-		)
 		(property "MPN" "MEM2090-00-145-00-A"
 			(at 35.56 154.94 0)
@@
 			)
 		)
-		(property "Height" "1.1"
-			(at 283.21 506.68 0)
-			(effects
-				(font
-					(size 1.27 1.27)
-				)
-				(justify left top)
-				(hide yes)
-			)
-		)
-		(property "Manufacturer_Name" "Hirose"
-			(at 283.21 606.68 0)
-			(effects
-				(font
-					(size 1.27 1.27)
-				)
-				(justify left top)
-				(hide yes)
-			)
-		)
-		(property "Arrow Part Number" ""
-			(at 283.21 1006.68 0)
-			(effects
-				(font
-					(size 1.27 1.27)
-				)
-				(justify left top)
-				(hide yes)
-			)
-		)
-		(property "Arrow Price/Stock" ""
-			(at 283.21 1106.68 0)
-			(effects
-				(font
-					(size 1.27 1.27)
-				)
-				(justify left top)
-				(hide yes)
-			)
-		)
 		(property "MPN" "FH34SRJ-24S-0.5SH(99)"
 			(at 261.62 111.76 0)
@@
 			)
 		)
-		(property "SnapEDA_Link" "https://www.snapeda.com/parts/HD-EMB1204-SM/PUI+Audio/view-part/?ref=snap"
-			(at 86.36 102.87 0)
-			(effects
-				(font
-					(size 1.27 1.27)
-				)
-				(justify bottom)
-				(hide yes)
-			)
-		)
-		(property "MAXIMUM_PACKAGE_HEIGHT" "3.4 mm"
-			(at 86.36 102.87 0)
-			(effects
-				(font
-					(size 1.27 1.27)
-				)
-				(justify bottom)
-				(hide yes)
-			)
-		)
-		(property "Package" "None"
-			(at 86.36 102.87 0)
-			(effects
-				(font
-					(size 1.27 1.27)
-				)
-				(justify bottom)
-				(hide yes)
-			)
-		)
-		(property "Check_prices" "https://www.snapeda.com/parts/HD-EMB1204-SM/PUI+Audio/view-part/?ref=eda"
-			(at 86.36 102.87 0)
-			(effects
-				(font
-					(size 1.27 1.27)
-				)
-				(justify bottom)
-				(hide yes)
-			)
-		)
-		(property "STANDARD" "Manufacturer Recommendations"
-			(at 86.36 102.87 0)
-			(effects
-				(font
-					(size 1.27 1.27)
-				)
-				(justify bottom)
-				(hide yes)
-			)
-		)
-		(property "PARTREV" "A"
-			(at 86.36 102.87 0)
-			(effects
-				(font
-					(size 1.27 1.27)
-				)
-				(justify bottom)
-				(hide yes)
-			)
-		)
-		(property "Description_1" "12X4MM ERM HAPTIC 12000RPM"
-			(at 86.36 102.87 0)
-			(effects
-				(font
-					(size 1.27 1.27)
-				)
-				(justify bottom)
-				(hide yes)
-			)
-		)
 		(property "MPN" " HD-EMB1204-SM "
 			(at 86.36 102.87 0)
@@
 				(hide yes)
 			)
-		)
-		(property "Height" "1.75"
-			(at 168.91 496.52 0)
-			(effects
-				(font
-					(size 1.27 1.27)
-				)
-				(justify left top)
-				(hide yes)
-			)
-		)
-		(property "Manufacturer_Name" "ams OSRAM"
-			(at 168.91 596.52 0)
-			(effects
-				(font
-					(size 1.27 1.27)
-				)
-				(justify left top)
-				(hide yes)
-			)
-		)
-		(property "Arrow Part Number" "AS5600-ASOM"
-			(at 168.91 996.52 0)
-			(effects
-				(font
-					(size 1.27 1.27)
-				)
-				(justify left top)
-				(hide yes)
-			)
-		)
-		(property "Arrow Price/Stock" "https://www.arrow.com/en/products/as5600-asom/ams-osram?utm_currency=USD&region=nac"
-			(at 168.91 1096.52 0)
-			(effects
-				(font
-					(size 1.27 1.27)
-				)
-				(justify left top)
-				(hide yes)
-			)

Commit message: started to implement nrf53
Parts:
- removed IC2: TCAL9538RSVR, TCAL9538RSVR:QFN40P180X260X55-16N, symbol TCAL9538RSVR:TCAL9538RSVR
- removed Q1, Q2: SS8050, Package_TO_SOT_SMD:SOT-23, symbol Transistor_BJT:SS8050
- removed R1, R14, R15, R2, R3, R4, R5, R6, R7, R8: 10k, Resistor_SMD:R_0402_1005Metric, symbol Device:R
- removed R30: 100k, Resistor_SMD:R_0402_1005Metric, symbol Device:R
- removed SW7: SW_Push, Button_Switch_SMD:SW_Push_SPST_NO_Alps_SKRK, symbol Switch:SW_Push
- removed TP1, TP2, TP3, TP4, TP6: TestPoint, TestPoint:TestPoint_Pad_D1.0mm, symbol Connector:TestPoint
- removed U1: ESP32-PICO-MINI-02, PCM_Espressif:ESP32-PICO-MINI-02, symbol PCM_Espressif:ESP32-PICO-MINI-02
- added C31, C32: 12pF, Capacitor_SMD:C_0402_1005Metric, symbol Device:C
- added C35, C37, C39, C59, C62, C63: 100nF, Capacitor_SMD:C_0402_1005Metric, symbol Device:C
- added C40: 10uF, Capacitor_SMD:C_0402_1005Metric, symbol Device:C
- added F1: 500mA, Fuse:Fuse_0603_1608Metric, symbol Device:Fuse
- added J3: USB_C_Receptacle_USB2.0_16P, Connector_USB:USB_C_Receptacle_GCT_USB4105-xx-A_16P_TopMnt_Horizontal, symbol Connector:USB_C_Receptacle_USB2.0_16P
- added R25, R26: 5.1k, Resistor_SMD:R_0402_1005Metric, symbol Device:R
- added U1: nRF5340-QKxx, Package_DFN_QFN:Nordic_AQFN-94-1EP_7x7mm_P0.4mm, symbol MCU_Nordic:nRF5340-QKxx
- added Y2: 32MHz, Crystal:Crystal_SMD_2520-4Pin_2.5x2.0mm, symbol Device:Crystal_GND24
- added Y4: 32.768 kHz, Crystal:Crystal_SMD_3215-2Pin_3.2x1.5mm, symbol Device:Crystal
- C15: value 1uF -> 12pF; LCSC (none) -> C106201; MPN CL05A105KO5NNNC -> (none)
- C6: value 100nF -> 12pF; LCSC (none) -> C106201; MPN CL05B104KO5NNNC -> (none)
- C60: value 4.7uF -> 100nF; MPN CL05A475KP5NRNC -> CL05B104KO5NNNC
Connections:
- net +3V3: no longer C15.2, C60.2, C61.1
- net AUDIO_DATA_CLK/BOOT: no longer C7.1
- net ESP_EN: no longer C6.1
- net GND: now also C15.2, C6.1, C31.2, C32.1, C40.2, J3.A1 (GND), J3.A12 (GND), J3.B1 (GND), J3.B12 (GND), J3.S1 (SHIELD), R25.2, R26.2, Y2.2, Y2.4; no longer C15.1, C6.2, C60.1, C61.2
- new net: U1.A19 (VDD), U1.AC1 (VDD), U1.AG1 (VDD), U1.AJ31 (VDD), U1.AL11 (VDD), U1.AL17 (VDD), U1.AL25 (VDD), U1.AL3 (VDD), U1.AL7 (VDD), U1.B28 (VDD), U1.B8 (VDD), U1.C1 (VDD), U1.E31 (VDD), U1.L1 (VDD), U1.N31 (VDD), U1.U1 (VDD)
- new net: F1.2, J3.A4 (VBUS), J3.A9 (VBUS), J3.B4 (VBUS), J3.B9 (VBUS)
- new net +5V: C40.1, F1.1
- new net CC1: J3.B5 (CC2), R25.1
- new net CC2: J3.A5 (CC1), R26.1
- new net D+: J3.A6 (D+), J3.B6 (D+)
- new net D-: J3.A7 (D-), J3.B7 (D-)
- new net XC1: C15.1, Y2.1
- new net XC2: C31.1, Y2.3
- new net XL1: C32.2, Y4.2
- new net XL2: C6.2, Y4.1
- no-connect marks 6 -> 7
Other:
- removed sheet USB
- note added: "External crystal C"
- note added: "External crystal L"
- note added: "USB PORT"
- note removed: "USB"
- note removed: "addr(dec.):112"

Commit message: continued work om nrf53
Parts:
- added AE1: Antenna_Chip, symbol Device:Antenna_Chip
- added C64, C70: 100nF, Capacitor_SMD:C_0402_1005Metric, symbol Device:C
- added C65: 0.7pF, Capacitor_SMD:C_0402_1005Metric, symbol Device:C
- added C66: N.C., Capacitor_SMD:C_0402_1005Metric, symbol Device:C
- added C67: 2.2nF, Capacitor_SMD:C_0402_1005Metric, symbol Device:C
- added C68, C69: 1uF, Capacitor_SMD:C_0402_1005Metric, symbol Device:C
- added C71, C72: 4.7uF, Capacitor_SMD:C_0402_1005Metric, symbol Device:C
- added L2, L3, L4: 10uH, symbol Device:L
- added R1: 2.2R, symbol Device:R
Connections:
- net D+: now also U1.B2 (D+)
- net D-: now also U1.B4 (D-)
- net GND: now also C32.2, C35.2, C37.2, C39.2, C59.2, C6.2, C60.2, C61.2, C62.2, C63.2, C64.2, C65.2, C66.2, C67.2, C68.2, C69.2, C70.2, C71.2, C72.2; no longer C32.1, C6.1
- net XC1: now also U1.C31 (XC1)
- net XC2: now also U1.B30 (XC2)
- net XL1: now also C32.1, U1.N1 (XL1/P0.00), Y4.1; no longer C32.2, Y4.2
- net XL2: now also C6.1, U1.R1 (XL2/P0.01), Y4.2; no longer C6.2, Y4.1
- net at C39.1: now also C35.1, C37.1, C59.1, C60.1, C61.1, C62.1, C63.1, U1.A19 (VDD), U1.AC1 (VDD), U1.AG1 (VDD), U1.AJ31 (VDD), U1.AL11 (VDD), U1.AL17 (VDD), U1.AL25 (VDD), U1.AL3 (VDD), U1.AL7 (VDD), U1.B28 (VDD), U1.B8 (VDD), U1.C1 (VDD), U1.E31 (VDD), U1.L1 (VDD), U1.N31 (VDD), U1.U1 (VDD)
- net at U1.A13 (DECA): now also C69.1
- net at U1.A15 (DECD): now also C64.1, L2.2
- net at U1.A21 (DCC): now also L4.1
- net at U1.A23 (DECN): now also C70.1
- net at U1.A27 (DECR): now also U1.G31 (DECRF), C67.1, C68.1, L4.2
- net at U1.A5 (VBUS): now also C71.1, R1.2
- net at U1.B10 (DCCD): now also L2.1
- net at U1.B6 (DECUSB): now also C72.1
- net at U1.L31 (ANT): now also C65.1, L3.1
- new net: AE1.2 (PCB_Trace), C66.1, L3.2
- no-connect marks 7 -> 8
Other:
- note removed: "External crystal C"
- note removed: "External crystal L"
- moved on the sheet: C15, C31, C32, C35, C37, C39, C59, C6, C60, C61, C62, C63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

Commit message: started to implement npm1300
Parts:
- removed R25, R26: 5.1k, Resistor_SMD:R_0402_1005Metric, symbol Device:R
- added BT1: Battery_Cell, S2B-PH-SM4-TB_LF__SN_:JST_S2B-PH-SM4-TB_LF__SN_, symbol Device:Battery_Cell
- added C23: 10uF, Capacitor_SMD:C_0402_1005Metric, symbol Device:C
- added C24: 4.7uF, Capacitor_SMD:C_0402_1005Metric, symbol Device:C
- added D13: PRTR5V0U2X, Package_TO_SOT_SMD:SOT-143, symbol Power_Protection:PRTR5V0U2X
- added L5, L6, L7: 10uH, symbol Device:L
- added SW7: SW_Push, Button_Switch_SMD:SW_Push_SPST_NO_Alps_SKRK, symbol Switch:SW_Push
- added U2: nPM1300-QEXX, Package_DFN_QFN:QFN-32-1EP_5x5mm_P0.5mm_EP3.6x3.6mm_ThermalVias, symbol PCM_nordic-lib-kicad-npm:nPM1300-QEXX
- C40: value 10uF -> 1uF
- C7: value 100nF -> 10uF; MPN CL05B104KO5NNNC -> CL05A106MQ5NUNC
- R1: value 2.2R -> 300k
Connections:
- net +3V3: now also C35.1, C37.1, C39.1, C59.1, C60.1, C61.1, C62.1, C63.1, U1.A19 (VDD), U1.AC1 (VDD), U1.AG1 (VDD), U1.AJ31 (VDD), U1.AL11 (VDD), U1.AL17 (VDD), U1.AL25 (VDD), U1.AL3 (VDD), U1.AL7 (VDD), U1.B28 (VDD), U1.B8 (VDD), U1.C1 (VDD), U1.E1 (VDDH), U1.E31 (VDD), U1.L1 (VDD), U1.N31 (VDD), U1.U1 (VDD), C23.1, L5.2, L7.1, U2.32 (VOUT2)
- net CC1: now also J3.A5 (CC1), U2.23 (CC1); no longer J3.B5 (CC2)
- net CC2: now also J3.B5 (CC2), U2.24 (CC2); no longer J3.A5 (CC1)
- net GND: now also R1.2, U1.EP (VSS), BT1.2 (-), C23.2, C24.1, SW7.1, U2.2 (PVSS1), U2.33 (AVSS), U2.6 (PVSS2)
- net I2C_SCL: now also U2.14 (SCL)
- net I2C_SDA: now also U2.13 (SDA)
- net at C7.1: now also L6.1, U2.1 (VOUT1)
- net VBUSOUT: now reaches C71.1, U1.A5 (VBUS)
- net VBUSOUT: now also U2.22 (VBUSOUT); no longer R1.2
- net at U1.J1 (DCCH): now also L5.1
- net at R1.1: now also U2.16 (VSET2)
- net +5V renamed VBUSIN
- net VBUSIN: now also U2.21 (VBUS)
- new net: SW7.2, U2.15 (SHPHLD)
- new net: L6.2, U2.3 (SW1)
- new net: L7.2, U2.5 (SW2)
- new net +BATT: BT1.1 (+), C24.2, U2.19 (VBAT)
- no-connect marks 8 -> 12
Other:
- note added: "BATTERY"
- note added: "I2C PULL-UPs"
- note removed: "ESP32"
- note removed: "I/O EXPANDER"
- note removed: "I2C_1 PULL-UPs"
- note removed: "this pull-up is larger, becouse i dont want to harm to fall times of the i2s clock"
- moved on the sheet: C11, C12, C13, C14, C17, C18, C19, C20, C21, C22, C30, C40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
