File: meko-pcb/power.kicad_sch (KiCad schematic)
At the start: 39 parts, among them IC3 LP5912-3.3DRVR, IC5 BQ27427YZFR, U10 LP5907SNX-1.8/NOPB, U2 BQ24075RGT, U3 LP5907SNX-3.3/NOPB, U4 LP5907SNX-3.3/NOPB, U6 LP5907SNX-3.3/NOPB, U7 LP5907SNX-1.8/NOPB

Commit message: component selection
Parts:
- IC3: Manufacturer_Part_Number LP5912-3.3DRVR -> (none); Mfr. No. (none) -> LP5912-3.3DRVR
- IC5: Manufacturer_Part_Number BQ27427YZFR -> (none); Mfr. No. (none) -> BQ27427YZFR
- R16, R18, R31: Mfr. No. (none) -> CRCW040210K0FKED
- R17: Mfr. No. (none) -> RC0402FR-0747KL
- R19, R32: Mfr. No. (none) -> RC0402FR-071K5L
- R20: value 1.7k -> 1.8k; Mfr. No. (none) -> RC0402FR-071K8L
- TP10, TP13, TP16, TP17, TP18: now left out of the parts list
- U10, U7: Mfr. No. (none) -> LP5907SNX-1.8/NOPB
- U2: Mfr. No. (none) -> BQ24075RGTR
- U3, U4, U6: Mfr. No. (none) -> LP5907SNX-3.3/NOPB
Changed lines of the file:
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@@
 			)
 		)
+		(property "Mfr. No." "RC0402FR-071K5L"
+			(at 99.06 45.72 90)
+			(effects
+				(font
+					(size 1.27 1.27)
+				)
+				(hide yes)
+			)
+		)
 		(pin "2"
 		)
@@
 			)
 		)
+		(property "Mfr. No." "LP5907SNX-3.3/NOPB"
+			(at 55.88 100.33 0)
+			(effects
+				(font
+					(size 1.27 1.27)
+				)
+				(hide yes)
+			)
+		)
 		(pin "3"
 		)
@@
 			)
 		)
-		(property "Manufacturer_Part_Number" "LP5912-3.3DRVR"
-			(at 241.3 723.19 0)
-			(effects
-				(font
-					(size 1.27 1.27)
-				)
-				(justify left top)
-				(hide yes)
-			)
-		)
 		(property "Mouser Part Number" "595-LP5912-3.3DRVR"
 			(at 241.3 823.19 0)
@@
 			)
 		)
+		(property "Mfr. No." "LP5912-3.3DRVR"
+			(at 262.89 128.27 0)
+			(effects
+				(font
+					(size 1.27 1.27)
+				)
+				(hide yes)
+			)
+		)
 		(pin "3"
 		)
@@
 			)
 		)
+		(property "Mfr. No." "LP5907SNX-1.8/NOPB"
+			(at 198.12 142.24 0)
+			(effects
+				(font
+					(size 1.27 1.27)
+				)
+				(hide yes)
+			)
+		)
 		(pin "2"
 		)
@@
 			)
 		)
+		(property "Mfr. No." "BQ24075RGTR"
+			(at 80.01 35.56 0)
+			(effects
+				(font
+					(size 1.27 1.27)
+				)
+				(hide yes)
+			)
+		)
 		(pin "10"
 		)
@@
 		(unit 1)
 		(exclude_from_sim no)
-		(in_bom yes)
+		(in_bom no)
 		(on_board yes)
 		(dnp no)
@@
 		(unit 1)
 		(exclude_from_sim no)
-		(in_bom yes)
+		(in_bom no)
 		(on_board yes)
 		(dnp no)
@@
 			)
 		)
+		(property "Mfr. No." "RC0402FR-071K5L"
+			(at 54.61 50.8 0)
+			(effects
+				(font
+					(size 1.27 1.27)
+				)
+				(hide yes)
+			)
+		)
 		(pin "2"
 		)
@@
 			)
 		)
+		(property "Mfr. No." "RC0402FR-0747KL"
+			(at 38.1 50.8 0)
+			(effects
+				(font
+					(size 1.27 1.27)
+				)
+				(hide yes)
+			)
+		)
 		(pin "2"
 		)
@@
 		(unit 1)
 		(exclude_from_sim no)
-		(in_bom yes)
+		(in_bom no)
 		(on_board yes)
 		(dnp no)
@@
 			)
 		)
+		(property "Mfr. No." "LP5907SNX-3.3/NOPB"
+			(at 55.88 142.24 0)
+			(effects
+				(font
+					(size 1.27 1.27)
+				)
+				(hide yes)
+			)
+		)
 		(pin "3"
 		)
@@
 			)
 		)
-		(property "Value" "1.7k"
+		(property "Value" "1.8k"
 			(at 57.658 52.324 0)
 			(effects
@@
 			)
 		)
+		(property "Mfr. No." "RC0402FR-071K8L"
+			(at 63.5 50.8 0)
+			(effects
+				(font
+					(size 1.27 1.27)
+				)
+				(hide yes)
+			)
+		)
 		(pin "2"
 		)
@@
 		(unit 1)
 		(exclude_from_sim no)
-		(in_bom yes)
+		(in_bom no)
 		(on_board yes)
 		(dnp no)
@@
 			)
 		)
+		(property "Mfr. No." "LP5907SNX-1.8/NOPB"
+			(at 134.62 142.24 0)
+			(effects
+				(font
+					(size 1.27 1.27)
+				)
+				(hide yes)
+			)
+		)
 		(pin "2"
 		)
@@
 			)
 		)
-		(property "Manufacturer_Part_Number" "BQ27427YZFR"
-			(at 200.66 646.99 0)
-			(effects
-				(font
-					(size 1.27 1.27)
-				)
-				(justify left top)
-				(hide yes)
-			)
-		)
 		(property "Mouser Part Number" "595-BQ27427YZFR"
 			(at 200.66 746.99 0)
@@
 			)
 		)
+		(property "Mfr. No." "BQ27427YZFR"
+			(at 173.99 52.07 0)
+			(effects
+				(font
+					(size 1.27 1.27)
+				)
+				(hide yes)
+			)
+		)
 		(pin "C1"
 		)
@@
 			)
 		)
+		(property "Mfr. No." "CRCW040210K0FKED"
+			(at 45.72 50.8 0)
+			(effects
+				(font
+					(size 1.27 1.27)
+				)
+				(hide yes)
+			)
+		)
 		(pin "1"
 		)
@@
 			)
 		)
+		(property "Mfr. No." "LP5907SNX-3.3/NOPB"
+			(at 134.62 100.33 0)
+			(effects
+				(font
+					(size 1.27 1.27)
+				)
+				(hide yes)
+			)
+		)
 		(pin "3"
 		)
@@
 			)
 		)
+		(property "Mfr. No." "CRCW040210K0FKED"
+			(at 114.3 44.45 0)
+			(effects
+				(font
+					(size 1.27 1.27)
+				)
+				(hide yes)
+			)
+		)
 		(pin "2"
 		)
@@
 			)
 		)
+		(property "Mfr. No." "CRCW040210K0FKED"
+			(at 168.91 64.77 0)
+			(effects
+				(font
+					(size 1.27 1.27)
+				)
+				(hide yes)
+			)
+		)
 		(pin "2"
 		)
@@
 		(unit 1)
 		(exclude_from_sim no)
-		(in_bom yes)
+		(in_bom no)
 		(on_board yes)
 		(dnp no)

Commit message: picked MPNs
Parts:
- BT1: MPN (none) -> S2B-PH-SM4-TB
- C23, C24, C25, C26, C33: MPN (none) -> CL05A475KP5NRNC
- C27, C28, C29, C34, C36, C38, C57, C58: MPN (none) -> CL05A105KO5NNNC
- D14: MPN (none) -> 150060AS75003
- IC3: MPN (none) -> LP5912-3.3DRVR; Mfr. No. LP5912-3.3DRVR -> (none); Mouser Part Number 595-LP5912-3.3DRVR -> (none); Mouser Price/Stock https://www.mouser.co.uk/ProductDetail/Texas-Instruments/LP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 -> (none)
- IC5: MPN (none) -> BQ27427YZFR; Mfr. No. BQ27427YZFR -> (none); Mouser Part Number 595-BQ27427YZFR -> (none); Mouser Price/Stock https://www.mouser.co.uk/ProductDetail/Texas-Instruments/BQ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 -> (none)
- R16, R18, R31: MPN (none) -> CRCW040210K0FKED; Mfr. No. CRCW040210K0FKED -> (none)
- R17: MPN (none) -> RC0402FR-0747KL; Mfr. No. RC0402FR-0747KL -> (none)
- R19, R32: MPN (none) -> RC0402FR-071K5L; Mfr. No. RC0402FR-071K5L -> (none)
- R20: MPN (none) -> RC0402FR-071K8L; Mfr. No. RC0402FR-071K8L -> (none)
- U10, U7: MPN (none) -> LP5907SNX-1.8/NOPB; Mfr. No. LP5907SNX-1.8/NOPB -> (none)
- U2: MPN (none) -> BQ24075RGTR; Mfr. No. BQ24075RGTR -> (none)
- U3, U4, U6: MPN (none) -> LP5907SNX-3.3/NOPB; Mfr. No. LP5907SNX-3.3/NOPB -> (none)
Changed lines of the file:
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@@
 			)
 		)
+		(property "MPN" "CL05A475KP5NRNC"
+			(at 267.97 132.08 0)
+			(effects
+				(font
+					(size 1.27 1.27)
+				)
+				(hide yes)
+			)
+		)
 		(pin "2"
 		)
@@
 			)
 		)
+		(property "MPN" "CL05A105KO5NNNC"
+			(at 109.22 93.98 0)
+			(effects
+				(font
+					(size 1.27 1.27)
+				)
+				(hide yes)
+			)
+		)
 		(pin "2"
 		)
@@
 			)
 		)
-		(property "Mfr. No." "RC0402FR-071K5L"
+		(property "MPN" "RC0402FR-071K5L"
 			(at 99.06 45.72 90)
 			(effects
@@
 			)
 		)
+		(property "MPN" "CL05A105KO5NNNC"
+			(at 173.99 135.89 0)
+			(effects
+				(font
+					(size 1.27 1.27)
+				)
+				(hide yes)
+			)
+		)
 		(pin "2"
 		)
@@
 			)
 		)
-		(property "Mfr. No." "LP5907SNX-3.3/NOPB"
+		(property "MPN" "LP5907SNX-3.3/NOPB"
 			(at 55.88 100.33 0)
 			(effects
@@
 			)
 		)
-		(property "Mouser Part Number" "595-LP5912-3.3DRVR"
-			(at 241.3 823.19 0)
-			(effects
-				(font
-					(size 1.27 1.27)
-				)
-				(justify left top)
-				(hide yes)
-			)
-		)
-		(property "Mouser Price/Stock" "https://www.mouser.co.uk/ProductDetail/Texas-Instruments/LP5912-3.3DRVR?qs=n%252BTO0c4TDSY0RMrHlK%2FGvQ%3D%3D"
-			(at 241.3 923.19 0)
-			(effects
-				(font
-					(size 1.27 1.27)
-				)
-				(justify left top)
-				(hide yes)
-			)
-		)
 		(property "Arrow Part Number" "LP5912-3.3DRVR"
 			(at 241.3 1023.19 0)
@@
 			)
 		)
-		(property "Mfr. No." "LP5912-3.3DRVR"
+		(property "MPN" "LP5912-3.3DRVR"
 			(at 262.89 128.27 0)
 			(effects
@@
 			)
 		)
-		(property "Mfr. No." "LP5907SNX-1.8/NOPB"
+		(property "MPN" "LP5907SNX-1.8/NOPB"
 			(at 198.12 142.24 0)
 			(effects
@@
 			)
 		)
-		(property "Mfr. No." "BQ24075RGTR"
+		(property "MPN" "BQ24075RGTR"
 			(at 80.01 35.56 0)
 			(effects
@@
 			)
 		)
+		(property "MPN" "CL05A105KO5NNNC"
+			(at 226.06 60.96 0)
+			(effects
+				(font
+					(size 1.27 1.27)
+				)
+				(hide yes)
+			)
+		)
 		(pin "2"
 		)
@@
 			)
 		)
+		(property "MPN" "S2B-PH-SM4-TB"
+			(at 270.51 59.69 90)
+			(effects
+				(font
+					(size 1.27 1.27)
+				)
+				(hide yes)
+			)
+		)
 		(pin "1"
 		)
@@
 			)
 		)
+		(property "MPN" "CL05A105KO5NNNC"
+			(at 236.22 60.96 0)
+			(effects
+				(font
+					(size 1.27 1.27)
+				)
+				(hide yes)
+			)
+		)
 		(pin "2"
 		)
@@
 			)
 		)
+		(property "MPN" "CL05A105KO5NNNC"
+			(at 29.21 93.98 0)
+			(effects
+				(font
+					(size 1.27 1.27)
+				)
+				(hide yes)
+			)
+		)
 		(pin "2"
 		)
@@
 			)
 		)
+		(property "MPN" "CL05A475KP5NRNC"
+			(at 123.19 43.18 0)
+			(effects
+				(font
+					(size 1.27 1.27)
+				)
+				(hide yes)
+			)
+		)
 		(pin "1"
 		)
@@
 			)
 		)
-		(property "Mfr. No." "RC0402FR-071K5L"
+		(property "MPN" "RC0402FR-071K5L"
 			(at 54.61 50.8 0)
 			(effects
@@
 			)
 		)
-		(property "Mfr. No." "RC0402FR-0747KL"
+		(property "MPN" "RC0402FR-0747KL"
 			(at 38.1 50.8 0)
 			(effects
@@
 			)
 		)
+		(property "MPN" "CL05A105KO5NNNC"
+			(at 29.21 135.89 0)
+			(effects
+				(font
+					(size 1.27 1.27)
+				)
+				(hide yes)
+			)
+		)
 		(pin "2"
 		)
@@
 			)
 		)
-		(property "Mfr. No." "LP5907SNX-3.3/NOPB"
+		(property "MPN" "LP5907SNX-3.3/NOPB"
 			(at 55.88 142.24 0)
 			(effects
@@
 			)
 		)
-		(property "Mfr. No." "RC0402FR-071K8L"
+		(property "MPN" "RC0402FR-071K8L"
 			(at 63.5 50.8 0)
 			(effects
@@
 			)
 		)
-		(property "Mfr. No." "LP5907SNX-1.8/NOPB"
+		(property "MPN" "LP5907SNX-1.8/NOPB"
 			(at 134.62 142.24 0)
 			(effects
@@
 			)
 		)
-		(property "Mouser Part Number" "595-BQ27427YZFR"
-			(at 200.66 746.99 0)
-			(effects
-				(font
-					(size 1.27 1.27)
-				)
-				(justify left top)
-				(hide yes)
-			)
-		)
-		(property "Mouser Price/Stock" "https://www.mouser.co.uk/ProductDetail/Texas-Instruments/BQ27427YZFR?qs=rQFj71Wb1eU5v%2FHj43hVJQ%3D%3D"
-			(at 200.66 846.99 0)
-			(effects
-				(font
-					(size 1.27 1.27)
-				)
-				(justify left top)
-				(hide yes)
-			)
-		)
 		(property "Arrow Part Number" "BQ27427YZFR"
 			(at 200.66 946.99 0)
@@
 			)
 		)
-		(property "Mfr. No." "BQ27427YZFR"
+		(property "MPN" "BQ27427YZFR"
 			(at 173.99 52.07 0)
 			(effects
@@
 			)
 		)
-		(property "Mfr. No." "CRCW040210K0FKED"
+		(property "MPN" "CRCW040210K0FKED"
 			(at 45.72 50.8 0)
 			(effects
@@
 			)
 		)
+		(property "MPN" "CL05A475KP5NRNC"
+			(at 26.67 40.64 0)
+			(effects
+				(font
+					(size 1.27 1.27)
+				)
+				(hide yes)
+			)
+		)
 		(pin "1"
 		)
@@
 			)
 		)
+		(property "MPN" "150060AS75003"
+			(at 105.41 50.8 90)
+			(effects
+				(font
+					(size 1.27 1.27)
+				)
+				(hide yes)
+			)
+		)
 		(pin "2"
 		)
@@
 			)
 		)
-		(property "Mfr. No." "LP5907SNX-3.3/NOPB"
+		(property "MPN" "LP5907SNX-3.3/NOPB"
 			(at 134.62 100.33 0)
 			(effects
@@
 			)
 		)
+		(property "MPN" "CL05A475KP5NRNC"
+			(at 134.62 43.18 0)
+			(effects
+				(font
+					(size 1.27 1.27)
+				)
+				(hide yes)
+			)
+		)
 		(pin "1"
 		)
@@
 			)
 		)
+		(property "MPN" "CL05A475KP5NRNC"
+			(at 264.16 63.5 0)
+			(effects
+				(font
+					(size 1.27 1.27)
+				)
+				(hide yes)
+			)
+		)
 		(pin "1"
 		)
@@
 			)
 		)
-		(property "Mfr. No." "CRCW040210K0FKED"
+		(property "MPN" "CRCW040210K0FKED"
 			(at 114.3 44.45 0)
 			(effects
@@
 			)
 		)
+		(property "MPN" "CL05A105KO5NNNC"
+			(at 110.49 135.89 0)
+			(effects
+				(font
+					(size 1.27 1.27)
+				)
+				(hide yes)
+			)
+		)
 		(pin "2"
 		)
@@
 			)
 		)
+		(property "MPN" "CL05A105KO5NNNC"
+			(at 78.74 93.98 0)
+			(effects
+				(font
+					(size 1.27 1.27)
+				)
+				(hide yes)
+			)
+		)
 		(pin "2"
 		)
@@
 			)
 		)
-		(property "Mfr. No." "CRCW040210K0FKED"
+		(property "MPN" "CRCW040210K0FKED"
 			(at 168.91 64.77 0)
 			(effects

Commit message: readme updates, removed unused fileds form kicad
Parts:
- C23, C24, C25, C26: LCSC C307423 -> (none)
- IC3: Arrow Part Number LP5912-3.3DRVR -> (none); Arrow Price/Stock https://www.arrow.com/en/products/lp5912-3.3drvr/texas-inst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 -> (none); Height 0.8 -> (none); Manufacturer_Name Texas Instruments -> (none)
- IC5: Arrow Part Number BQ27427YZFR -> (none); Arrow Price/Stock https://www.arrow.com/en/products/bq27427yzfr/texas-instrum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 -> (none); Height 0.625 -> (none); Manufacturer_Name Texas Instruments -> (none)
- R16, R31, R32: LCSC C25744 -> (none)
- R17: LCSC C93943 -> (none)
- R19: LCSC C25867 -> (none)
- R20: LCSC C131467 -> (none)
Changed lines of the file:
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@@
 			)
 		)
-		(property "LCSC" "C25744"
-			(at 99.06 45.72 0)
-			(effects
-				(font
-					(size 1.27 1.27)
-				)
-				(hide yes)
-			)
-		)
 		(property "MPN" "RC0402FR-071K5L"
 			(at 99.06 45.72 90)
@@
 			)
 		)
-		(property "Height" "0.8"
-			(at 241.3 523.19 0)
-			(effects
-				(font
-					(size 1.27 1.27)
-				)
-				(justify left top)
-				(hide yes)
-			)
-		)
-		(property "Manufacturer_Name" "Texas Instruments"
-			(at 241.3 623.19 0)
-			(effects
-				(font
-					(size 1.27 1.27)
-				)
-				(justify left top)
-				(hide yes)
-			)
-		)
-		(property "Arrow Part Number" "LP5912-3.3DRVR"
-			(at 241.3 1023.19 0)
-			(effects
-				(font
-					(size 1.27 1.27)
-				)
-				(justify left top)
-				(hide yes)
-			)
-		)
-		(property "Arrow Price/Stock" "https://www.arrow.com/en/products/lp5912-3.3drvr/texas-instruments?utm_currency=USD&region=nac"
-			(at 241.3 1123.19 0)
-			(effects
-				(font
-					(size 1.27 1.27)
-				)
-				(justify left top)
-				(hide yes)
-			)
-		)
 		(property "MPN" "LP5912-3.3DRVR"
 			(at 262.89 128.27 0)
@@
 			)
 		)
-		(property "LCSC" "C307423"
-			(at 123.19 43.18 0)
-			(effects
-				(font
-					(size 1.27 1.27)
-				)
-				(hide yes)
-			)
-		)
 		(property "MPN" "CL05A475KP5NRNC"
 			(at 123.19 43.18 0)
@@
 			)
 		)
-		(property "LCSC" "C25867"
-			(at 54.61 50.8 0)
-			(effects
-				(font
-					(size 1.27 1.27)
-				)
-				(hide yes)
-			)
-		)
 		(property "MPN" "RC0402FR-071K5L"
 			(at 54.61 50.8 0)
@@
 			)
 		)
-		(property "LCSC" " C93943"
-			(at 38.1 50.8 0)
-			(effects
-				(font
-					(size 1.27 1.27)
-				)
-				(hide yes)
-			)
-		)
 		(property "MPN" "RC0402FR-0747KL"
 			(at 38.1 50.8 0)
@@
 			)
 		)
-		(property "LCSC" "C131467"
-			(at 63.5 50.8 0)
-			(effects
-				(font
-					(size 1.27 1.27)
-				)
-				(hide yes)
-			)
-		)
 		(property "MPN" "RC0402FR-071K8L"
 			(at 63.5 50.8 0)
@@
 			)
 		)
-		(property "Height" "0.625"
-			(at 200.66 446.99 0)
-			(effects
-				(font
-					(size 1.27 1.27)
-				)
-				(justify left top)
-				(hide yes)
-			)
-		)
-		(property "Manufacturer_Name" "Texas Instruments"
-			(at 200.66 546.99 0)
-			(effects
-				(font
-					(size 1.27 1.27)
-				)
-				(justify left top)
-				(hide yes)
-			)
-		)
-		(property "Arrow Part Number" "BQ27427YZFR"
-			(at 200.66 946.99 0)
-			(effects
-				(font
-					(size 1.27 1.27)
-				)
-				(justify left top)
-				(hide yes)
-			)
-		)
-		(property "Arrow Price/Stock" "https://www.arrow.com/en/products/bq27427yzfr/texas-instruments?utm_currency=USD&region=nac"
-			(at 200.66 1046.99 0)
-			(effects
-				(font
-					(size 1.27 1.27)
-				)
-				(justify left top)
-				(hide yes)
-			)
-		)
 		(property "MPN" "BQ27427YZFR"
 			(at 173.99 52.07 0)
@@
 			)
 		)
-		(property "LCSC" "C307423"
-			(at 26.67 40.64 0)
-			(effects
-				(font
-					(size 1.27 1.27)
-				)
-				(hide yes)
-			)
-		)
 		(property "MPN" "CL05A475KP5NRNC"
 			(at 26.67 40.64 0)
@@
 			)
 		)
-		(property "LCSC" "C307423"
-			(at 134.62 43.18 0)
-			(effects
-				(font
-					(size 1.27 1.27)
-				)
-				(hide yes)
-			)
-		)
 		(property "MPN" "CL05A475KP5NRNC"
 			(at 134.62 43.18 0)
@@
 			)
 		)
-		(property "LCSC" "C307423"
-			(at 264.16 63.5 0)
-			(effects
-				(font
-					(size 1.27 1.27)
-				)
-				(hide yes)
-			)
-		)
 		(property "MPN" "CL05A475KP5NRNC"
 			(at 264.16 63.5 0)
@@
 			)
 		)
-		(property "LCSC" "C25744"
-			(at 114.3 44.45 0)
-			(effects
-				(font
-					(size 1.27 1.27)
-				)
-				(hide yes)
-			)
-		)
 		(property "MPN" "CRCW040210K0FKED"
 			(at 114.3 44.45 0)
@@
 			(at 168.91 64.77 0)
 			(effects
-				(font
-					(size 1.27 1.27)
-				)
-				(hide yes)
-			)
-		)
-		(property "LCSC" "C25744"
-			(at 168.91 64.77 0)
-			(effects

Commit message: continued work om nrf53
Parts:
- removed C25, C26: 4.7uF, Capacitor_SMD:C_0402_1005Metric, symbol Device:C
- removed C57, C58: 1uF, Capacitor_SMD:C_0402_1005Metric, symbol Device:C
- removed IC5: BQ27427YZFR, BQ27427YZFR:BGA9C50P3X3_158X162X62, symbol BQ27427YZFR:BQ27427YZFR
- removed R16, R18, R31: 10k, Resistor_SMD:R_0402_1005Metric, symbol Device:R
- removed R17: 47k, Resistor_SMD:R_0402_1005Metric, symbol Device:R
- removed R19, R32: 1.5k, Resistor_SMD:R_0402_1005Metric, symbol Device:R
- removed R20: 1.8k, Resistor_SMD:R_0402_1005Metric, symbol Device:R
- removed TP10: TestPoint, TestPoint:TestPoint_Pad_D1.0mm, symbol Connector:TestPoint
- removed U2: BQ24075RGT, Package_DFN_QFN:VQFN-16-1EP_3x3mm_P0.5mm_EP1.6x1.6mm, symbol Battery_Management:BQ24075RGT
- added R2, R3: 5k, symbol Device:R
- added U2: TP4056-42-ESOP8, Package_SO:SOIC-8-1EP_3.9x4.9mm_P1.27mm_EP2.41x3.3mm_ThermalVias, symbol Battery_Management:TP4056-42-ESOP8
- C23: value 4.7uF -> 10uF; footprint Capacitor_SMD:C_0402_1005Metric -> (none); MPN CL05A475KP5NRNC -> (none)
Connections:
- net +5V: no longer C23.2
- net +BATT: now also C23.1, D14.2 (A), U2.4 (V_{CC}), U2.8 (CE)
- net GND: now also C23.2, R2.2, U2.1 (TEMP), U2.3 (GND), U2.9 (EPAD); no longer C23.1, D14.1 (K)
- new net: R2.1, U2.2 (PROG)
- new net: D14.1 (K), U2.7 (~{CHRG})
- no-connect marks 2 -> 3
Other:
- note removed: "FUEAL GAUGE"
- note removed: "RISET = 890A*OHM / ICHG ICHG <=1.5A ILIM does no matter, becouse en1 and en2 set it to usb500mA"
- note removed: "TODO: change values if needed"
- note removed: "addr(dec.):85"
- moved on the sheet: D14
