File: meko-pcb/_autosave-meko-pcb.kicad_sch (KiCad schematic)
At the start: 209 parts, among them IC2 TPS7A2033PDBVR, IC4 TAD5212IRGER, IC5 AS5600-ASOM, J1 USB_C_Receptacle_USB2.0_16P, J2 Conn_ARM_JTAG_SWD_10, J3 GDEY0154D67, J5 503398-1892, Q1 SS8050, Q2 Si1308EDL, SW1 SW_Push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

Commit message: places all the testpoints
Parts:
- removed TP32: DISPL_SCL, TestPoint:TestPoint_Pad_D1.0mm, symbol Connector:TestPoint
- L7: footprint Inductor_SMD:L_TDK_MLZ2012_h1.25mm -> Inductor_SMD:L_0805_2012Metric
Connections:
- net DISPL_SCL: now also TP29.1; no longer TP27.1
- net DISPL_SDA: now also TP27.1; no longer TP29.1
- no-connect marks 12 -> 13
Other:
- moved on the sheet: TP27, TP29
Changed lines of the file:
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@@
 	)
 	(no_connect
+		(at 195.58 153.67)
+	)
+	(no_connect
 		(at 361.95 101.6)
 	)
@@
 	(wire
 		(pts
-			(xy 176.53 153.67) (xy 193.04 153.67)
+			(xy 176.53 153.67) (xy 195.58 153.67)
 		)
 		(stroke
@@
 	(symbol
 		(lib_id "Connector:TestPoint")
-		(at 193.04 140.97 270)
+		(at 193.04 146.05 270)
 		(mirror x)
 		(unit 1)
@@
 		(dnp no)
 		(property "Reference" "TP27"
-			(at 197.866 140.97 90)
+			(at 197.866 146.05 90)
 			(effects
 				(font
@@
 		)
 		(property "Value" "DISPL_SDA"
-			(at 195.0721 138.43 0)
+			(at 195.0721 143.51 0)
 			(effects
 				(font
@@
 		)
 		(property "Footprint" "TestPoint:TestPoint_Pad_D1.0mm"
-			(at 193.04 135.89 0)
+			(at 193.04 140.97 0)
 			(effects
 				(font
@@
 		)
 		(property "Datasheet" "~"
-			(at 193.04 135.89 0)
+			(at 193.04 140.97 0)
 			(effects
 				(font
@@
 		)
 		(property "Description" "test point"
-			(at 193.04 140.97 0)
+			(at 193.04 146.05 0)
 			(effects
 				(font
@@
 	(symbol
 		(lib_id "Connector:TestPoint")
-		(at 193.04 146.05 270)
+		(at 193.04 140.97 270)
 		(mirror x)
 		(unit 1)
@@
 		(dnp no)
 		(property "Reference" "TP29"
-			(at 197.866 146.05 90)
+			(at 197.866 140.97 90)
 			(effects
 				(font
@@
 		)
 		(property "Value" "DISPL_SCL"
-			(at 195.0721 143.51 0)
+			(at 195.0721 138.43 0)
 			(effects
 				(font
@@
 		)
 		(property "Footprint" "TestPoint:TestPoint_Pad_D1.0mm"
-			(at 193.04 140.97 0)
+			(at 193.04 135.89 0)
 			(effects
 				(font
@@
 		)
 		(property "Datasheet" "~"
-			(at 193.04 140.97 0)
+			(at 193.04 135.89 0)
 			(effects
 				(font
@@
 		)
 		(property "Description" "test point"
-			(at 193.04 146.05 0)
+			(at 193.04 140.97 0)
 			(effects
 				(font
@@
 	)
 	(symbol
-		(lib_id "Connector:TestPoint")
-		(at 193.04 153.67 270)
-		(mirror x)
-		(unit 1)
-		(exclude_from_sim no)
-		(in_bom no)
-		(on_board yes)
-		(dnp no)
-		(property "Reference" "TP32"
-			(at 197.866 153.67 90)
-			(effects
-				(font
-					(size 1.27 1.27)
-				)
-				(justify left)
-			)
-		)
-		(property "Value" "DISPL_SCL"
-			(at 195.0721 151.13 0)
-			(effects
-				(font
-					(size 1.27 1.27)
-				)
-				(justify left)
-				(hide yes)
-			)
-		)
-		(property "Footprint" "TestPoint:TestPoint_Pad_D1.0mm"
-			(at 193.04 148.59 0)
-			(effects
-				(font
-					(size 1.27 1.27)
-				)
-				(hide yes)
-			)
-		)
-		(property "Datasheet" "~"
-			(at 193.04 148.59 0)
-			(effects
-				(font
-					(size 1.27 1.27)
-				)
-				(hide yes)
-			)
-		)
-		(property "Description" "test point"
-			(at 193.04 153.67 0)
-			(effects
-				(font
-					(size 1.27 1.27)
-				)
-				(hide yes)
-			)
-		)
-		(pin "1"
-		)
-		(instances
-			(project "meko-pcb"
-				(path "/bdd43acd-23c1-472b-909a-8e24eb60d56d"
-					(reference "TP32")
-					(unit 1)
-				)
-			)
-		)
-	)
-	(symbol
 		(lib_id "power:GND")
 		(at 234.95 363.22 0)
@@
 			)
 		)
-		(property "Footprint" "Inductor_SMD:L_TDK_MLZ2012_h1.25mm"
+		(property "Footprint" "Inductor_SMD:L_0805_2012Metric"
 			(at 322.58 290.83 0)
 			(effects
