File: hardware/pcb/usb.kicad_sch (KiCad schematic)
At the start: 0 parts

Commit message: usb power
Parts:
- added D1, D2, D3: ESD441, ESD441DPLR:ESD441DPLR, symbol Device:D_Small
- added J1: USB_C_Receptacle_USB2.0_14P, PCM_ckl-connector:USB_C_Receptacle_HRO_TYPE-C-31-M-12, symbol Connector:USB_C_Receptacle_USB2.0_14P
- added U5: ECMF02-2AMX6, Package_DFN_QFN:ST_UQFN-6L_1.5x1.7mm_P0.5mm, symbol Power_Protection:ECMF02-2AMX6
Connections:
- new net CC1: D1.1 (K), J1.A5 (CC1)
- new net CC2: D2.1 (K), J1.B5 (CC2)
- new net D+: U5.6 (D+_out)
- new net D-: U5.5 (D-_out)
- new net DIRTY_D+: J1.A6 (D+), J1.B6 (D+), U5.1 (D+_in)
- new net DIRTY_D-: J1.A7 (D-), J1.B7 (D-), U5.2 (D-_in)
- new net GND: D1.2 (A), D2.2 (A), D3.2 (A), J1.A1 (GND), J1.A12 (GND), J1.B1 (GND), J1.B12 (GND), J1.SH (SHIELD), U5.3 (GND)
- new net VBUS: D3.1 (K), J1.A4 (VBUS), J1.A9 (VBUS), J1.B4 (VBUS), J1.B9 (VBUS)

Commit message: finished power
Parts:
- removed J1: USB_C_Receptacle_USB2.0_14P, PCM_ckl-connector:USB_C_Receptacle_HRO_TYPE-C-31-M-12, symbol Connector:USB_C_Receptacle_USB2.0_14P
- added C21: 10u, symbol Device:C_Small
- added J?: USB_C_Receptacle_USB2.0_16P, symbol Connector:USB_C_Receptacle_USB2.0_16P
Connections:
- net CC1: now also J?.A5 (CC1)
- net CC2: now also J?.B5 (CC2)
- net DIRTY_D+: now also J?.A6 (D+), J?.B6 (D+)
- net DIRTY_D-: now also J?.A7 (D-), J?.B7 (D-)
- net GND: now also C21.1, J?.A1 (GND), J?.A12 (GND), J?.B1 (GND), J?.B12 (GND), J?.SH (SHIELD)
- net VBUS: now also C21.2, J?.A4 (VBUS), J?.A9 (VBUS), J?.B4 (VBUS), J?.B9 (VBUS)
- no-connect marks 0 -> 2
Other:
- moved on the sheet: D1, D2, D3

Commit message: contiunued working
Parts:
- gave numbers to parts that had none: 1
Changed lines of the file:
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@@
+			)
+		)
+		(property "KLC_S3.3" ""
+			(at 143.51 44.45 90)
+			(hide yes)
+			(show_name no)
+			(do_not_autoplace no)
+			(effects
+				(font
+					(size 1.27 1.27)
+				)
+			)
+		)
+		(property "KLC_S4.1" ""
+			(at 143.51 44.45 90)
+			(hide yes)
+			(show_name no)
+			(do_not_autoplace no)
+			(effects
+				(font
+					(size 1.27 1.27)
+				)
 			)
 		)
@@
 			)
 		)
+		(property "KLC_S3.3" ""
+			(at 121.92 66.04 0)
+			(hide yes)
+			(show_name no)
+			(do_not_autoplace no)
+			(effects
+				(font
+					(size 1.27 1.27)
+				)
+			)
+		)
+		(property "KLC_S4.1" ""
+			(at 121.92 66.04 0)
+			(hide yes)
+			(show_name no)
+			(do_not_autoplace no)
+			(effects
+				(font
+					(size 1.27 1.27)
+				)
+			)
+		)
 		(pin "6"
 		)
@@
 			)
 		)
+		(property "KLC_S3.3" ""
+			(at 106.68 33.02 0)
+			(hide yes)
+			(show_name no)
+			(do_not_autoplace no)
+			(effects
+				(font
+					(size 1.27 1.27)
+				)
+			)
+		)
+		(property "KLC_S4.1" ""
+			(at 106.68 33.02 0)
+			(hide yes)
+			(show_name no)
+			(do_not_autoplace no)
+			(effects
+				(font
+					(size 1.27 1.27)
+				)
+			)
+		)
 		(pin "1"
 		)
@@
 		(dnp no)
 		(fields_autoplaced yes)
-		(property "Reference" "J?"
+		(property "Reference" "J3"
 			(at 86.36 40.64 0)
 			(show_name no)
@@
 		)
 		(property "Description" "USB 2.0-only 16P Type-C Receptacle connector"
+			(at 86.36 63.5 0)
+			(hide yes)
+			(show_name no)
+			(do_not_autoplace no)
+			(effects
+				(font
+					(size 1.27 1.27)
+				)
+			)
+		)
+		(property "KLC_S3.3" ""
+			(at 86.36 63.5 0)
+			(hide yes)
+			(show_name no)
+			(do_not_autoplace no)
+			(effects
+				(font
+					(size 1.27 1.27)
+				)
+			)
+		)
+		(property "KLC_S4.1" ""
 			(at 86.36 63.5 0)
 			(hide yes)
@@
 			(project "meko"
 				(path "/da54f10a-146b-4941-a9c7-55c7173bb101/13ed9585-0f16-442f-add9-c716aca8a0ac"
-					(reference "J?")
+					(reference "J3")
 					(unit 1)
 				)
@@
 			)
 		)
+		(property "KLC_S3.3" ""
+			(at 130.81 44.45 90)
+			(hide yes)
+			(show_name no)
+			(do_not_autoplace no)
+			(effects
+				(font
+					(size 1.27 1.27)
+				)
+			)
+		)
+		(property "KLC_S4.1" ""
+			(at 130.81 44.45 90)
+			(hide yes)
+			(show_name no)
+			(do_not_autoplace no)
+			(effects
+				(font
+					(size 1.27 1.27)
+				)
+			)
+		)
 		(pin "2"
 		)
@@
 			(hide yes)
 			(show_name no)
+			(do_not_autoplace no)
+			(effects
+				(font
+					(size 1.27 1.27)
+				)
+			)
+		)
+		(property "KLC_S3.3" ""
+			(at 137.16 44.45 90)
+			(hide yes)
+			(show_name no)
+			(do_not_autoplace no)
+			(effects
+				(font
+					(size 1.27 1.27)
+				)
+			)
+		)
+		(property "KLC_S4.1" ""
+			(at 137.16 44.45 90)
+			(hide yes)
+			(show_name no)

Commit message: bunch of small changes
Other:
- note added: "ESD"
- moved on the sheet: C21, D1, D2, D3

Commit message: bunch of small audio changes
Parts:
- J3: footprint (none) -> PCM_ckl-connector:USB_C_Receptacle_HRO_TYPE-C-31-M-12
Changed lines of the file:
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@@
 			)
 		)
-		(property "Footprint" ""
+		(property "Footprint" "PCM_ckl-connector:USB_C_Receptacle_HRO_TYPE-C-31-M-12"
 			(at 90.17 63.5 0)
 			(hide yes)

Commit message: bunch of small audio changes
Parts:
- C21: value 10u -> 1u
Changed lines of the file:
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@@
 			)
 		)
-		(property "Value" "10u"
+		(property "Value" "1u"
 			(at 125.222 43.942 0)
 			(show_name no)

Commit message: assigning pins
Changed lines of the file:
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@@
 	)
 	(hierarchical_label "{USB}"
-		(shape input)
+		(shape bidirectional)
 		(at 139.7 60.96 0)
 		(effects
@@
 	)
 	(hierarchical_label "{USB_CC}"
-		(shape input)
+		(shape bidirectional)
 		(at 110.49 50.8 0)
 		(effects

Commit message: looking over stuff, added caps
Parts:
- C21: footprint (none) -> Capacitor_SMD:C_0402_1005Metric
Changed lines of the file:
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@@
 			)
 		)
-		(property "Footprint" ""
+		(property "Footprint" "Capacitor_SMD:C_0402_1005Metric"
 			(at 130.81 43.18 0)
 			(hide yes)
