File: hardware/pcb/usb.kicad_sch (KiCad schematic)
At the start: 9 parts, among them J3 USB_C_Receptacle_USB2.0_16P, U6 ECMF02-2AMX6

Commit message: didn't save last time :sob:
Parts:
- renumbered C112 to C113
Changed lines of the file:
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@@
 		(in_pos_files yes)
 		(dnp no)
-		(property "Reference" "#PWR098"
+		(property "Reference" "#PWR099"
 			(at 36.83 93.98 0)
 			(hide yes)
@@
 			(project "meko"
 				(path "/da54f10a-146b-4941-a9c7-55c7173bb101/13ed9585-0f16-442f-add9-c716aca8a0ac"
-					(reference "#PWR098")
+					(reference "#PWR099")
 					(unit 1)
 				)
@@
 		(in_pos_files yes)
 		(dnp no)
-		(property "Reference" "#PWR0100"
+		(property "Reference" "#PWR0101"
 			(at 73.66 81.28 0)
 			(hide yes)
@@
 			(project "meko"
 				(path "/da54f10a-146b-4941-a9c7-55c7173bb101/13ed9585-0f16-442f-add9-c716aca8a0ac"
-					(reference "#PWR0100")
+					(reference "#PWR0101")
 					(unit 1)
 				)
@@
 		(in_pos_files yes)
 		(dnp no)
-		(property "Reference" "#PWR0102"
+		(property "Reference" "#PWR0103"
 			(at 81.28 53.34 0)
 			(hide yes)
@@
 			(project "meko"
 				(path "/da54f10a-146b-4941-a9c7-55c7173bb101/13ed9585-0f16-442f-add9-c716aca8a0ac"
-					(reference "#PWR0102")
+					(reference "#PWR0103")
 					(unit 1)
 				)
@@
 		(in_pos_files yes)
 		(dnp no)
-		(property "Reference" "#PWR0103"
+		(property "Reference" "#PWR0104"
 			(at 92.71 45.72 0)
 			(hide yes)
@@
 			(project "meko"
 				(path "/da54f10a-146b-4941-a9c7-55c7173bb101/13ed9585-0f16-442f-add9-c716aca8a0ac"
-					(reference "#PWR0103")
+					(reference "#PWR0104")
 					(unit 1)
 				)
@@
 		(in_pos_files yes)
 		(dnp no)
-		(property "Reference" "#PWR0104"
+		(property "Reference" "#PWR0105"
 			(at 99.06 55.88 0)
 			(hide yes)
@@
 			(project "meko"
 				(path "/da54f10a-146b-4941-a9c7-55c7173bb101/13ed9585-0f16-442f-add9-c716aca8a0ac"
-					(reference "#PWR0104")
+					(reference "#PWR0105")
 					(unit 1)
 				)
@@
 		(in_pos_files yes)
 		(dnp no)
-		(property "Reference" "#PWR099"
+		(property "Reference" "#PWR0100"
 			(at 57.15 50.8 0)
 			(hide yes)
@@
 			(project "meko"
 				(path "/da54f10a-146b-4941-a9c7-55c7173bb101/13ed9585-0f16-442f-add9-c716aca8a0ac"
-					(reference "#PWR099")
+					(reference "#PWR0100")
 					(unit 1)
 				)
@@
 		(in_pos_files yes)
 		(dnp no)
-		(property "Reference" "C112"
+		(property "Reference" "C113"
 			(at 79.502 42.164 0)
 			(show_name no)
@@
 			(project "meko"
 				(path "/da54f10a-146b-4941-a9c7-55c7173bb101/13ed9585-0f16-442f-add9-c716aca8a0ac"
-					(reference "C112")
+					(reference "C113")
 					(unit 1)
 				)
@@
 		(in_pos_files yes)
 		(dnp no)
-		(property "Reference" "#PWR0101"
+		(property "Reference" "#PWR0102"
 			(at 81.28 43.18 0)
 			(hide yes)
@@
 			(project "meko"
 				(path "/da54f10a-146b-4941-a9c7-55c7173bb101/13ed9585-0f16-442f-add9-c716aca8a0ac"
-					(reference "#PWR0101")
-					(unit 1)
-				)
+					(reference "#PWR0102")
+					(unit 1)
+				)

Commit message: vendored in a bunch of footprints
Parts:
- J3: footprint PCM_ckl-connector:USB_C_Receptacle_HRO_TYPE-C-31-M-12 -> ckl:USB_C_Receptacle_HRO_TYPE-C-31-M-12
Changed lines of the file:
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@@
 			)
 		)
-		(property "Footprint" "PCM_ckl-connector:USB_C_Receptacle_HRO_TYPE-C-31-M-12"
+		(property "Footprint" "ckl:USB_C_Receptacle_HRO_TYPE-C-31-M-12"
 			(at 40.64 63.5 0)
 			(hide yes)

Commit message: small stuff
Parts:
- added C127: 1u, Capacitor_SMD:C_0402_1005Metric, symbol Device:C_Small
Connections:
- net D+: now also U6.5 (D-_out); no longer U6.6 (D+_out)
- net D-: now also U6.6 (D+_out); no longer U6.5 (D-_out)
- net DIRTY_D+: now also U6.2 (D-_in); no longer U6.1 (D+_in)
- net DIRTY_D-: now also U6.1 (D+_in); no longer U6.2 (D-_in)
- net GND: now also C127.1
- net VBUS: now also C127.2
Other:
- moved on the sheet: U6

Commit message: small changes
Parts:
- U6: footprint Package_DFN_QFN:ST_UQFN-6L_1.5x1.7mm_P0.5mm -> ECMF02-2AMX6:ST_UQFN-6L_1.5x1.7mm_P0.5mm; symbol Power_Protection:ECMF02-2AMX6 -> ECMF02-2AMX6:ECMF02-2AMX6
Changed lines of the file:
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@@
-	(wire
-		(pts
-			(xy 68.58 63.5) (xy 68.58 66.04)
-		)
-		(stroke
-			(width 0)
-			(type default)
-		)
-	)
 	(wire
 		(pts
@@
 	(wire
 		(pts
-			(xy 66.04 66.04) (xy 66.04 64.77)
-		)
-		(stroke
-			(width 0)
-			(type default)
-		)
-	)
-	(wire
-		(pts
 			(xy 92.71 48.26) (xy 92.71 49.53)
 		)
@@
 	(wire
 		(pts
-			(xy 53.34 63.5) (xy 68.58 63.5)
+			(xy 53.34 63.5) (xy 73.66 63.5)
 		)
 		(stroke
@@
 	(wire
 		(pts
-			(xy 68.58 66.04) (xy 73.66 66.04)
-		)
-		(stroke
-			(width 0)
-			(type default)
-		)
-	)
-	(wire
-		(pts
 			(xy 72.39 46.99) (xy 81.28 46.99)
 		)
@@
 	(wire
 		(pts
-			(xy 66.04 64.77) (xy 71.12 64.77)
-		)
-		(stroke
-			(width 0)
-			(type default)
-		)
-	)
-	(wire
-		(pts
 			(xy 93.98 63.5) (xy 97.79 63.5)
 		)
@@
 	(wire
 		(pts
-			(xy 71.12 63.5) (xy 73.66 63.5)
-		)
-		(stroke
-			(width 0)
-			(type default)
-		)
-	)
-	(wire
-		(pts
-			(xy 53.34 66.04) (xy 66.04 66.04)
+			(xy 53.34 66.04) (xy 73.66 66.04)
 		)
 		(stroke
@@
 		(pts
 			(xy 125.73 76.2) (xy 125.73 78.74)
-		)
-		(stroke
-			(width 0)
-			(type default)
-		)
-	)
-	(wire
-		(pts
-			(xy 71.12 64.77) (xy 71.12 63.5)
 		)
 		(stroke
@@
 	)
 	(label "DIRTY_D+"
-		(at 54.61 63.5 0)
+		(at 54.61 66.04 0)
 		(effects
 			(font
@@
 	)
 	(label "DIRTY_D-"
-		(at 54.61 66.04 0)
+		(at 54.61 63.5 0)
 		(effects
 			(font
@@
 	)
 	(symbol
-		(lib_id "Power_Protection:ECMF02-2AMX6")
+		(lib_id "ECMF02-2AMX6:ECMF02-2AMX6")
 		(at 83.82 66.04 0)
 		(unit 1)
@@
 			)
 		)
-		(property "Footprint" "Package_DFN_QFN:ST_UQFN-6L_1.5x1.7mm_P0.5mm"
+		(property "Footprint" "ECMF02-2AMX6:ST_UQFN-6L_1.5x1.7mm_P0.5mm"
 			(at 83.82 86.36 0)
 			(hide yes)
@@
 		)
 		(property "Footprint" "ckl:USB_C_Receptacle_HRO_TYPE-C-31-M-12"
-			(at 40.64 63.5 0)
+			(at 33.274 31.496 0)
 			(hide yes)
 			(show_name no)
@@
 		)
 		(property "Datasheet" "https://www.usb.org/sites/default/files/documents/usb_type-c.zip"
-			(at 40.64 63.5 0)
+			(at 34.036 35.814 0)
 			(hide yes)
 			(show_name no)
@@
 		)
 		(property "Description" "USB 2.0-only 16P Type-C Receptacle connector"
-			(at 36.83 63.5 0)
-			(hide yes)
-			(show_name no)
+			(at 30.226 35.814 0)
+			(hide yes)
+			(show_name no)
