File: hardware/pcb/wireless.kicad_sch (KiCad schematic)
At the start: 15 parts, among them IC2 MAYA-W386-00B, Y3 32kHz768

Commit message: mainboard: reannotated schematic
Parts:
- renumbered C42 to C106, C39 to C107, C30 to C108, C31 to C109, R38 to R23, R39 to R24, R29 to R25, R30 to R26, R31 to R27, R32 to R28, R33 to R29, R34 to R30, R35 to R31
Changed lines of the file:
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@@
 		(in_pos_files yes)
 		(dnp no)
-		(property "Reference" "C42"
+		(property "Reference" "C106"
 			(at 146.304 35.56 90)
 			(show_name no)
@@
 			(project "meko"
 				(path "/da54f10a-146b-4941-a9c7-55c7173bb101/cf3a540d-b7d8-4416-baa0-bfc874a83584"
-					(reference "C42")
+					(reference "C106")
 					(unit 1)
 				)
@@
 		(in_pos_files yes)
 		(dnp no)
-		(property "Reference" "C39"
+		(property "Reference" "C107"
 			(at 161.544 35.56 90)
 			(show_name no)
@@
 			(project "meko"
 				(path "/da54f10a-146b-4941-a9c7-55c7173bb101/cf3a540d-b7d8-4416-baa0-bfc874a83584"
-					(reference "C39")
+					(reference "C107")
 					(unit 1)
 				)
@@
 		(in_pos_files yes)
 		(dnp no)
-		(property "Reference" "#PWR0106"
+		(property "Reference" "#PWR088"
 			(at 142.24 41.91 0)
 			(hide yes)
@@
 			(project "meko"
 				(path "/da54f10a-146b-4941-a9c7-55c7173bb101/cf3a540d-b7d8-4416-baa0-bfc874a83584"
-					(reference "#PWR0106")
+					(reference "#PWR088")
 					(unit 1)
 				)
@@
 		(in_pos_files yes)
 		(dnp no)
-		(property "Reference" "#PWR0105"
+		(property "Reference" "#PWR089"
 			(at 167.64 41.91 0)
 			(hide yes)
@@
 			(project "meko"
 				(path "/da54f10a-146b-4941-a9c7-55c7173bb101/cf3a540d-b7d8-4416-baa0-bfc874a83584"
-					(reference "#PWR0105")
+					(reference "#PWR089")
 					(unit 1)
 				)
@@
 		(in_pos_files yes)
 		(dnp no)
-		(property "Reference" "R32"
+		(property "Reference" "R28"
 			(at 73.152 132.715 0)
 			(show_name no)
@@
 			(project "meko"
 				(path "/da54f10a-146b-4941-a9c7-55c7173bb101/cf3a540d-b7d8-4416-baa0-bfc874a83584"
-					(reference "R32")
+					(reference "R28")
 					(unit 1)
 				)
@@
 		(in_pos_files yes)
 		(dnp no)
-		(property "Reference" "#PWR0107"
+		(property "Reference" "#PWR092"
 			(at 57.15 130.81 0)
 			(hide yes)
@@
 			(project "meko"
 				(path "/da54f10a-146b-4941-a9c7-55c7173bb101/cf3a540d-b7d8-4416-baa0-bfc874a83584"
-					(reference "#PWR0107")
+					(reference "#PWR092")
 					(unit 1)
 				)
@@
 		(in_pos_files yes)
 		(dnp no)
-		(property "Reference" "R31"
+		(property "Reference" "R27"
 			(at 66.802 132.715 0)
 			(show_name no)
@@
 			(project "meko"
 				(path "/da54f10a-146b-4941-a9c7-55c7173bb101/cf3a540d-b7d8-4416-baa0-bfc874a83584"
-					(reference "R31")
+					(reference "R27")
 					(unit 1)
 				)
@@
 		(in_pos_files yes)
 		(dnp no)
-		(property "Reference" "#PWR0102"
+		(property "Reference" "#PWR087"
 			(at 156.21 35.56 0)
 			(hide yes)
@@
 			(project "meko"
 				(path "/da54f10a-146b-4941-a9c7-55c7173bb101/cf3a540d-b7d8-4416-baa0-bfc874a83584"
-					(reference "#PWR0102")
+					(reference "#PWR087")
 					(unit 1)
 				)
@@
 		(in_pos_files yes)
 		(dnp no)
-		(property "Reference" "#PWR0103"
+		(property "Reference" "#PWR086"
 			(at 153.67 35.56 0)
 			(hide yes)
@@
 			(project "meko"
 				(path "/da54f10a-146b-4941-a9c7-55c7173bb101/cf3a540d-b7d8-4416-baa0-bfc874a83584"
-					(reference "#PWR0103")
+					(reference "#PWR086")
 					(unit 1)
 				)
@@
 		(in_pos_files yes)
 		(dnp no)
-		(property "Reference" "C31"
+		(property "Reference" "C109"
 			(at 210.312 129.54 90)
 			(show_name no)
@@
 			(project "meko"
 				(path "/da54f10a-146b-4941-a9c7-55c7173bb101/cf3a540d-b7d8-4416-baa0-bfc874a83584"
-					(reference "C31")
+					(reference "C109")
 					(unit 1)
 				)
@@
 		(in_pos_files yes)
 		(dnp no)
-		(property "Reference" "R30"
+		(property "Reference" "R26"
 			(at 60.452 132.715 0)
 			(show_name no)
@@
 			(project "meko"
 				(path "/da54f10a-146b-4941-a9c7-55c7173bb101/cf3a540d-b7d8-4416-baa0-bfc874a83584"
-					(reference "R30")
+					(reference "R26")
 					(unit 1)
 				)
@@
 		(in_pos_files yes)
 		(dnp no)
-		(property "Reference" "R38"
+		(property "Reference" "R23"
 			(at 86.868 77.978 0)
 			(show_name no)
@@
 			(project "meko"
 				(path "/da54f10a-146b-4941-a9c7-55c7173bb101/cf3a540d-b7d8-4416-baa0-bfc874a83584"
-					(reference "R38")
+					(reference "R23")
 					(unit 1)
 				)
@@
 		(in_pos_files yes)
 		(dnp no)
-		(property "Reference" "C30"
+		(property "Reference" "C108"
 			(at 210.312 121.92 90)
 			(show_name no)
@@
 			(project "meko"
 				(path "/da54f10a-146b-4941-a9c7-55c7173bb101/cf3a540d-b7d8-4416-baa0-bfc874a83584"
-					(reference "C30")
+					(reference "C108")
 					(unit 1)
 				)
@@
 		(dnp no)
 		(fields_autoplaced yes)
-		(property "Reference" "#PWR0109"
+		(property "Reference" "#PWR090"
 			(at 90.17 88.9 0)
 			(hide yes)
@@
 			(project "meko"
 				(path "/da54f10a-146b-4941-a9c7-55c7173bb101/cf3a540d-b7d8-4416-baa0-bfc874a83584"
-					(reference "#PWR0109")
+					(reference "#PWR090")
 					(unit 1)
 				)
@@
 		(in_pos_files yes)
 		(dnp no)
-		(property "Reference" "#PWR069"
+		(property "Reference" "#PWR093"
 			(at 215.9 138.43 0)
 			(hide yes)
@@
 			(project "meko"
 				(path "/da54f10a-146b-4941-a9c7-55c7173bb101/cf3a540d-b7d8-4416-baa0-bfc874a83584"
-					(reference "#PWR069")
+					(reference "#PWR093")
 					(unit 1)
 				)
@@
 		(in_pos_files yes)
 		(dnp no)
-		(property "Reference" "R35"
+		(property "Reference" "R31"
 			(at 118.618 159.258 0)
 			(show_name no)
@@
 			(project "meko"
 				(path "/da54f10a-146b-4941-a9c7-55c7173bb101/cf3a540d-b7d8-4416-baa0-bfc874a83584"
-					(reference "R35")
+					(reference "R31")
 					(unit 1)
 				)
@@
 		(in_pos_files yes)
 		(dnp no)
-		(property "Reference" "#PWR0104"
+		(property "Reference" "#PWR091"
 			(at 186.69 97.79 0)
 			(hide yes)
@@
 			(project "meko"
 				(path "/da54f10a-146b-4941-a9c7-55c7173bb101/cf3a540d-b7d8-4416-baa0-bfc874a83584"
-					(reference "#PWR0104")
+					(reference "#PWR091")
 					(unit 1)
 				)
@@
 		(in_pos_files yes)
 		(dnp no)
-		(property "Reference" "R39"
+		(property "Reference" "R24"
 			(at 93.218 77.978 0)
 			(show_name no)
@@
 			(project "meko"
 				(path "/da54f10a-146b-4941-a9c7-55c7173bb101/cf3a540d-b7d8-4416-baa0-bfc874a83584"
-					(reference "R39")
+					(reference "R24")
 					(unit 1)
 				)
@@
 		(dnp no)
 		(fields_autoplaced yes)
-		(property "Reference" "#PWR0108"
+		(property "Reference" "#PWR094"
 			(at 115.57 170.18 0)
 			(hide yes)
@@
 			(project "meko"
 				(path "/da54f10a-146b-4941-a9c7-55c7173bb101/cf3a540d-b7d8-4416-baa0-bfc874a83584"
-					(reference "#PWR0108")
+					(reference "#PWR094")
 					(unit 1)
 				)
@@
 		(in_pos_files yes)
 		(dnp no)
-		(property "Reference" "R29"
+		(property "Reference" "R25"
 			(at 54.102 132.715 0)
 			(show_name no)
@@
 			(project "meko"
 				(path "/da54f10a-146b-4941-a9c7-55c7173bb101/cf3a540d-b7d8-4416-baa0-bfc874a83584"
-					(reference "R29")
+					(reference "R25")
 					(unit 1)
 				)
@@
 		(in_pos_files yes)
 		(dnp no)
-		(property "Reference" "R34"
+		(property "Reference" "R30"
 			(at 112.268 159.258 0)
 			(show_name no)
@@
 			(project "meko"
 				(path "/da54f10a-146b-4941-a9c7-55c7173bb101/cf3a540d-b7d8-4416-baa0-bfc874a83584"
-					(reference "R34")
+					(reference "R30")
 					(unit 1)
 				)
@@
 		(in_pos_files yes)
 		(dnp no)
-		(property "Reference" "R33"
+		(property "Reference" "R29"
 			(at 79.502 132.715 0)
 			(show_name no)
@@
 			(project "meko"
 				(path "/da54f10a-146b-4941-a9c7-55c7173bb101/cf3a540d-b7d8-4416-baa0-bfc874a83584"
-					(reference "R33")
+					(reference "R29")
 					(unit 1)
 				)
@@
 		(dnp no)
 		(fields_autoplaced yes)
-		(property "Reference" "#PWR09"
+		(property "Reference" "#PWR095"
 			(at 154.94 170.18 0)
 			(hide yes)
@@
 			(project "meko"
 				(path "/da54f10a-146b-4941-a9c7-55c7173bb101/cf3a540d-b7d8-4416-baa0-bfc874a83584"
-					(reference "#PWR09")
+					(reference "#PWR095")
 					(unit 1)
 				)
