File: hardware/pcb/wireless.kicad_sch (KiCad schematic)
At the start: 15 parts, among them IC2 MAYA-W386-00B, Y3 32kHz768

Commit message: added a bunch testpoints
Parts:
- added TP30: BT_H_WAKE, TestPoint:TestPoint_Pad_D1.0mm, symbol Connector:TestPoint
- added TP31: BT_D_WAKE, TestPoint:TestPoint_Pad_D1.0mm, symbol Connector:TestPoint
- added TP32: BT_EN, TestPoint:TestPoint_Pad_D1.0mm, symbol Connector:TestPoint
- added TP33: WL_H_WAKE, TestPoint:TestPoint_Pad_D1.0mm, symbol Connector:TestPoint
- added TP34: WL_D_WAKE, TestPoint:TestPoint_Pad_D1.0mm, symbol Connector:TestPoint
- added TP35: WL_EN, TestPoint:TestPoint_Pad_D1.0mm, symbol Connector:TestPoint
- added TP36: RF_RX, TestPoint:TestPoint_Pad_D1.0mm, symbol Connector:TestPoint
- added TP37: RF_TX, TestPoint:TestPoint_Pad_D1.0mm, symbol Connector:TestPoint
- added TP38: RF_~{CTS}, TestPoint:TestPoint_Pad_D1.0mm, symbol Connector:TestPoint
- added TP39: RF_~{RTS}, TestPoint:TestPoint_Pad_D1.0mm, symbol Connector:TestPoint
- added TP40: RF_MCLK, TestPoint:TestPoint_Pad_D1.0mm, symbol Connector:TestPoint
- added TP41: RF_BCLK, TestPoint:TestPoint_Pad_D1.0mm, symbol Connector:TestPoint
- added TP42: RF_FSYNC, TestPoint:TestPoint_Pad_D1.0mm, symbol Connector:TestPoint
- added TP43: RF_DOUT, TestPoint:TestPoint_Pad_D1.0mm, symbol Connector:TestPoint
- added TP44: RF_DIN, TestPoint:TestPoint_Pad_D1.0mm, symbol Connector:TestPoint
- added TP45: RF_CK, TestPoint:TestPoint_Pad_D1.0mm, symbol Connector:TestPoint
- added TP46: RF_CMD, TestPoint:TestPoint_Pad_D1.0mm, symbol Connector:TestPoint
- added TP47: RF_DAT0, TestPoint:TestPoint_Pad_D1.0mm, symbol Connector:TestPoint
- added TP48: RF_DAT1, TestPoint:TestPoint_Pad_D1.0mm, symbol Connector:TestPoint
- added TP49: RF_DAT2, TestPoint:TestPoint_Pad_D1.0mm, symbol Connector:TestPoint
- added TP50: RF_DAT3, TestPoint:TestPoint_Pad_D1.0mm, symbol Connector:TestPoint
Connections:
- net BCLK: now also TP41.1
- net BT.DEV_WAKE: now also TP31.1
- net BT.EN: now also TP32.1
- net BT.HOST_WAKE: now also TP30.1
- net CK: now also TP45.1
- net CMD: now also TP46.1
- net DAT0: now also TP47.1
- net DAT1: now also TP48.1
- net DAT2: now also TP49.1
- net DAT3: now also TP50.1
- net DIN: now also TP44.1
- net DOUT: now also TP43.1
- net FSYNC: now also TP42.1
- net MCLK: now also TP40.1
- net RX: now also TP36.1
- net TX: now also TP37.1
- net WL.DEV_WAKE: now also TP34.1
- net WL.EN: now also TP35.1
- net WL.HOST_WAKE: now also TP33.1
- net CTSN renamed ~{CTS}
- net ~{CTS}: now also TP38.1
- net RTSN renamed ~{RTS}
- net ~{RTS}: now also TP39.1
Other:
- moved on the sheet: C107

Commit message: removed testpoints on sd cards, since I can probe the pins there
Parts:
- renumbered R25 to R23, R26 to R24, R27 to R25, R28 to R26, R29 to R27, R23 to R28, R24 to R29, TP30 to TP26, TP31 to TP27, TP32 to TP28, TP36 to TP29, TP37 to TP30, TP38 to TP31, TP39 to TP32, TP40 to TP33, TP41 to TP34, TP42 to TP35, TP43 to TP36, TP44 to TP37, TP33 to TP38, TP34 to TP39, TP35 to TP40, TP45 to TP41, TP46 to TP42, TP47 to TP43, TP48 to TP44, TP49 to TP45, TP50 to TP46

Commit message: added capacitor to sama ddr vref pin
Parts:
- renumbered C106 to C108, C107 to C109, C108 to C110, C109 to C111, R23 to R25, R24 to R26, R25 to R27, R26 to R28, R27 to R29, R28 to R30, R29 to R31, R30 to R32, R31 to R33
Changed lines of the file:
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@@
 		(in_pos_files yes)
 		(dnp no)
-		(property "Reference" "C106"
+		(property "Reference" "C108"
 			(at 146.304 35.56 90)
 			(show_name no)
@@
 			(project "meko"
 				(path "/da54f10a-146b-4941-a9c7-55c7173bb101/cf3a540d-b7d8-4416-baa0-bfc874a83584"
-					(reference "C106")
+					(reference "C108")
 					(unit 1)
 				)
@@
 		(in_pos_files yes)
 		(dnp no)
-		(property "Reference" "C107"
+		(property "Reference" "C109"
 			(at 162.814 35.56 90)
 			(show_name no)
@@
 			(project "meko"
 				(path "/da54f10a-146b-4941-a9c7-55c7173bb101/cf3a540d-b7d8-4416-baa0-bfc874a83584"
-					(reference "C107")
+					(reference "C109")
 					(unit 1)
 				)
@@
 		(in_pos_files yes)
 		(dnp no)
-		(property "Reference" "#PWR089"
+		(property "Reference" "#PWR091"
 			(at 139.7 41.91 0)
 			(hide yes)
@@
 			(project "meko"
 				(path "/da54f10a-146b-4941-a9c7-55c7173bb101/cf3a540d-b7d8-4416-baa0-bfc874a83584"
-					(reference "#PWR089")
+					(reference "#PWR091")
 					(unit 1)
 				)
@@
 		(in_pos_files yes)
 		(dnp no)
-		(property "Reference" "#PWR093"
+		(property "Reference" "#PWR095"
 			(at 170.18 41.91 0)
 			(hide yes)
@@
 			(project "meko"
 				(path "/da54f10a-146b-4941-a9c7-55c7173bb101/cf3a540d-b7d8-4416-baa0-bfc874a83584"
-					(reference "#PWR093")
+					(reference "#PWR095")
 					(unit 1)
 				)
@@
 		(in_pos_files yes)
 		(dnp no)
-		(property "Reference" "R26"
+		(property "Reference" "R28"
 			(at 73.152 132.715 0)
 			(show_name no)
@@
 			(project "meko"
 				(path "/da54f10a-146b-4941-a9c7-55c7173bb101/cf3a540d-b7d8-4416-baa0-bfc874a83584"
-					(reference "R26")
+					(reference "R28")
 					(unit 1)
 				)
@@
 		(in_pos_files yes)
 		(dnp no)
-		(property "Reference" "#PWR086"
+		(property "Reference" "#PWR088"
 			(at 57.15 130.81 0)
 			(hide yes)
@@
 			(project "meko"
 				(path "/da54f10a-146b-4941-a9c7-55c7173bb101/cf3a540d-b7d8-4416-baa0-bfc874a83584"
-					(reference "#PWR086")
+					(reference "#PWR088")
 					(unit 1)
 				)
@@
 		(in_pos_files yes)
 		(dnp no)
-		(property "Reference" "R25"
+		(property "Reference" "R27"
 			(at 66.802 132.715 0)
 			(show_name no)
@@
 			(project "meko"
 				(path "/da54f10a-146b-4941-a9c7-55c7173bb101/cf3a540d-b7d8-4416-baa0-bfc874a83584"
-					(reference "R25")
+					(reference "R27")
 					(unit 1)
 				)
@@
 		(in_pos_files yes)
 		(dnp no)
-		(property "Reference" "#PWR092"
+		(property "Reference" "#PWR094"
 			(at 156.21 35.56 0)
 			(hide yes)
@@
 			(project "meko"
 				(path "/da54f10a-146b-4941-a9c7-55c7173bb101/cf3a540d-b7d8-4416-baa0-bfc874a83584"
-					(reference "#PWR092")
+					(reference "#PWR094")
 					(unit 1)
 				)
@@
 		(in_pos_files yes)
 		(dnp no)
-		(property "Reference" "#PWR090"
+		(property "Reference" "#PWR092"
 			(at 153.67 35.56 0)
 			(hide yes)
@@
 			(project "meko"
 				(path "/da54f10a-146b-4941-a9c7-55c7173bb101/cf3a540d-b7d8-4416-baa0-bfc874a83584"
-					(reference "#PWR090")
+					(reference "#PWR092")
 					(unit 1)
 				)
@@
 		(in_pos_files yes)
 		(dnp no)
-		(property "Reference" "C109"
+		(property "Reference" "C111"
 			(at 210.312 129.54 90)
 			(show_name no)
@@
 			(project "meko"
 				(path "/da54f10a-146b-4941-a9c7-55c7173bb101/cf3a540d-b7d8-4416-baa0-bfc874a83584"
-					(reference "C109")
+					(reference "C111")
 					(unit 1)
 				)
@@
 		(in_pos_files yes)
 		(dnp no)
-		(property "Reference" "R24"
+		(property "Reference" "R26"
 			(at 60.452 132.715 0)
 			(show_name no)
@@
 			(project "meko"
 				(path "/da54f10a-146b-4941-a9c7-55c7173bb101/cf3a540d-b7d8-4416-baa0-bfc874a83584"
-					(reference "R24")
+					(reference "R26")
 					(unit 1)
 				)
@@
 		(in_pos_files yes)
 		(dnp no)
-		(property "Reference" "R28"
+		(property "Reference" "R30"
 			(at 86.868 77.978 0)
 			(show_name no)
@@
 			(project "meko"
 				(path "/da54f10a-146b-4941-a9c7-55c7173bb101/cf3a540d-b7d8-4416-baa0-bfc874a83584"
-					(reference "R28")
+					(reference "R30")
 					(unit 1)
 				)
@@
 		(in_pos_files yes)
 		(dnp no)
-		(property "Reference" "C108"
+		(property "Reference" "C110"
 			(at 210.312 121.92 90)
 			(show_name no)
@@
 			(project "meko"
 				(path "/da54f10a-146b-4941-a9c7-55c7173bb101/cf3a540d-b7d8-4416-baa0-bfc874a83584"
-					(reference "C108")
+					(reference "C110")
 					(unit 1)
 				)
@@
 		(dnp no)
 		(fields_autoplaced yes)
-		(property "Reference" "#PWR087"
+		(property "Reference" "#PWR089"
 			(at 90.17 88.9 0)
 			(hide yes)
@@
 			(project "meko"
 				(path "/da54f10a-146b-4941-a9c7-55c7173bb101/cf3a540d-b7d8-4416-baa0-bfc874a83584"
-					(reference "#PWR087")
+					(reference "#PWR089")
 					(unit 1)
 				)
@@
 		(in_pos_files yes)
 		(dnp no)
-		(property "Reference" "#PWR095"
+		(property "Reference" "#PWR097"
 			(at 215.9 138.43 0)
 			(hide yes)
@@
 			(project "meko"
 				(path "/da54f10a-146b-4941-a9c7-55c7173bb101/cf3a540d-b7d8-4416-baa0-bfc874a83584"
-					(reference "#PWR095")
+					(reference "#PWR097")
 					(unit 1)
 				)
@@
 		(in_pos_files yes)
 		(dnp no)
-		(property "Reference" "R31"
+		(property "Reference" "R33"
 			(at 118.618 159.258 0)
 			(show_name no)
@@
 			(project "meko"
 				(path "/da54f10a-146b-4941-a9c7-55c7173bb101/cf3a540d-b7d8-4416-baa0-bfc874a83584"
-					(reference "R31")
+					(reference "R33")
 					(unit 1)
 				)
@@
 		(in_pos_files yes)
 		(dnp no)
-		(property "Reference" "#PWR094"
+		(property "Reference" "#PWR096"
 			(at 186.69 97.79 0)
 			(hide yes)
@@
 			(project "meko"
 				(path "/da54f10a-146b-4941-a9c7-55c7173bb101/cf3a540d-b7d8-4416-baa0-bfc874a83584"
-					(reference "#PWR094")
+					(reference "#PWR096")
 					(unit 1)
 				)
@@
 		(in_pos_files yes)
 		(dnp no)
-		(property "Reference" "R29"
+		(property "Reference" "R31"
 			(at 93.218 77.978 0)
 			(show_name no)
@@
 			(project "meko"
 				(path "/da54f10a-146b-4941-a9c7-55c7173bb101/cf3a540d-b7d8-4416-baa0-bfc874a83584"
-					(reference "R29")
+					(reference "R31")
 					(unit 1)
 				)
@@
 		(dnp no)
 		(fields_autoplaced yes)
-		(property "Reference" "#PWR088"
+		(property "Reference" "#PWR090"
 			(at 115.57 170.18 0)
 			(hide yes)
@@
 			(project "meko"
 				(path "/da54f10a-146b-4941-a9c7-55c7173bb101/cf3a540d-b7d8-4416-baa0-bfc874a83584"
-					(reference "#PWR088")
+					(reference "#PWR090")
 					(unit 1)
 				)
@@
 		(in_pos_files yes)
 		(dnp no)
-		(property "Reference" "R23"
+		(property "Reference" "R25"
 			(at 54.102 132.715 0)
 			(show_name no)
@@
 			(project "meko"
 				(path "/da54f10a-146b-4941-a9c7-55c7173bb101/cf3a540d-b7d8-4416-baa0-bfc874a83584"
-					(reference "R23")
+					(reference "R25")
 					(unit 1)
 				)
@@
 		(in_pos_files yes)
 		(dnp no)
-		(property "Reference" "R30"
+		(property "Reference" "R32"
 			(at 112.268 159.258 0)
 			(show_name no)
@@
 			(project "meko"
 				(path "/da54f10a-146b-4941-a9c7-55c7173bb101/cf3a540d-b7d8-4416-baa0-bfc874a83584"
-					(reference "R30")
+					(reference "R32")
 					(unit 1)
 				)
@@
 		(in_pos_files yes)
 		(dnp no)
-		(property "Reference" "R27"
+		(property "Reference" "R29"
 			(at 79.502 132.715 0)
 			(show_name no)
@@
 			(project "meko"
 				(path "/da54f10a-146b-4941-a9c7-55c7173bb101/cf3a540d-b7d8-4416-baa0-bfc874a83584"
-					(reference "R27")
+					(reference "R29")
 					(unit 1)
 				)
@@
 		(dnp no)
 		(fields_autoplaced yes)
-		(property "Reference" "#PWR091"
+		(property "Reference" "#PWR093"
 			(at 154.94 170.18 0)
 			(hide yes)
@@
 			(project "meko"
 				(path "/da54f10a-146b-4941-a9c7-55c7173bb101/cf3a540d-b7d8-4416-baa0-bfc874a83584"
-					(reference "#PWR091")
+					(reference "#PWR093")
 					(unit 1)
 				)

Commit message: didn't save last time :sob:
Parts:
- renumbered C108 to C109, C109 to C110, C110 to C111, C111 to C112
Changed lines of the file:
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@@
 		(in_pos_files yes)
 		(dnp no)
-		(property "Reference" "C108"
+		(property "Reference" "C109"
 			(at 146.304 35.56 90)
 			(show_name no)
@@
 			(project "meko"
 				(path "/da54f10a-146b-4941-a9c7-55c7173bb101/cf3a540d-b7d8-4416-baa0-bfc874a83584"
-					(reference "C108")
+					(reference "C109")
 					(unit 1)
 				)
@@
 		(in_pos_files yes)
 		(dnp no)
-		(property "Reference" "C109"
+		(property "Reference" "C110"
 			(at 162.814 35.56 90)
 			(show_name no)
@@
 			(project "meko"
 				(path "/da54f10a-146b-4941-a9c7-55c7173bb101/cf3a540d-b7d8-4416-baa0-bfc874a83584"
-					(reference "C109")
+					(reference "C110")
 					(unit 1)
 				)
@@
 		(in_pos_files yes)
 		(dnp no)
-		(property "Reference" "#PWR091"
+		(property "Reference" "#PWR092"
 			(at 139.7 41.91 0)
 			(hide yes)
@@
 			(project "meko"
 				(path "/da54f10a-146b-4941-a9c7-55c7173bb101/cf3a540d-b7d8-4416-baa0-bfc874a83584"
-					(reference "#PWR091")
+					(reference "#PWR092")
 					(unit 1)
 				)
@@
 		(in_pos_files yes)
 		(dnp no)
-		(property "Reference" "#PWR095"
+		(property "Reference" "#PWR096"
 			(at 170.18 41.91 0)
 			(hide yes)
@@
 			(project "meko"
 				(path "/da54f10a-146b-4941-a9c7-55c7173bb101/cf3a540d-b7d8-4416-baa0-bfc874a83584"
-					(reference "#PWR095")
+					(reference "#PWR096")
 					(unit 1)
 				)
@@
 		(in_pos_files yes)
 		(dnp no)
-		(property "Reference" "#PWR088"
+		(property "Reference" "#PWR089"
 			(at 57.15 130.81 0)
 			(hide yes)
@@
 			(project "meko"
 				(path "/da54f10a-146b-4941-a9c7-55c7173bb101/cf3a540d-b7d8-4416-baa0-bfc874a83584"
-					(reference "#PWR088")
+					(reference "#PWR089")
 					(unit 1)
 				)
@@
 		(in_pos_files yes)
 		(dnp no)
-		(property "Reference" "#PWR094"
+		(property "Reference" "#PWR095"
 			(at 156.21 35.56 0)
 			(hide yes)
@@
 			(project "meko"
 				(path "/da54f10a-146b-4941-a9c7-55c7173bb101/cf3a540d-b7d8-4416-baa0-bfc874a83584"
-					(reference "#PWR094")
+					(reference "#PWR095")
 					(unit 1)
 				)
@@
 		(in_pos_files yes)
 		(dnp no)
-		(property "Reference" "#PWR092"
+		(property "Reference" "#PWR093"
 			(at 153.67 35.56 0)
 			(hide yes)
@@
 			(project "meko"
 				(path "/da54f10a-146b-4941-a9c7-55c7173bb101/cf3a540d-b7d8-4416-baa0-bfc874a83584"
-					(reference "#PWR092")
+					(reference "#PWR093")
 					(unit 1)
 				)
@@
 		(in_pos_files yes)
 		(dnp no)
-		(property "Reference" "C111"
+		(property "Reference" "C112"
 			(at 210.312 129.54 90)
 			(show_name no)
@@
 			(project "meko"
 				(path "/da54f10a-146b-4941-a9c7-55c7173bb101/cf3a540d-b7d8-4416-baa0-bfc874a83584"
-					(reference "C111")
+					(reference "C112")
 					(unit 1)
 				)
@@
 		(in_pos_files yes)
 		(dnp no)
-		(property "Reference" "C110"
+		(property "Reference" "C111"
 			(at 210.312 121.92 90)
 			(show_name no)
@@
 			(project "meko"
 				(path "/da54f10a-146b-4941-a9c7-55c7173bb101/cf3a540d-b7d8-4416-baa0-bfc874a83584"
-					(reference "C110")
+					(reference "C111")
 					(unit 1)
 				)
@@
 		(dnp no)
 		(fields_autoplaced yes)
-		(property "Reference" "#PWR089"
+		(property "Reference" "#PWR090"
 			(at 90.17 88.9 0)
 			(hide yes)
@@
 			(project "meko"
 				(path "/da54f10a-146b-4941-a9c7-55c7173bb101/cf3a540d-b7d8-4416-baa0-bfc874a83584"
-					(reference "#PWR089")
+					(reference "#PWR090")
 					(unit 1)
 				)
@@
 		(in_pos_files yes)
 		(dnp no)
-		(property "Reference" "#PWR097"
+		(property "Reference" "#PWR098"
 			(at 215.9 138.43 0)
 			(hide yes)
@@
 			(project "meko"
 				(path "/da54f10a-146b-4941-a9c7-55c7173bb101/cf3a540d-b7d8-4416-baa0-bfc874a83584"
-					(reference "#PWR097")
+					(reference "#PWR098")
 					(unit 1)
 				)
@@
 		(in_pos_files yes)
 		(dnp no)
-		(property "Reference" "#PWR096"
+		(property "Reference" "#PWR097"
 			(at 186.69 97.79 0)
 			(hide yes)
@@
 			(project "meko"
 				(path "/da54f10a-146b-4941-a9c7-55c7173bb101/cf3a540d-b7d8-4416-baa0-bfc874a83584"
-					(reference "#PWR096")
+					(reference "#PWR097")
 					(unit 1)
 				)
@@
 		(dnp no)
 		(fields_autoplaced yes)
-		(property "Reference" "#PWR090"
+		(property "Reference" "#PWR091"
 			(at 115.57 170.18 0)
 			(hide yes)
@@
 			(project "meko"
 				(path "/da54f10a-146b-4941-a9c7-55c7173bb101/cf3a540d-b7d8-4416-baa0-bfc874a83584"
-					(reference "#PWR090")
+					(reference "#PWR091")
 					(unit 1)
 				)
@@
 		(dnp no)
 		(fields_autoplaced yes)
-		(property "Reference" "#PWR093"
+		(property "Reference" "#PWR094"
 			(at 154.94 170.18 0)
 			(hide yes)
@@
 			(project "meko"
 				(path "/da54f10a-146b-4941-a9c7-55c7173bb101/cf3a540d-b7d8-4416-baa0-bfc874a83584"
-					(reference "#PWR093")
+					(reference "#PWR094")
 					(unit 1)
 				)

Commit message: added pullups for jtag
Parts:
- renumbered R30 to R31, R31 to R32, R25 to R33, R26 to R34, R27 to R35, R28 to R36, R29 to R37, R32 to R38, R33 to R39
Changed lines of the file:
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@@
 		(in_pos_files yes)
 		(dnp no)
-		(property "Reference" "#PWR096"
+		(property "Reference" "#PWR093"
 			(at 170.18 41.91 0)
 			(hide yes)
@@
 			(project "meko"
 				(path "/da54f10a-146b-4941-a9c7-55c7173bb101/cf3a540d-b7d8-4416-baa0-bfc874a83584"
-					(reference "#PWR096")
+					(reference "#PWR093")
 					(unit 1)
 				)
@@
 		(in_pos_files yes)
 		(dnp no)
-		(property "Reference" "R28"
+		(property "Reference" "R36"
 			(at 73.152 132.715 0)
 			(show_name no)
@@
 			(project "meko"
 				(path "/da54f10a-146b-4941-a9c7-55c7173bb101/cf3a540d-b7d8-4416-baa0-bfc874a83584"
-					(reference "R28")
+					(reference "R36")
 					(unit 1)
 				)
@@
 		(in_pos_files yes)
 		(dnp no)
-		(property "Reference" "#PWR089"
+		(property "Reference" "#PWR096"
 			(at 57.15 130.81 0)
 			(hide yes)
@@
 			(project "meko"
 				(path "/da54f10a-146b-4941-a9c7-55c7173bb101/cf3a540d-b7d8-4416-baa0-bfc874a83584"
-					(reference "#PWR089")
+					(reference "#PWR096")
 					(unit 1)
 				)
@@
 		(in_pos_files yes)
 		(dnp no)
-		(property "Reference" "R27"
+		(property "Reference" "R35"
 			(at 66.802 132.715 0)
 			(show_name no)
@@
 			(project "meko"
 				(path "/da54f10a-146b-4941-a9c7-55c7173bb101/cf3a540d-b7d8-4416-baa0-bfc874a83584"
-					(reference "R27")
+					(reference "R35")
 					(unit 1)
 				)
@@
 		(in_pos_files yes)
 		(dnp no)
-		(property "Reference" "#PWR095"
+		(property "Reference" "#PWR091"
 			(at 156.21 35.56 0)
 			(hide yes)
@@
 			(project "meko"
 				(path "/da54f10a-146b-4941-a9c7-55c7173bb101/cf3a540d-b7d8-4416-baa0-bfc874a83584"
-					(reference "#PWR095")
+					(reference "#PWR091")
 					(unit 1)
 				)
@@
 		(in_pos_files yes)
 		(dnp no)
-		(property "Reference" "#PWR093"
+		(property "Reference" "#PWR090"
 			(at 153.67 35.56 0)
 			(hide yes)
@@
 			(project "meko"
 				(path "/da54f10a-146b-4941-a9c7-55c7173bb101/cf3a540d-b7d8-4416-baa0-bfc874a83584"
-					(reference "#PWR093")
+					(reference "#PWR090")
 					(unit 1)
 				)
@@
 		(in_pos_files yes)
 		(dnp no)
-		(property "Reference" "R26"
+		(property "Reference" "R34"
 			(at 60.452 132.715 0)
 			(show_name no)
@@
 			(project "meko"
 				(path "/da54f10a-146b-4941-a9c7-55c7173bb101/cf3a540d-b7d8-4416-baa0-bfc874a83584"
-					(reference "R26")
+					(reference "R34")
 					(unit 1)
 				)
@@
 		(in_pos_files yes)
 		(dnp no)
-		(property "Reference" "R30"
+		(property "Reference" "R31"
 			(at 86.868 77.978 0)
 			(show_name no)
@@
 			(project "meko"
 				(path "/da54f10a-146b-4941-a9c7-55c7173bb101/cf3a540d-b7d8-4416-baa0-bfc874a83584"
-					(reference "R30")
+					(reference "R31")
 					(unit 1)
 				)
@@
 		(dnp no)
 		(fields_autoplaced yes)
-		(property "Reference" "#PWR090"
+		(property "Reference" "#PWR094"
 			(at 90.17 88.9 0)
 			(hide yes)
@@
 			(project "meko"
 				(path "/da54f10a-146b-4941-a9c7-55c7173bb101/cf3a540d-b7d8-4416-baa0-bfc874a83584"
-					(reference "#PWR090")
+					(reference "#PWR094")
 					(unit 1)
 				)
@@
 		(in_pos_files yes)
 		(dnp no)
-		(property "Reference" "#PWR098"
+		(property "Reference" "#PWR097"
 			(at 215.9 138.43 0)
 			(hide yes)
@@
 			(project "meko"
 				(path "/da54f10a-146b-4941-a9c7-55c7173bb101/cf3a540d-b7d8-4416-baa0-bfc874a83584"
-					(reference "#PWR098")
+					(reference "#PWR097")
 					(unit 1)
 				)
@@
 		(in_pos_files yes)
 		(dnp no)
-		(property "Reference" "R33"
+		(property "Reference" "R39"
 			(at 118.618 159.258 0)
 			(show_name no)
@@
 			(project "meko"
 				(path "/da54f10a-146b-4941-a9c7-55c7173bb101/cf3a540d-b7d8-4416-baa0-bfc874a83584"
-					(reference "R33")
+					(reference "R39")
 					(unit 1)
 				)
@@
 		(in_pos_files yes)
 		(dnp no)
-		(property "Reference" "#PWR097"
+		(property "Reference" "#PWR095"
 			(at 186.69 97.79 0)
 			(hide yes)
@@
 			(project "meko"
 				(path "/da54f10a-146b-4941-a9c7-55c7173bb101/cf3a540d-b7d8-4416-baa0-bfc874a83584"
-					(reference "#PWR097")
+					(reference "#PWR095")
 					(unit 1)
 				)
@@
 		(in_pos_files yes)
 		(dnp no)
-		(property "Reference" "R31"
+		(property "Reference" "R32"
 			(at 93.218 77.978 0)
 			(show_name no)
@@
 			(project "meko"
 				(path "/da54f10a-146b-4941-a9c7-55c7173bb101/cf3a540d-b7d8-4416-baa0-bfc874a83584"
-					(reference "R31")
+					(reference "R32")
 					(unit 1)
 				)
@@
 		(dnp no)
 		(fields_autoplaced yes)
-		(property "Reference" "#PWR091"
+		(property "Reference" "#PWR098"
 			(at 115.57 170.18 0)
 			(hide yes)
@@
 			(project "meko"
 				(path "/da54f10a-146b-4941-a9c7-55c7173bb101/cf3a540d-b7d8-4416-baa0-bfc874a83584"
-					(reference "#PWR091")
+					(reference "#PWR098")
 					(unit 1)
 				)
@@
 		(in_pos_files yes)
 		(dnp no)
-		(property "Reference" "R25"
+		(property "Reference" "R33"
 			(at 54.102 132.715 0)
 			(show_name no)
@@
 			(project "meko"
 				(path "/da54f10a-146b-4941-a9c7-55c7173bb101/cf3a540d-b7d8-4416-baa0-bfc874a83584"
-					(reference "R25")
+					(reference "R33")
 					(unit 1)
 				)
@@
 		(in_pos_files yes)
 		(dnp no)
-		(property "Reference" "R32"
+		(property "Reference" "R38"
 			(at 112.268 159.258 0)
 			(show_name no)
@@
 			(project "meko"
 				(path "/da54f10a-146b-4941-a9c7-55c7173bb101/cf3a540d-b7d8-4416-baa0-bfc874a83584"
-					(reference "R32")
+					(reference "R38")
 					(unit 1)
 				)
@@
 		(in_pos_files yes)
 		(dnp no)
-		(property "Reference" "R29"
+		(property "Reference" "R37"
 			(at 79.502 132.715 0)
 			(show_name no)
@@
 			(project "meko"
 				(path "/da54f10a-146b-4941-a9c7-55c7173bb101/cf3a540d-b7d8-4416-baa0-bfc874a83584"
-					(reference "R29")
+					(reference "R37")
 					(unit 1)
 				)
@@
 		(dnp no)
 		(fields_autoplaced yes)
-		(property "Reference" "#PWR094"
+		(property "Reference" "#PWR099"
 			(at 154.94 170.18 0)
 			(hide yes)
@@
 			(project "meko"
 				(path "/da54f10a-146b-4941-a9c7-55c7173bb101/cf3a540d-b7d8-4416-baa0-bfc874a83584"
-					(reference "#PWR094")
+					(reference "#PWR099")
 					(unit 1)
 				)

Commit message: moved some caps to 0201
Parts:
- C111, C112: footprint Capacitor_SMD:C_0402_1005Metric -> Capacitor_SMD:C_0201_0603Metric
Changed lines of the file:
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@@
 			)
 		)
-		(property "Footprint" "Capacitor_SMD:C_0402_1005Metric"
+		(property "Footprint" "Capacitor_SMD:C_0201_0603Metric"
 			(at 209.55 130.81 0)
 			(hide yes)
@@
 			)
 		)
-		(property "Footprint" "Capacitor_SMD:C_0402_1005Metric"
+		(property "Footprint" "Capacitor_SMD:C_0201_0603Metric"
 			(at 209.55 120.65 0)
 			(hide yes)
