File: hardware/pcb/wireless.kicad_sch (KiCad schematic)
At the start: 36 parts, among them IC2 MAYA-W386-00B, Y3 32kHz768

Commit message: more routing
Connections:
- net ANT: now reaches IC2.K9 (RF_ANT1), IC2.L9 (ANT_EXT_FEED)
Changed lines of the file:
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@@
 	(text "Connecting the output to the integrated PCB antenna"
 		(exclude_from_sim no)
-		(at 187.452 99.314 0)
+		(at 195.072 99.06 0)
 		(effects
 			(font
@@
 	(wire
 		(pts
-			(xy 185.42 100.33) (xy 186.69 100.33)
+			(xy 185.42 100.33) (xy 194.31 100.33)
 		)
 		(stroke
@@
 	(wire
 		(pts
-			(xy 186.69 97.79) (xy 186.69 100.33)
+			(xy 194.31 97.79) (xy 194.31 100.33)
 		)
 		(stroke
@@
 	(wire
 		(pts
-			(xy 185.42 97.79) (xy 186.69 97.79)
+			(xy 185.42 97.79) (xy 194.31 97.79)
 		)
 		(stroke
@@
 	(label "RX"
 		(at 232.41 33.02 0)
+		(effects
+			(font
+				(size 1.27 1.27)
+			)
+			(justify left bottom)
+		)
+	)
+	(label "ANT"
+		(at 186.69 97.79 0)
 		(effects
 			(font
@@
 			)
 		)
+	)
+	(netclass_flag ""
+		(length 2.54)
+		(shape round)
+		(at 194.31 97.79 0)
+		(fields_autoplaced yes)
+		(effects
+			(font
+				(size 1.27 1.27)
+			)
+			(justify left bottom)
+		)
+		(property "Netclass" "ANT"
+			(at 195.0085 95.25 0)
+			(show_name no)
+			(do_not_autoplace no)
+			(effects
+				(font
+					(size 1.27 1.27)
+				)
+				(justify left)
+			)
+		)
+		(property "Component Class" ""
+			(at -3.81 3.81 0)
+			(show_name no)
+			(do_not_autoplace no)
+			(effects
+				(font
+					(size 1.27 1.27)
+					(italic yes)
+				)
+			)
+		)

Commit message: cleanup, tespoints, passives
Parts:
- removed TP26: BT_H_WAKE, TestPoint:TestPoint_Pad_D1.0mm, symbol Connector:TestPoint
- removed TP27: BT_D_WAKE, TestPoint:TestPoint_Pad_D1.0mm, symbol Connector:TestPoint
- removed TP38: WL_H_WAKE, TestPoint:TestPoint_Pad_D1.0mm, symbol Connector:TestPoint
- removed TP39: WL_D_WAKE, TestPoint:TestPoint_Pad_D1.0mm, symbol Connector:TestPoint
Other:
- moved on the sheet: TP28, TP29, TP30, TP31, TP32, TP33, TP34, TP35, TP36, TP37, TP40, TP41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
