File: hardware/pcb/display.kicad_sch (KiCad schematic)
At the start: 0 parts

Commit message: bunch of small audio changes
Parts:
- added C32, C37: 1u, symbol Device:C_Small
- added C33: 100n, symbol Device:C_Small
- added J5: 503480-1000, 503480-1000:5034801000, symbol 503480-1000:503480-1000
Connections:
- new net +3V3: C32.2, C37.2, J5.6, J5.7
- new net DISP: C33.2, J5.5
- new net GND: C32.1, C33.1, C37.1, J5.10, J5.11 (MP_1), J5.12 (MP_2), J5.4, J5.8, J5.9
- new net SCLK: J5.1
- new net SCS: J5.3
- new net SI: J5.2
Other:
- note added: "100n ommited, because DISP is not connected to 3V3 by default"

Commit message: looking over stuff, added caps
Parts:
- added R42: 10k, Resistor_SMD:R_0402_1005Metric, symbol Device:R_Small
- C32, C33, C37: footprint (none) -> Capacitor_SMD:C_0402_1005Metric
Connections:
- net DISP: now also R42.2
- net GND: now also R42.1
Other:
- moved on the sheet: C32, C33, C37, J5

Commit message: started cleaning up schematic
Other:
- company: (none) -> Gensis
- title: (none) -> Display
Changed lines of the file:
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@@
 	(generator_version "10.0")
 	(paper "A5")
+	(title_block
+		(title "Display")
+		(rev "v1.0.0")
+		(company "Gensis")
+	)
 	(text "100n ommited, because DISP is not\nconnected to 3V3 by default"
 		(exclude_from_sim no)

Commit message: mainboard: reannotated schematic
Parts:
- renumbered C33 to C118, C32 to C119, C37 to C120, J5 to J8, R42 to R47
Changed lines of the file:
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@@
 		(dnp no)
 		(fields_autoplaced yes)
-		(property "Reference" "#PWR074"
+		(property "Reference" "#PWR0128"
 			(at 105.41 90.17 0)
 			(hide yes)
@@
 			(project "meko"
 				(path "/da54f10a-146b-4941-a9c7-55c7173bb101/122d9c1c-6abd-41a6-b885-d015d8fca76e"
-					(reference "#PWR074")
+					(reference "#PWR0128")
 					(unit 1)
 				)
@@
 		(in_pos_files yes)
 		(dnp no)
-		(property "Reference" "R42"
+		(property "Reference" "R47"
 			(at 83.82 76.454 0)
 			(show_name no)
@@
 			(project "meko"
 				(path "/da54f10a-146b-4941-a9c7-55c7173bb101/122d9c1c-6abd-41a6-b885-d015d8fca76e"
-					(reference "R42")
+					(reference "R47")
 					(unit 1)
 				)
@@
 		(in_pos_files yes)
 		(dnp no)
-		(property "Reference" "#PWR084"
+		(property "Reference" "#PWR0126"
 			(at 99.06 67.31 0)
 			(hide yes)
@@
 			(project "meko"
 				(path "/da54f10a-146b-4941-a9c7-55c7173bb101/122d9c1c-6abd-41a6-b885-d015d8fca76e"
-					(reference "#PWR084")
+					(reference "#PWR0126")
 					(unit 1)
 				)
@@
 		(in_pos_files yes)
 		(dnp no)
-		(property "Reference" "J5"
+		(property "Reference" "J8"
 			(at 130.81 52.07 0)
 			(show_name no)
@@
 			(project "meko"
 				(path "/da54f10a-146b-4941-a9c7-55c7173bb101/122d9c1c-6abd-41a6-b885-d015d8fca76e"
-					(reference "J5")
+					(reference "J8")
 					(unit 1)
 				)
@@
 		(in_pos_files yes)
 		(dnp no)
-		(property "Reference" "C37"
+		(property "Reference" "C120"
 			(at 99.568 76.708 0)
 			(show_name no)
@@
 			(project "meko"
 				(path "/da54f10a-146b-4941-a9c7-55c7173bb101/122d9c1c-6abd-41a6-b885-d015d8fca76e"
-					(reference "C37")
+					(reference "C120")
 					(unit 1)
 				)
@@
 		(in_pos_files yes)
 		(dnp yes)
-		(property "Reference" "C33"
+		(property "Reference" "C118"
 			(at 74.422 76.454 0)
 			(show_name no)
@@
 			(project "meko"
 				(path "/da54f10a-146b-4941-a9c7-55c7173bb101/122d9c1c-6abd-41a6-b885-d015d8fca76e"
-					(reference "C33")
+					(reference "C118")
 					(unit 1)
 				)
@@
 		(dnp no)
 		(fields_autoplaced yes)
-		(property "Reference" "#PWR073"
+		(property "Reference" "#PWR0129"
 			(at 144.78 90.17 0)
 			(hide yes)
@@
 			(project "meko"
 				(path "/da54f10a-146b-4941-a9c7-55c7173bb101/122d9c1c-6abd-41a6-b885-d015d8fca76e"
-					(reference "#PWR073")
+					(reference "#PWR0129")
 					(unit 1)
 				)
@@
 		(in_pos_files yes)
 		(dnp no)
-		(property "Reference" "#PWR085"
+		(property "Reference" "#PWR0127"
 			(at 97.79 72.39 0)
 			(hide yes)
@@
 			(project "meko"
 				(path "/da54f10a-146b-4941-a9c7-55c7173bb101/122d9c1c-6abd-41a6-b885-d015d8fca76e"
-					(reference "#PWR085")
+					(reference "#PWR0127")
 					(unit 1)
 				)
@@
 		(in_pos_files yes)
 		(dnp no)
-		(property "Reference" "C32"
+		(property "Reference" "C119"
 			(at 91.948 76.708 0)
 			(show_name no)
@@
 			(project "meko"
 				(path "/da54f10a-146b-4941-a9c7-55c7173bb101/122d9c1c-6abd-41a6-b885-d015d8fca76e"
-					(reference "C32")
+					(reference "C119")
 					(unit 1)
 				)

Commit message: added a bunch testpoints
Parts:
- added TP74: DISP_CLK, TestPoint:TestPoint_Pad_D1.0mm, symbol Connector:TestPoint
- added TP75: DISP_SI, TestPoint:TestPoint_Pad_D1.0mm, symbol Connector:TestPoint
- added TP76: DISP_CS, TestPoint:TestPoint_Pad_D1.0mm, symbol Connector:TestPoint
- added TP77: DISP_EN, TestPoint:TestPoint_Pad_D1.0mm, symbol Connector:TestPoint
Connections:
- net DISP: now also TP77.1
- net SCLK: now also TP74.1
- net SCS: now also TP76.1
- net SI: now also TP75.1

Commit message: removed testpoints on sd cards, since I can probe the pins there
Parts:
- renumbered TP74 to TP58, TP75 to TP59, TP76 to TP60, TP77 to TP61
Changed lines of the file:
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@@
 		(in_pos_files yes)
 		(dnp no)
-		(property "Reference" "#PWR0126"
+		(property "Reference" "#PWR0127"
 			(at 99.06 67.31 0)
 			(hide yes)
@@
 			(project "meko"
 				(path "/da54f10a-146b-4941-a9c7-55c7173bb101/122d9c1c-6abd-41a6-b885-d015d8fca76e"
-					(reference "#PWR0126")
+					(reference "#PWR0127")
 					(unit 1)
 				)
@@
 		(in_pos_files yes)
 		(dnp no)
-		(property "Reference" "TP75"
+		(property "Reference" "TP59"
 			(at 170.942 68.58 90)
 			(show_name no)
@@
 			(project "meko"
 				(path "/da54f10a-146b-4941-a9c7-55c7173bb101/122d9c1c-6abd-41a6-b885-d015d8fca76e"
-					(reference "TP75")
+					(reference "TP59")
 					(unit 1)
 				)
@@
 		(in_pos_files yes)
 		(dnp no)
-		(property "Reference" "TP76"
+		(property "Reference" "TP60"
 			(at 170.942 71.12 90)
 			(show_name no)
@@
 			(project "meko"
 				(path "/da54f10a-146b-4941-a9c7-55c7173bb101/122d9c1c-6abd-41a6-b885-d015d8fca76e"
-					(reference "TP76")
+					(reference "TP60")
 					(unit 1)
 				)
@@
 		(in_pos_files yes)
 		(dnp no)
-		(property "Reference" "TP77"
+		(property "Reference" "TP61"
 			(at 170.942 73.66 90)
 			(show_name no)
@@
 			(project "meko"
 				(path "/da54f10a-146b-4941-a9c7-55c7173bb101/122d9c1c-6abd-41a6-b885-d015d8fca76e"
-					(reference "TP77")
+					(reference "TP61")
 					(unit 1)
 				)
@@
 		(in_pos_files yes)
 		(dnp no)
-		(property "Reference" "#PWR0127"
+		(property "Reference" "#PWR0126"
 			(at 97.79 72.39 0)
 			(hide yes)
@@
 			(project "meko"
 				(path "/da54f10a-146b-4941-a9c7-55c7173bb101/122d9c1c-6abd-41a6-b885-d015d8fca76e"
-					(reference "#PWR0127")
+					(reference "#PWR0126")
 					(unit 1)
 				)
@@
 		(in_pos_files yes)
 		(dnp no)
-		(property "Reference" "TP74"
+		(property "Reference" "TP58"
 			(at 170.942 66.04 90)
 			(show_name no)
@@
 			(project "meko"
 				(path "/da54f10a-146b-4941-a9c7-55c7173bb101/122d9c1c-6abd-41a6-b885-d015d8fca76e"
-					(reference "TP74")
-					(unit 1)
-				)
+					(reference "TP58")
+					(unit 1)
+				)

Commit message: added capacitor to sama ddr vref pin
Parts:
- renumbered C118 to C120, C119 to C121, C120 to C122, R47 to R49
Changed lines of the file:
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@@
 		(dnp no)
 		(fields_autoplaced yes)
-		(property "Reference" "#PWR0128"
+		(property "Reference" "#PWR0130"
 			(at 105.41 90.17 0)
 			(hide yes)
@@
 			(project "meko"
 				(path "/da54f10a-146b-4941-a9c7-55c7173bb101/122d9c1c-6abd-41a6-b885-d015d8fca76e"
-					(reference "#PWR0128")
+					(reference "#PWR0130")
 					(unit 1)
 				)
@@
 		(in_pos_files yes)
 		(dnp no)
-		(property "Reference" "R47"
+		(property "Reference" "R49"
 			(at 83.82 76.454 0)
 			(show_name no)
@@
 			(project "meko"
 				(path "/da54f10a-146b-4941-a9c7-55c7173bb101/122d9c1c-6abd-41a6-b885-d015d8fca76e"
-					(reference "R47")
+					(reference "R49")
 					(unit 1)
 				)
@@
 		(in_pos_files yes)
 		(dnp no)
-		(property "Reference" "#PWR0127"
+		(property "Reference" "#PWR0129"
 			(at 99.06 67.31 0)
 			(hide yes)
@@
 			(project "meko"
 				(path "/da54f10a-146b-4941-a9c7-55c7173bb101/122d9c1c-6abd-41a6-b885-d015d8fca76e"
-					(reference "#PWR0127")
+					(reference "#PWR0129")
 					(unit 1)
 				)
@@
 		(in_pos_files yes)
 		(dnp no)
-		(property "Reference" "C120"
+		(property "Reference" "C122"
 			(at 99.568 76.708 0)
 			(show_name no)
@@
 			(project "meko"
 				(path "/da54f10a-146b-4941-a9c7-55c7173bb101/122d9c1c-6abd-41a6-b885-d015d8fca76e"
-					(reference "C120")
+					(reference "C122")
 					(unit 1)
 				)
@@
 		(in_pos_files yes)
 		(dnp yes)
-		(property "Reference" "C118"
+		(property "Reference" "C120"
 			(at 74.422 76.454 0)
 			(show_name no)
@@
 			(project "meko"
 				(path "/da54f10a-146b-4941-a9c7-55c7173bb101/122d9c1c-6abd-41a6-b885-d015d8fca76e"
-					(reference "C118")
+					(reference "C120")
 					(unit 1)
 				)
@@
 		(dnp no)
 		(fields_autoplaced yes)
-		(property "Reference" "#PWR0129"
+		(property "Reference" "#PWR0131"
 			(at 144.78 90.17 0)
 			(hide yes)
@@
 			(project "meko"
 				(path "/da54f10a-146b-4941-a9c7-55c7173bb101/122d9c1c-6abd-41a6-b885-d015d8fca76e"
-					(reference "#PWR0129")
+					(reference "#PWR0131")
 					(unit 1)
 				)
@@
 		(in_pos_files yes)
 		(dnp no)
-		(property "Reference" "#PWR0126"
+		(property "Reference" "#PWR0128"
 			(at 97.79 72.39 0)
 			(hide yes)
@@
 			(project "meko"
 				(path "/da54f10a-146b-4941-a9c7-55c7173bb101/122d9c1c-6abd-41a6-b885-d015d8fca76e"
-					(reference "#PWR0126")
+					(reference "#PWR0128")
 					(unit 1)
 				)
@@
 		(in_pos_files yes)
 		(dnp no)
-		(property "Reference" "C119"
+		(property "Reference" "C121"
 			(at 91.948 76.708 0)
 			(show_name no)
@@
 			(project "meko"
 				(path "/da54f10a-146b-4941-a9c7-55c7173bb101/122d9c1c-6abd-41a6-b885-d015d8fca76e"
-					(reference "C119")
-					(unit 1)
-				)
+					(reference "C121")
+					(unit 1)
+				)

Commit message: didn't save last time :sob:
Parts:
- renumbered C120 to C121, C121 to C122, C122 to C123
Changed lines of the file:
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@@
 		(dnp no)
 		(fields_autoplaced yes)
-		(property "Reference" "#PWR0130"
+		(property "Reference" "#PWR0131"
 			(at 105.41 90.17 0)
 			(hide yes)
@@
 			(project "meko"
 				(path "/da54f10a-146b-4941-a9c7-55c7173bb101/122d9c1c-6abd-41a6-b885-d015d8fca76e"
-					(reference "#PWR0130")
+					(reference "#PWR0131")
 					(unit 1)
 				)
@@
 		(in_pos_files yes)
 		(dnp no)
-		(property "Reference" "#PWR0129"
+		(property "Reference" "#PWR0130"
 			(at 99.06 67.31 0)
 			(hide yes)
@@
 			(project "meko"
 				(path "/da54f10a-146b-4941-a9c7-55c7173bb101/122d9c1c-6abd-41a6-b885-d015d8fca76e"
-					(reference "#PWR0129")
+					(reference "#PWR0130")
 					(unit 1)
 				)
@@
 		(in_pos_files yes)
 		(dnp no)
-		(property "Reference" "C122"
+		(property "Reference" "C123"
 			(at 99.568 76.708 0)
 			(show_name no)
@@
 			(project "meko"
 				(path "/da54f10a-146b-4941-a9c7-55c7173bb101/122d9c1c-6abd-41a6-b885-d015d8fca76e"
-					(reference "C122")
+					(reference "C123")
 					(unit 1)
 				)
@@
 		(in_pos_files yes)
 		(dnp yes)
-		(property "Reference" "C120"
+		(property "Reference" "C121"
 			(at 74.422 76.454 0)
 			(show_name no)
@@
 			(project "meko"
 				(path "/da54f10a-146b-4941-a9c7-55c7173bb101/122d9c1c-6abd-41a6-b885-d015d8fca76e"
-					(reference "C120")
+					(reference "C121")
 					(unit 1)
 				)
@@
 		(dnp no)
 		(fields_autoplaced yes)
-		(property "Reference" "#PWR0131"
+		(property "Reference" "#PWR0132"
 			(at 144.78 90.17 0)
 			(hide yes)
@@
 			(project "meko"
 				(path "/da54f10a-146b-4941-a9c7-55c7173bb101/122d9c1c-6abd-41a6-b885-d015d8fca76e"
-					(reference "#PWR0131")
+					(reference "#PWR0132")
 					(unit 1)
 				)
@@
 		(in_pos_files yes)
 		(dnp no)
-		(property "Reference" "#PWR0128"
+		(property "Reference" "#PWR0129"
 			(at 97.79 72.39 0)
 			(hide yes)
@@
 			(project "meko"
 				(path "/da54f10a-146b-4941-a9c7-55c7173bb101/122d9c1c-6abd-41a6-b885-d015d8fca76e"
-					(reference "#PWR0128")
+					(reference "#PWR0129")
 					(unit 1)
 				)
@@
 		(in_pos_files yes)
 		(dnp no)
-		(property "Reference" "C121"
+		(property "Reference" "C122"
 			(at 91.948 76.708 0)
 			(show_name no)
@@
 			(project "meko"
 				(path "/da54f10a-146b-4941-a9c7-55c7173bb101/122d9c1c-6abd-41a6-b885-d015d8fca76e"
-					(reference "C121")
-					(unit 1)
-				)
+					(reference "C122")
+					(unit 1)
+				)
