File: hardware/pcb/display.kicad_sch (KiCad schematic)
At the start: 9 parts, among them J8 503480-1000

Commit message: added pullups for jtag
Parts:
- renumbered R49 to R55
Changed lines of the file:
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@@
 		(dnp no)
 		(fields_autoplaced yes)
-		(property "Reference" "#PWR0131"
+		(property "Reference" "#PWR0132"
 			(at 105.41 90.17 0)
 			(hide yes)
@@
 			(project "meko"
 				(path "/da54f10a-146b-4941-a9c7-55c7173bb101/122d9c1c-6abd-41a6-b885-d015d8fca76e"
-					(reference "#PWR0131")
+					(reference "#PWR0132")
 					(unit 1)
 				)
@@
 		(in_pos_files yes)
 		(dnp no)
-		(property "Reference" "R49"
+		(property "Reference" "R55"
 			(at 83.82 76.454 0)
 			(show_name no)
@@
 			(project "meko"
 				(path "/da54f10a-146b-4941-a9c7-55c7173bb101/122d9c1c-6abd-41a6-b885-d015d8fca76e"
-					(reference "R49")
+					(reference "R55")
 					(unit 1)
 				)
@@
 		(dnp no)
 		(fields_autoplaced yes)
-		(property "Reference" "#PWR0132"
+		(property "Reference" "#PWR0133"
 			(at 144.78 90.17 0)
 			(hide yes)
@@
 			(project "meko"
 				(path "/da54f10a-146b-4941-a9c7-55c7173bb101/122d9c1c-6abd-41a6-b885-d015d8fca76e"
-					(reference "#PWR0132")
+					(reference "#PWR0133")
 					(unit 1)
 				)
@@
 		(in_pos_files yes)
 		(dnp no)
-		(property "Reference" "#PWR0129"
+		(property "Reference" "#PWR0131"
 			(at 97.79 72.39 0)
 			(hide yes)
@@
 			(project "meko"
 				(path "/da54f10a-146b-4941-a9c7-55c7173bb101/122d9c1c-6abd-41a6-b885-d015d8fca76e"
-					(reference "#PWR0129")
-					(unit 1)
-				)
+					(reference "#PWR0131")
+					(unit 1)
+				)

Commit message: moved some caps to 0201
Parts:
- C121: footprint Capacitor_SMD:C_0402_1005Metric -> Capacitor_SMD:C_0201_0603Metric
Changed lines of the file:
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@@
 		(dnp no)
 		(fields_autoplaced yes)
-		(property "Reference" "#PWR0132"
+		(property "Reference" "#PWR0133"
 			(at 105.41 90.17 0)
 			(hide yes)
@@
 			(project "meko"
 				(path "/da54f10a-146b-4941-a9c7-55c7173bb101/122d9c1c-6abd-41a6-b885-d015d8fca76e"
-					(reference "#PWR0132")
+					(reference "#PWR0133")
 					(unit 1)
 				)
@@
 		(in_pos_files yes)
 		(dnp no)
-		(property "Reference" "#PWR0130"
+		(property "Reference" "#PWR0131"
 			(at 99.06 67.31 0)
 			(hide yes)
@@
 			(project "meko"
 				(path "/da54f10a-146b-4941-a9c7-55c7173bb101/122d9c1c-6abd-41a6-b885-d015d8fca76e"
-					(reference "#PWR0130")
+					(reference "#PWR0131")
 					(unit 1)
 				)
@@
 			)
 		)
-		(property "Footprint" "Capacitor_SMD:C_0402_1005Metric"
+		(property "Footprint" "Capacitor_SMD:C_0201_0603Metric"
 			(at 76.2 77.47 0)
 			(hide yes)
@@
 		(dnp no)
 		(fields_autoplaced yes)
-		(property "Reference" "#PWR0133"
+		(property "Reference" "#PWR0134"
 			(at 144.78 90.17 0)
 			(hide yes)
@@
 			(project "meko"
 				(path "/da54f10a-146b-4941-a9c7-55c7173bb101/122d9c1c-6abd-41a6-b885-d015d8fca76e"
-					(reference "#PWR0133")
+					(reference "#PWR0134")
 					(unit 1)
 				)
@@
 		(in_pos_files yes)
 		(dnp no)
-		(property "Reference" "#PWR0131"
+		(property "Reference" "#PWR0132"
 			(at 97.79 72.39 0)
 			(hide yes)
@@
 			(project "meko"
 				(path "/da54f10a-146b-4941-a9c7-55c7173bb101/122d9c1c-6abd-41a6-b885-d015d8fca76e"
-					(reference "#PWR0131")
-					(unit 1)
-				)
+					(reference "#PWR0132")
+					(unit 1)
+				)

Commit message: added disaplay datasheet to schematic
Other:
- note added: "Display Datasheet"
Changed lines of the file:
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@@
+		)
+	)
+	(text "Display Datasheet"
+		(exclude_from_sim no)
+		(at 114.3 42.418 0)
+		(effects
+			(font
+				(size 1.27 1.27)
+				(thickness 0.254)
+				(bold yes)
+			)
+			(href "https://mm.digikey.com/Volume0/opasdata/d220001/medias/docus/6488/425_PdfFile792090.pdf")
 		)
 	)

Commit message: added lcsc part nr to display conn
Parts:
- J8: LCSC (none) -> C127355
Changed lines of the file:
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@@
+			)
+		)
+		(property "LCSC" "C127355"
+			(at 130.81 69.85 0)
+			(hide yes)
+			(show_name no)
+			(do_not_autoplace no)
+			(effects
+				(font
+					(size 1.27 1.27)
+				)
 			)
 		)

Commit message: cleanup, tespoints, passives
Parts:
- removed C123: 1u, Capacitor_SMD:C_0402_1005Metric, symbol Device:C_Small
Other:
- moved on the sheet: C121, C122, R55
