File: hardware/pcb/display.kicad_sch (KiCad schematic)
At the start: 8 parts, among them J8 503480-1000

Commit message: found issue with PMIC wake-up pullup, other small fixes
Other:
- note added: "Link: Display Datasheet"
- note removed: "Display Datasheet"
Changed lines of the file:
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@@
 		)
 	)
-	(text "Display Datasheet"
+	(text "Link: Display Datasheet"
 		(exclude_from_sim no)
 		(at 114.3 42.418 0)
