File: hardware/pcb/buttons.kicad_sch (KiCad schematic)
At the start: 0 parts

Commit message: added buttons
Parts:
- added C26: 100n, symbol Device:C_Small
- added R41: 10k, symbol Device:R_Small
- added SW1, SW2, SW3, SW4, SW5: SW_Push, symbol Switch:SW_Push
Connections:
- new net: R41.1, SW1.2
- new net GND: C26.1, SW1.1, SW2.1, SW3.1, SW4.1, SW5.1
- new net PWR: C26.2, R41.2
- new net SIDE_L: SW4.2
- new net SIDE_R: SW5.2
- new net VOL+: SW2.2
- new net VOL-: SW3.2

Commit message: looking over stuff, added caps
Parts:
- C26: footprint (none) -> Capacitor_SMD:C_0402_1005Metric
- R41: footprint (none) -> Resistor_SMD:R_0402_1005Metric
Changed lines of the file:
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@@
 			)
 		)
-		(property "Footprint" ""
+		(property "Footprint" "Resistor_SMD:R_0402_1005Metric"
 			(at 99.06 52.07 0)
 			(hide yes)
@@
 			)
 		)
-		(property "Footprint" ""
+		(property "Footprint" "Capacitor_SMD:C_0402_1005Metric"
 			(at 95.25 55.88 0)
 			(hide yes)

Commit message: added buttons
Parts:
- removed SW1, SW2, SW3, SW4, SW5: SW_Push, symbol Switch:SW_Push
- added SW10, SW6, SW7, SW8, SW9: SW_Push, Button_Switch_SMD:SW_Push_1P1T-MP_NO_Horizontal_Alps_SKRTLAE010, symbol Switch:SW_Push
Connections:
- net GND: now also SW10.1, SW6.1, SW7.1, SW8.1, SW9.1
- net SIDE_L: now also SW9.2
- net SIDE_R: now also SW10.2
- net VOL+: now also SW7.2
- net VOL-: now also SW8.2
- net at R41.1: now also SW6.2

Commit message: started cleaning up schematic
Other:
- company: (none) -> Gensis
- title: (none) -> Buttons
Changed lines of the file:
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@@
 	(generator_version "10.0")
 	(paper "A5")
+	(title_block
+		(title "Buttons")
+		(rev "v1.0.0")
+		(company "Gensis")
+	)
 	(junction
 		(at 106.68 52.07)

Commit message: mainboard: reannotated schematic
Parts:
- renumbered C26 to C123, R41 to R48, SW6 to SW1, SW7 to SW2, SW8 to SW3, SW9 to SW4, SW10 to SW5
Changed lines of the file:
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@@
 		(in_pos_files yes)
 		(dnp no)
-		(property "Reference" "R41"
+		(property "Reference" "R48"
 			(at 97.028 51.054 90)
 			(show_name no)
@@
 			(project "meko"
 				(path "/da54f10a-146b-4941-a9c7-55c7173bb101/e40fc879-1a0f-4948-9e1c-6c4ee1733e71"
-					(reference "R41")
+					(reference "R48")
 					(unit 1)
 				)
@@
 		(in_pos_files yes)
 		(dnp no)
-		(property "Reference" "SW9"
+		(property "Reference" "SW4"
 			(at 88.646 72.644 0)
 			(show_name no)
@@
 			(project "meko"
 				(path "/da54f10a-146b-4941-a9c7-55c7173bb101/e40fc879-1a0f-4948-9e1c-6c4ee1733e71"
-					(reference "SW9")
+					(reference "SW4")
 					(unit 1)
 				)
@@
 		(in_pos_files yes)
 		(dnp no)
-		(property "Reference" "SW6"
+		(property "Reference" "SW1"
 			(at 88.646 49.784 0)
 			(show_name no)
@@
 			(project "meko"
 				(path "/da54f10a-146b-4941-a9c7-55c7173bb101/e40fc879-1a0f-4948-9e1c-6c4ee1733e71"
-					(reference "SW6")
+					(reference "SW1")
 					(unit 1)
 				)
@@
 		(in_pos_files yes)
 		(dnp no)
-		(property "Reference" "SW7"
+		(property "Reference" "SW2"
 			(at 88.646 59.944 0)
 			(show_name no)
@@
 			(project "meko"
 				(path "/da54f10a-146b-4941-a9c7-55c7173bb101/e40fc879-1a0f-4948-9e1c-6c4ee1733e71"
-					(reference "SW7")
+					(reference "SW2")
 					(unit 1)
 				)
@@
 		(in_pos_files yes)
 		(dnp no)
-		(property "Reference" "SW10"
+		(property "Reference" "SW5"
 			(at 88.646 78.994 0)
 			(show_name no)
@@
 			(project "meko"
 				(path "/da54f10a-146b-4941-a9c7-55c7173bb101/e40fc879-1a0f-4948-9e1c-6c4ee1733e71"
-					(reference "SW10")
+					(reference "SW5")
 					(unit 1)
 				)
@@
 		(in_pos_files yes)
 		(dnp no)
-		(property "Reference" "C26"
+		(property "Reference" "C123"
 			(at 93.98 57.404 90)
 			(show_name no)
@@
 			(project "meko"
 				(path "/da54f10a-146b-4941-a9c7-55c7173bb101/e40fc879-1a0f-4948-9e1c-6c4ee1733e71"
-					(reference "C26")
+					(reference "C123")
 					(unit 1)
 				)
@@
 		(in_pos_files yes)
 		(dnp no)
-		(property "Reference" "#PWR036"
+		(property "Reference" "#PWR0137"
 			(at 82.55 91.44 0)
 			(hide yes)
@@
 			(project "meko"
 				(path "/da54f10a-146b-4941-a9c7-55c7173bb101/e40fc879-1a0f-4948-9e1c-6c4ee1733e71"
-					(reference "#PWR036")
+					(reference "#PWR0137")
 					(unit 1)
 				)
@@
 		(in_pos_files yes)
 		(dnp no)
-		(property "Reference" "SW8"
+		(property "Reference" "SW3"
 			(at 88.646 66.294 0)
 			(show_name no)
@@
 			(project "meko"
 				(path "/da54f10a-146b-4941-a9c7-55c7173bb101/e40fc879-1a0f-4948-9e1c-6c4ee1733e71"
-					(reference "SW8")
+					(reference "SW3")
 					(unit 1)
 				)

Commit message: added capacitor to sama ddr vref pin
Parts:
- renumbered C123 to C125, R48 to R50
Changed lines of the file:
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@@
 		(in_pos_files yes)
 		(dnp no)
-		(property "Reference" "R48"
+		(property "Reference" "R50"
 			(at 97.028 51.054 90)
 			(show_name no)
@@
 			(project "meko"
 				(path "/da54f10a-146b-4941-a9c7-55c7173bb101/e40fc879-1a0f-4948-9e1c-6c4ee1733e71"
-					(reference "R48")
+					(reference "R50")
 					(unit 1)
 				)
@@
 		(in_pos_files yes)
 		(dnp no)
-		(property "Reference" "C123"
+		(property "Reference" "C125"
 			(at 93.98 57.404 90)
 			(show_name no)
@@
 			(project "meko"
 				(path "/da54f10a-146b-4941-a9c7-55c7173bb101/e40fc879-1a0f-4948-9e1c-6c4ee1733e71"
-					(reference "C123")
+					(reference "C125")
 					(unit 1)
 				)
@@
 		(in_pos_files yes)
 		(dnp no)
-		(property "Reference" "#PWR0137"
+		(property "Reference" "#PWR0139"
 			(at 82.55 91.44 0)
 			(hide yes)
@@
 			(project "meko"
 				(path "/da54f10a-146b-4941-a9c7-55c7173bb101/e40fc879-1a0f-4948-9e1c-6c4ee1733e71"
-					(reference "#PWR0137")
+					(reference "#PWR0139")
 					(unit 1)
 				)

Commit message: didn't save last time :sob:
Parts:
- renumbered C125 to C126
Changed lines of the file:
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@@
 		(in_pos_files yes)
 		(dnp no)
-		(property "Reference" "C125"
+		(property "Reference" "C126"
 			(at 93.98 57.404 90)
 			(show_name no)
@@
 			(project "meko"
 				(path "/da54f10a-146b-4941-a9c7-55c7173bb101/e40fc879-1a0f-4948-9e1c-6c4ee1733e71"
-					(reference "C125")
+					(reference "C126")
 					(unit 1)
 				)
@@
 		(in_pos_files yes)
 		(dnp no)
-		(property "Reference" "#PWR0139"
+		(property "Reference" "#PWR0140"
 			(at 82.55 91.44 0)
 			(hide yes)
@@
 			(project "meko"
 				(path "/da54f10a-146b-4941-a9c7-55c7173bb101/e40fc879-1a0f-4948-9e1c-6c4ee1733e71"
-					(reference "#PWR0139")
+					(reference "#PWR0140")
 					(unit 1)
 				)

Commit message: added pullups for jtag
Parts:
- renumbered R50 to R56
Changed lines of the file:
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@@
 		(in_pos_files yes)
 		(dnp no)
-		(property "Reference" "R50"
+		(property "Reference" "R56"
 			(at 97.028 51.054 90)
 			(show_name no)
@@
 			(project "meko"
 				(path "/da54f10a-146b-4941-a9c7-55c7173bb101/e40fc879-1a0f-4948-9e1c-6c4ee1733e71"
-					(reference "R50")
+					(reference "R56")
 					(unit 1)
 				)
@@
 		(in_pos_files yes)
 		(dnp no)
-		(property "Reference" "#PWR0140"
+		(property "Reference" "#PWR0141"
 			(at 82.55 91.44 0)
 			(hide yes)
@@
 			(project "meko"
 				(path "/da54f10a-146b-4941-a9c7-55c7173bb101/e40fc879-1a0f-4948-9e1c-6c4ee1733e71"
-					(reference "#PWR0140")
+					(reference "#PWR0141")
 					(unit 1)
 				)
