File: hardware/pcb/power.kicad_sch (KiCad schematic)
At the start: 41 parts, among them IC1 MCP16502AB, U3 TPS7A2033PDBV, U4 BQ25640, U5 MAX17260

Commit message: assigned missing footprints
Parts:
- JP3: footprint (none) -> Jumper:SolderJumper-2_P1.3mm_Open_RoundedPad1.0x1.5mm
Changed lines of the file:
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@@
 			)
 		)
-		(property "Footprint" ""
+		(property "Footprint" "Jumper:SolderJumper-2_P1.3mm_Open_RoundedPad1.0x1.5mm"
 			(at 104.14 134.62 0)
 			(hide yes)

Commit message: added a bunch testpoints
Parts:
- added TP10, TP29: +3V3, TestPoint:TestPoint_Pad_D1.0mm, symbol Connector:TestPoint
- added TP11: +1V35, TestPoint:TestPoint_Pad_D1.0mm, symbol Connector:TestPoint
- added TP12: +1V15_CORE, TestPoint:TestPoint_Pad_D1.0mm, symbol Connector:TestPoint
- added TP13: +1V15_CPU, TestPoint:TestPoint_Pad_D1.0mm, symbol Connector:TestPoint
- added TP15: +1V8_BATT, TestPoint:TestPoint_Pad_D1.0mm, symbol Connector:TestPoint
- added TP16: +1V8, TestPoint:TestPoint_Pad_D1.0mm, symbol Connector:TestPoint
- added TP22: F_~{INT}, TestPoint:TestPoint_Pad_D1.0mm, symbol Connector:TestPoint
- added TP23: PM_~{INT}, TestPoint:TestPoint_Pad_D1.0mm, symbol Connector:TestPoint
- added TP24: PM_~{RST}, TestPoint:TestPoint_Pad_D1.0mm, symbol Connector:TestPoint
- added TP25: ~{WKUP}, TestPoint:TestPoint_Pad_D1.0mm, symbol Connector:TestPoint
- added TP26: PWRHLD, TestPoint:TestPoint_Pad_D1.0mm, symbol Connector:TestPoint
- added TP27: LPM, TestPoint:TestPoint_Pad_D1.0mm, symbol Connector:TestPoint
- added TP28: HPM, TestPoint:TestPoint_Pad_D1.0mm, symbol Connector:TestPoint
Connections:
- net +1V15_CORE: now also TP12.1
- net +1V15_CPU: now also TP13.1
- net +1V35_DDR: now also TP11.1
- net +1V8: now also TP16.1
- net +1V8_BATT_CPU: now also TP15.1
- net +3V3: now also TP10.1
- net +3V3_AVDD: now also TP29.1
- net FUEL_~{INT}: now also TP22.1
- net HPM: now also TP28.1
- net LPM: now also TP27.1
- net PWRHLD: now also TP26.1
- net ~{INT}: now also TP23.1
- net ~{RST}: now also TP24.1
- net ~{WKUP}: now also TP25.1
Other:
- moved on the sheet: C87, C89, C90, U3

Commit message: removed testpoints on sd cards, since I can probe the pins there
Parts:
- renumbered C95 to C100, C97 to C101, C100 to C102, C105 to C103, C89 to C104, C90 to C105, C102 to C87, C99 to C88, C92 to C89, C94 to C90, C87 to C91, C88 to C92, C96 to C94, C98 to C95, C101 to C96, C103 to C97, C104 to C98, C91 to C99, L2 to L1, L1 to L2, R18 to R15, R21 to R16, R19 to R17, R22 to R18, R20 to R19, R15 to R20, R16 to R21, R17 to R22, TP22 to TP12, TP23 to TP13, TP24 to TP14, TP25 to TP15, TP26 to TP16, TP27 to TP17, TP28 to TP18, TP10 to TP19, TP11 to TP20, TP12 to TP21, TP13 to TP22, TP15 to TP23, TP16 to TP24, TP29 to TP25, U5 to U3, U3 to U5

Commit message: added capacitor to sama ddr vref pin
Parts:
- renumbered C98 to C100, C99 to C101, C100 to C102, C101 to C103, C102 to C104, C103 to C105, C104 to C106, C105 to C107, C85 to C87, C86 to C88, C87 to C89, C88 to C90, C89 to C91, C90 to C92, C91 to C93, C92 to C94, C93 to C95, C94 to C96, C95 to C97, C96 to C98, C97 to C99, R15 to R17, R16 to R18, R17 to R19, R18 to R20, R19 to R21, R20 to R22, R21 to R23, R22 to R24

Commit message: didn't save last time :sob:
Parts:
- renumbered C99 to C100, C100 to C101, C101 to C102, C102 to C103, C103 to C104, C104 to C105, C105 to C106, C106 to C107, C107 to C108, C87 to C88, C88 to C89, C89 to C90, C90 to C91, C91 to C92, C92 to C93, C93 to C94, C94 to C95, C95 to C96, C96 to C97, C97 to C98, C98 to C99

Commit message: wrote journal
Parts:
- added R51, R52: 1k, Resistor_SMD:R_0402_1005Metric, symbol Device:R_Small
- added R53: 10k, Resistor_SMD:R_0402_1005Metric, symbol Device:R_Small
Connections:
- net GND: now also R53.1; no longer IC1.18 (SELVL1)
- net HPM: now also R52.2; no longer IC1.23 (HPM)
- net PWRHLD: now also R51.2; no longer IC1.8 (PWRHLD)
- new net: IC1.23 (HPM), R52.1
- new net: IC1.18 (SELVL1), R53.2
- new net: IC1.8 (PWRHLD), R51.1

Commit message: added pullups for jtag
Parts:
- renumbered C104 to C100, C98 to C101, C91 to C102, C105 to C103, C99 to C104, C90 to C105, C100 to C106, C101 to C107, C106 to C108, C94 to C90, C95 to C91, C107 to C92, C108 to C93, C102 to C94, C92 to C95, C93 to C97, C103 to C98, C97 to C99, L2 to L1, L1 to L2, R22 to R20, R23 to R21, R24 to R22, R17 to R23, R19 to R24, R21 to R25, R51 to R26, R52 to R27, R18 to R28, R20 to R29, R53 to R30, TP25 to TP12, TP19 to TP13, TP20 to TP14, TP21 to TP15, TP22 to TP16, TP12 to TP17, TP23 to TP18, TP24 to TP19, TP13 to TP20, TP14 to TP21, TP15 to TP22, TP16 to TP23, TP17 to TP24, TP18 to TP25, U5 to U3, U3 to U5

Commit message: moved some caps to 0201
Parts:
- C102, C105, C95: footprint Capacitor_SMD:C_0402_1005Metric -> Capacitor_SMD:C_0201_0603Metric
Changed lines of the file:
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@@
 			)
 		)
-		(property "Footprint" "Capacitor_SMD:C_0402_1005Metric"
+		(property "Footprint" "Capacitor_SMD:C_0201_0603Metric"
 			(at 132.08 166.37 0)
 			(hide yes)
@@
 		(pin "19"
 		)
-		(pin ""
+		(pin "7"
 		)
 		(instances
@@
 			)
 		)
-		(property "Footprint" "Capacitor_SMD:C_0402_1005Metric"
+		(property "Footprint" "Capacitor_SMD:C_0201_0603Metric"
 			(at 135.89 97.79 0)
 			(hide yes)
@@
 			)
 		)
-		(property "Footprint" "Capacitor_SMD:C_0402_1005Metric"
+		(property "Footprint" "Capacitor_SMD:C_0201_0603Metric"
 			(at 102.87 190.5 0)
 			(hide yes)
