File: hardware/pcb/sd.kicad_sch (KiCad schematic)
At the start: 31 parts, among them J6 Micro_SD_Card_Det1, J7 Micro_SD_Card_Det1

Commit message: removed testpoints on sd cards, since I can probe the pins there
Parts:
- removed TP60: BOOT_DAT2, TestPoint:TestPoint_Pad_D1.0mm, symbol Connector:TestPoint
- removed TP61: BOOT_DAT3, TestPoint:TestPoint_Pad_D1.0mm, symbol Connector:TestPoint
- removed TP62: BOOT_DAT0, TestPoint:TestPoint_Pad_D1.0mm, symbol Connector:TestPoint
- removed TP63: BOOT_DAT1, TestPoint:TestPoint_Pad_D1.0mm, symbol Connector:TestPoint
- removed TP64: BOOT_CMD, TestPoint:TestPoint_Pad_D1.0mm, symbol Connector:TestPoint
- removed TP65: BOOT_CK, TestPoint:TestPoint_Pad_D1.0mm, symbol Connector:TestPoint
- removed TP66: BOOT_CD, TestPoint:TestPoint_Pad_D1.0mm, symbol Connector:TestPoint
- removed TP67: EXT_DAT2, TestPoint:TestPoint_Pad_D1.0mm, symbol Connector:TestPoint
- removed TP68: EXT_DAT3, TestPoint:TestPoint_Pad_D1.0mm, symbol Connector:TestPoint
- removed TP69: EXT_CMD, TestPoint:TestPoint_Pad_D1.0mm, symbol Connector:TestPoint
- removed TP70: EXT_CK, TestPoint:TestPoint_Pad_D1.0mm, symbol Connector:TestPoint
- removed TP71: EXT_DAT0, TestPoint:TestPoint_Pad_D1.0mm, symbol Connector:TestPoint
- removed TP72: EXT_DAT1, TestPoint:TestPoint_Pad_D1.0mm, symbol Connector:TestPoint
- removed TP73: EXT_CD, TestPoint:TestPoint_Pad_D1.0mm, symbol Connector:TestPoint
- renumbered R41 to R36, R36 to R37, R42 to R38, R37 to R39, R43 to R40, R38 to R41, R44 to R42, R39 to R43, R45 to R44, R40 to R45

Commit message: added capacitor to sama ddr vref pin
Parts:
- renumbered C115 to C117, C116 to C118, C117 to C119, R35 to R37, R36 to R38, R37 to R39, R38 to R40, R39 to R41, R40 to R42, R41 to R43, R42 to R44, R43 to R45, R44 to R46, R45 to R47, R46 to R48
Changed lines of the file:
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@@
 		(in_pos_files yes)
 		(dnp no)
-		(property "Reference" "R43"
+		(property "Reference" "R45"
 			(at 86.868 36.195 0)
 			(show_name no)
@@
 			(project "meko"
 				(path "/da54f10a-146b-4941-a9c7-55c7173bb101/45aa24d2-e0af-4ebb-a68a-61b6a12c0eec"
-					(reference "R43")
+					(reference "R45")
 					(unit 1)
 				)
@@
 		(in_pos_files yes)
 		(dnp no)
-		(property "Reference" "R35"
+		(property "Reference" "R37"
 			(at 61.468 36.195 0)
 			(show_name no)
@@
 			(project "meko"
 				(path "/da54f10a-146b-4941-a9c7-55c7173bb101/45aa24d2-e0af-4ebb-a68a-61b6a12c0eec"
-					(reference "R35")
+					(reference "R37")
 					(unit 1)
 				)
@@
 		(in_pos_files yes)
 		(dnp no)
-		(property "Reference" "#PWR0116"
+		(property "Reference" "#PWR0118"
 			(at 102.87 55.88 0)
 			(hide yes)
@@
 			(project "meko"
 				(path "/da54f10a-146b-4941-a9c7-55c7173bb101/45aa24d2-e0af-4ebb-a68a-61b6a12c0eec"
-					(reference "#PWR0116")
+					(reference "#PWR0118")
 					(unit 1)
 				)
@@
 		(in_pos_files yes)
 		(dnp no)
-		(property "Reference" "C116"
+		(property "Reference" "C118"
 			(at 155.448 123.444 0)
 			(show_name no)
@@
 			(project "meko"
 				(path "/da54f10a-146b-4941-a9c7-55c7173bb101/45aa24d2-e0af-4ebb-a68a-61b6a12c0eec"
-					(reference "C116")
+					(reference "C118")
 					(unit 1)
 				)
@@
 		(in_pos_files yes)
 		(dnp no)
-		(property "Reference" "R36"
+		(property "Reference" "R38"
 			(at 61.468 104.775 0)
 			(show_name no)
@@
 			(project "meko"
 				(path "/da54f10a-146b-4941-a9c7-55c7173bb101/45aa24d2-e0af-4ebb-a68a-61b6a12c0eec"
-					(reference "R36")
+					(reference "R38")
 					(unit 1)
 				)
@@
 		(in_pos_files yes)
 		(dnp no)
-		(property "Reference" "#PWR0125"
+		(property "Reference" "#PWR0127"
 			(at 153.67 134.62 0)
 			(hide yes)
@@
 			(project "meko"
 				(path "/da54f10a-146b-4941-a9c7-55c7173bb101/45aa24d2-e0af-4ebb-a68a-61b6a12c0eec"
-					(reference "#PWR0125")
+					(reference "#PWR0127")
 					(unit 1)
 				)
@@
 		(in_pos_files yes)
 		(dnp no)
-		(property "Reference" "R42"
+		(property "Reference" "R44"
 			(at 80.518 104.775 0)
 			(show_name no)
@@
 			(project "meko"
 				(path "/da54f10a-146b-4941-a9c7-55c7173bb101/45aa24d2-e0af-4ebb-a68a-61b6a12c0eec"
-					(reference "R42")
+					(reference "R44")
 					(unit 1)
 				)
@@
 		(in_pos_files yes)
 		(dnp no)
-		(property "Reference" "#PWR0114"
+		(property "Reference" "#PWR0116"
 			(at 58.42 34.29 0)
 			(hide yes)
@@
 			(project "meko"
 				(path "/da54f10a-146b-4941-a9c7-55c7173bb101/45aa24d2-e0af-4ebb-a68a-61b6a12c0eec"
-					(reference "#PWR0114")
+					(reference "#PWR0116")
 					(unit 1)
 				)
@@
 		(in_pos_files yes)
 		(dnp no)
-		(property "Reference" "R44"
+		(property "Reference" "R46"
 			(at 86.868 104.775 0)
 			(show_name no)
@@
 			(project "meko"
 				(path "/da54f10a-146b-4941-a9c7-55c7173bb101/45aa24d2-e0af-4ebb-a68a-61b6a12c0eec"
-					(reference "R44")
+					(reference "R46")
 					(unit 1)
 				)
@@
 		(in_pos_files yes)
 		(dnp no)
-		(property "Reference" "R45"
+		(property "Reference" "R47"
 			(at 93.218 36.195 0)
 			(show_name no)
@@
 			(project "meko"
 				(path "/da54f10a-146b-4941-a9c7-55c7173bb101/45aa24d2-e0af-4ebb-a68a-61b6a12c0eec"
-					(reference "R45")
+					(reference "R47")
 					(unit 1)
 				)
@@
 		(in_pos_files yes)
 		(dnp no)
-		(property "Reference" "R38"
+		(property "Reference" "R40"
 			(at 67.818 104.775 0)
 			(show_name no)
@@
 			(project "meko"
 				(path "/da54f10a-146b-4941-a9c7-55c7173bb101/45aa24d2-e0af-4ebb-a68a-61b6a12c0eec"
-					(reference "R38")
+					(reference "R40")
 					(unit 1)
 				)
@@
 		(in_pos_files yes)
 		(dnp no)
-		(property "Reference" "R40"
+		(property "Reference" "R42"
 			(at 74.168 104.775 0)
 			(show_name no)
@@
 			(project "meko"
 				(path "/da54f10a-146b-4941-a9c7-55c7173bb101/45aa24d2-e0af-4ebb-a68a-61b6a12c0eec"
-					(reference "R40")
+					(reference "R42")
 					(unit 1)
 				)
@@
 		(in_pos_files yes)
 		(dnp no)
-		(property "Reference" "C115"
+		(property "Reference" "C117"
 			(at 155.448 54.864 0)
 			(show_name no)
@@
 			(project "meko"
 				(path "/da54f10a-146b-4941-a9c7-55c7173bb101/45aa24d2-e0af-4ebb-a68a-61b6a12c0eec"
-					(reference "C115")
+					(reference "C117")
 					(unit 1)
 				)
@@
 		(in_pos_files yes)
 		(dnp no)
-		(property "Reference" "#PWR0118"
+		(property "Reference" "#PWR0120"
 			(at 102.87 124.46 0)
 			(hide yes)
@@
 			(project "meko"
 				(path "/da54f10a-146b-4941-a9c7-55c7173bb101/45aa24d2-e0af-4ebb-a68a-61b6a12c0eec"
-					(reference "#PWR0118")
+					(reference "#PWR0120")
 					(unit 1)
 				)
@@
 		(in_pos_files yes)
 		(dnp no)
-		(property "Reference" "#PWR0117"
+		(property "Reference" "#PWR0119"
 			(at 92.71 60.96 0)
 			(hide yes)
@@
 			(project "meko"
 				(path "/da54f10a-146b-4941-a9c7-55c7173bb101/45aa24d2-e0af-4ebb-a68a-61b6a12c0eec"
-					(reference "#PWR0117")
+					(reference "#PWR0119")
 					(unit 1)
 				)
@@
 		(in_pos_files yes)
 		(dnp no)
-		(property "Reference" "#PWR0124"
+		(property "Reference" "#PWR0126"
 			(at 153.67 124.46 0)
 			(hide yes)
@@
 			(project "meko"
 				(path "/da54f10a-146b-4941-a9c7-55c7173bb101/45aa24d2-e0af-4ebb-a68a-61b6a12c0eec"
-					(reference "#PWR0124")
+					(reference "#PWR0126")
 					(unit 1)
 				)
@@
 		(in_pos_files yes)
 		(dnp no)
-		(property "Reference" "#PWR0119"
+		(property "Reference" "#PWR0121"
 			(at 92.71 129.54 0)
 			(hide yes)
@@
 			(project "meko"
 				(path "/da54f10a-146b-4941-a9c7-55c7173bb101/45aa24d2-e0af-4ebb-a68a-61b6a12c0eec"
-					(reference "#PWR0119")
+					(reference "#PWR0121")
 					(unit 1)
 				)
@@
 		(in_pos_files yes)
 		(dnp no)
-		(property "Reference" "#PWR0120"
+		(property "Reference" "#PWR0122"
 			(at 144.78 78.74 0)
 			(hide yes)
@@
 			(project "meko"
 				(path "/da54f10a-146b-4941-a9c7-55c7173bb101/45aa24d2-e0af-4ebb-a68a-61b6a12c0eec"
-					(reference "#PWR0120")
+					(reference "#PWR0122")
 					(unit 1)
 				)
@@
 		(in_pos_files yes)
 		(dnp no)
-		(property "Reference" "#PWR0122"
+		(property "Reference" "#PWR0124"
 			(at 153.67 55.88 0)
 			(hide yes)
@@
 			(project "meko"
 				(path "/da54f10a-146b-4941-a9c7-55c7173bb101/45aa24d2-e0af-4ebb-a68a-61b6a12c0eec"
-					(reference "#PWR0122")
+					(reference "#PWR0124")
 					(unit 1)
 				)
@@
 		(in_pos_files yes)
 		(dnp no)
-		(property "Reference" "#PWR0123"
+		(property "Reference" "#PWR0125"
 			(at 153.67 66.04 0)
 			(hide yes)
@@
 			(project "meko"
 				(path "/da54f10a-146b-4941-a9c7-55c7173bb101/45aa24d2-e0af-4ebb-a68a-61b6a12c0eec"
-					(reference "#PWR0123")
+					(reference "#PWR0125")
 					(unit 1)
 				)
@@
 		(in_pos_files yes)
 		(dnp no)
-		(property "Reference" "R37"
+		(property "Reference" "R39"
 			(at 67.818 36.195 0)
 			(show_name no)
@@
 			(project "meko"
 				(path "/da54f10a-146b-4941-a9c7-55c7173bb101/45aa24d2-e0af-4ebb-a68a-61b6a12c0eec"
-					(reference "R37")
+					(reference "R39")
 					(unit 1)
 				)
@@
 		(in_pos_files yes)
 		(dnp no)
-		(property "Reference" "R39"
+		(property "Reference" "R41"
 			(at 74.168 36.195 0)
 			(show_name no)
@@
 			(project "meko"
 				(path "/da54f10a-146b-4941-a9c7-55c7173bb101/45aa24d2-e0af-4ebb-a68a-61b6a12c0eec"
-					(reference "R39")
+					(reference "R41")
 					(unit 1)
 				)
@@
 		(in_pos_files yes)
 		(dnp no)
-		(property "Reference" "#PWR0121"
+		(property "Reference" "#PWR0123"
 			(at 144.78 147.32 0)
 			(hide yes)
@@
 			(project "meko"
 				(path "/da54f10a-146b-4941-a9c7-55c7173bb101/45aa24d2-e0af-4ebb-a68a-61b6a12c0eec"
-					(reference "#PWR0121")
+					(reference "#PWR0123")
 					(unit 1)
 				)
@@
 		(in_pos_files yes)
 		(dnp no)
-		(property "Reference" "C117"
+		(property "Reference" "C119"
 			(at 163.068 123.444 0)
 			(show_name no)
@@
 			(project "meko"
 				(path "/da54f10a-146b-4941-a9c7-55c7173bb101/45aa24d2-e0af-4ebb-a68a-61b6a12c0eec"
-					(reference "C117")
+					(reference "C119")
 					(unit 1)
 				)
@@
 		(in_pos_files yes)
 		(dnp no)
-		(property "Reference" "R41"
+		(property "Reference" "R43"
 			(at 80.518 36.195 0)
 			(show_name no)
@@
 			(project "meko"
 				(path "/da54f10a-146b-4941-a9c7-55c7173bb101/45aa24d2-e0af-4ebb-a68a-61b6a12c0eec"
-					(reference "R41")
+					(reference "R43")
 					(unit 1)
 				)
@@
 		(in_pos_files yes)
 		(dnp no)
-		(property "Reference" "R46"
+		(property "Reference" "R48"
 			(at 93.218 104.775 0)
 			(show_name no)
@@
 			(project "meko"
 				(path "/da54f10a-146b-4941-a9c7-55c7173bb101/45aa24d2-e0af-4ebb-a68a-61b6a12c0eec"
-					(reference "R46")
+					(reference "R48")
 					(unit 1)
 				)
@@
 		(in_pos_files yes)
 		(dnp no)
-		(property "Reference" "#PWR0115"
+		(property "Reference" "#PWR0117"
 			(at 58.42 102.87 0)
 			(hide yes)
@@
 			(project "meko"
 				(path "/da54f10a-146b-4941-a9c7-55c7173bb101/45aa24d2-e0af-4ebb-a68a-61b6a12c0eec"
-					(reference "#PWR0115")
-					(unit 1)
-				)
+					(reference "#PWR0117")
+					(unit 1)
+				)

Commit message: didn't save last time :sob:
Parts:
- renumbered C117 to C118, C118 to C119, C119 to C120
Changed lines of the file:
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@@
 		(in_pos_files yes)
 		(dnp no)
-		(property "Reference" "#PWR0118"
+		(property "Reference" "#PWR0119"
 			(at 102.87 55.88 0)
 			(hide yes)
@@
 			(project "meko"
 				(path "/da54f10a-146b-4941-a9c7-55c7173bb101/45aa24d2-e0af-4ebb-a68a-61b6a12c0eec"
-					(reference "#PWR0118")
+					(reference "#PWR0119")
 					(unit 1)
 				)
@@
 		(in_pos_files yes)
 		(dnp no)
-		(property "Reference" "C118"
+		(property "Reference" "C119"
 			(at 155.448 123.444 0)
 			(show_name no)
@@
 			(project "meko"
 				(path "/da54f10a-146b-4941-a9c7-55c7173bb101/45aa24d2-e0af-4ebb-a68a-61b6a12c0eec"
-					(reference "C118")
+					(reference "C119")
 					(unit 1)
 				)
@@
 		(in_pos_files yes)
 		(dnp no)
-		(property "Reference" "#PWR0127"
+		(property "Reference" "#PWR0128"
 			(at 153.67 134.62 0)
 			(hide yes)
@@
 			(project "meko"
 				(path "/da54f10a-146b-4941-a9c7-55c7173bb101/45aa24d2-e0af-4ebb-a68a-61b6a12c0eec"
-					(reference "#PWR0127")
+					(reference "#PWR0128")
 					(unit 1)
 				)
@@
 		(in_pos_files yes)
 		(dnp no)
-		(property "Reference" "#PWR0116"
+		(property "Reference" "#PWR0117"
 			(at 58.42 34.29 0)
 			(hide yes)
@@
 			(project "meko"
 				(path "/da54f10a-146b-4941-a9c7-55c7173bb101/45aa24d2-e0af-4ebb-a68a-61b6a12c0eec"
-					(reference "#PWR0116")
+					(reference "#PWR0117")
 					(unit 1)
 				)
@@
 		(in_pos_files yes)
 		(dnp no)
-		(property "Reference" "C117"
+		(property "Reference" "C118"
 			(at 155.448 54.864 0)
 			(show_name no)
@@
 			(project "meko"
 				(path "/da54f10a-146b-4941-a9c7-55c7173bb101/45aa24d2-e0af-4ebb-a68a-61b6a12c0eec"
-					(reference "C117")
+					(reference "C118")
 					(unit 1)
 				)
@@
 		(in_pos_files yes)
 		(dnp no)
-		(property "Reference" "#PWR0120"
+		(property "Reference" "#PWR0121"
 			(at 102.87 124.46 0)
 			(hide yes)
@@
 			(project "meko"
 				(path "/da54f10a-146b-4941-a9c7-55c7173bb101/45aa24d2-e0af-4ebb-a68a-61b6a12c0eec"
-					(reference "#PWR0120")
+					(reference "#PWR0121")
 					(unit 1)
 				)
@@
 		(in_pos_files yes)
 		(dnp no)
-		(property "Reference" "#PWR0119"
+		(property "Reference" "#PWR0120"
 			(at 92.71 60.96 0)
 			(hide yes)
@@
 			(project "meko"
 				(path "/da54f10a-146b-4941-a9c7-55c7173bb101/45aa24d2-e0af-4ebb-a68a-61b6a12c0eec"
-					(reference "#PWR0119")
+					(reference "#PWR0120")
 					(unit 1)
 				)
@@
 		(in_pos_files yes)
 		(dnp no)
-		(property "Reference" "#PWR0126"
+		(property "Reference" "#PWR0127"
 			(at 153.67 124.46 0)
 			(hide yes)
@@
 			(project "meko"
 				(path "/da54f10a-146b-4941-a9c7-55c7173bb101/45aa24d2-e0af-4ebb-a68a-61b6a12c0eec"
-					(reference "#PWR0126")
+					(reference "#PWR0127")
 					(unit 1)
 				)
@@
 		(in_pos_files yes)
 		(dnp no)
-		(property "Reference" "#PWR0121"
+		(property "Reference" "#PWR0122"
 			(at 92.71 129.54 0)
 			(hide yes)
@@
 			(project "meko"
 				(path "/da54f10a-146b-4941-a9c7-55c7173bb101/45aa24d2-e0af-4ebb-a68a-61b6a12c0eec"
-					(reference "#PWR0121")
+					(reference "#PWR0122")
 					(unit 1)
 				)
@@
 		(in_pos_files yes)
 		(dnp no)
-		(property "Reference" "#PWR0122"
+		(property "Reference" "#PWR0123"
 			(at 144.78 78.74 0)
 			(hide yes)
@@
 			(project "meko"
 				(path "/da54f10a-146b-4941-a9c7-55c7173bb101/45aa24d2-e0af-4ebb-a68a-61b6a12c0eec"
-					(reference "#PWR0122")
+					(reference "#PWR0123")
 					(unit 1)
 				)
@@
 		(in_pos_files yes)
 		(dnp no)
-		(property "Reference" "#PWR0124"
+		(property "Reference" "#PWR0125"
 			(at 153.67 55.88 0)
 			(hide yes)
@@
 			(project "meko"
 				(path "/da54f10a-146b-4941-a9c7-55c7173bb101/45aa24d2-e0af-4ebb-a68a-61b6a12c0eec"
-					(reference "#PWR0124")
+					(reference "#PWR0125")
 					(unit 1)
 				)
@@
 		(in_pos_files yes)
 		(dnp no)
-		(property "Reference" "#PWR0125"
+		(property "Reference" "#PWR0126"
 			(at 153.67 66.04 0)
 			(hide yes)
@@
 			(project "meko"
 				(path "/da54f10a-146b-4941-a9c7-55c7173bb101/45aa24d2-e0af-4ebb-a68a-61b6a12c0eec"
-					(reference "#PWR0125")
+					(reference "#PWR0126")
 					(unit 1)
 				)
@@
 		(in_pos_files yes)
 		(dnp no)
-		(property "Reference" "#PWR0123"
+		(property "Reference" "#PWR0124"
 			(at 144.78 147.32 0)
 			(hide yes)
@@
 			(project "meko"
 				(path "/da54f10a-146b-4941-a9c7-55c7173bb101/45aa24d2-e0af-4ebb-a68a-61b6a12c0eec"
-					(reference "#PWR0123")
+					(reference "#PWR0124")
 					(unit 1)
 				)
@@
 		(in_pos_files yes)
 		(dnp no)
-		(property "Reference" "C119"
+		(property "Reference" "C120"
 			(at 163.068 123.444 0)
 			(show_name no)
@@
 			(project "meko"
 				(path "/da54f10a-146b-4941-a9c7-55c7173bb101/45aa24d2-e0af-4ebb-a68a-61b6a12c0eec"
-					(reference "C119")
+					(reference "C120")
 					(unit 1)
 				)
@@
 		(in_pos_files yes)
 		(dnp no)
-		(property "Reference" "#PWR0117"
+		(property "Reference" "#PWR0118"
 			(at 58.42 102.87 0)
 			(hide yes)
@@
 			(project "meko"
 				(path "/da54f10a-146b-4941-a9c7-55c7173bb101/45aa24d2-e0af-4ebb-a68a-61b6a12c0eec"
-					(reference "#PWR0117")
-					(unit 1)
-				)
+					(reference "#PWR0118")
+					(unit 1)
+				)
