File: hardware/pcb/sama.kicad_sch (KiCad schematic)
At the start: 95 parts, among them J1 Conn_01x02_Pin, J2 Conn_ARM_JTAG_SWD_10, U1 SAMA7D65-4HB, Y1 24MHz, Y2 32kHz768

Commit message: laid out caps for vdd ddr, added custom rule area for bgas
Parts:
- added C128: 100n, Capacitor_SMD:C_0201_0603Metric, symbol Device:C_Small
Connections:
- net +1V35_DDR: now also C128.1
- net BT.DEV_WAKE: now also U1.H12 (PD15); no longer U1.M12 (PB20)
- net BT.EN: now also U1.E18 (PD16); no longer U1.R19 (PB11)
- net BT.HOST_WAKE: now also U1.C18 (PD14); no longer U1.L14 (PB19)
- net GND: now also C128.2
- net ZQ: now reaches R3.1, U1.AA2 (DDR_ZQ)
- no-connect marks 87 -> 84
Other:
- moved on the sheet: R3

Commit message: ddr routing, and mucking around
Parts:
- C14, C23, C27, C34, C42, C50, C52: footprint Capacitor_SMD:C_0201_0603Metric -> PCM_ckl-misc:C_0201_0603Metric_Dense
Changed lines of the file:
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@@
 			)
 		)
-		(property "Footprint" "Capacitor_SMD:C_0201_0603Metric"
+		(property "Footprint" "PCM_ckl-misc:C_0201_0603Metric_Dense"
 			(at 552.45 304.8 0)
 			(hide yes)
@@
 			)
 		)
-		(property "Footprint" "Capacitor_SMD:C_0201_0603Metric"
+		(property "Footprint" "PCM_ckl-misc:C_0201_0603Metric_Dense"
 			(at 528.32 255.27 0)
 			(hide yes)
@@
 			)
 		)
-		(property "Footprint" "Capacitor_SMD:C_0201_0603Metric"
+		(property "Footprint" "PCM_ckl-misc:C_0201_0603Metric_Dense"
 			(at 552.45 300.99 0)
 			(hide yes)
@@
 			)
 		)
-		(property "Footprint" "Capacitor_SMD:C_0201_0603Metric"
+		(property "Footprint" "PCM_ckl-misc:C_0201_0603Metric_Dense"
 			(at 552.45 285.75 0)
 			(hide yes)
@@
 			)
 		)
-		(property "Footprint" "Capacitor_SMD:C_0201_0603Metric"
+		(property "Footprint" "PCM_ckl-misc:C_0201_0603Metric_Dense"
 			(at 552.45 262.89 0)
 			(hide yes)
@@
 			)
 		)
-		(property "Footprint" "Capacitor_SMD:C_0201_0603Metric"
+		(property "Footprint" "PCM_ckl-misc:C_0201_0603Metric_Dense"
 			(at 552.45 266.7 0)
 			(hide yes)
@@
 			)
 		)
-		(property "Footprint" "Capacitor_SMD:C_0201_0603Metric"
+		(property "Footprint" "PCM_ckl-misc:C_0201_0603Metric_Dense"
 			(at 552.45 274.32 0)
 			(hide yes)

Commit message: routed ddr addr/cmd/clk
Parts:
- C37: footprint Capacitor_SMD:C_0201_0603Metric -> PCM_ckl-misc:C_0201_0603Metric_Dense
- R3: footprint Resistor_SMD:R_0402_1005Metric -> Resistor_SMD:R_0201_0603Metric
Changed lines of the file:
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@@
 			)
 		)
-		(property "Footprint" "Capacitor_SMD:C_0201_0603Metric"
+		(property "Footprint" "PCM_ckl-misc:C_0201_0603Metric_Dense"
 			(at 552.45 278.13 0)
 			(hide yes)
@@
 			)
 		)
-		(property "Footprint" "Resistor_SMD:R_0402_1005Metric"
+		(property "Footprint" "Resistor_SMD:R_0201_0603Metric"
 			(at 464.82 124.968 90)
 			(hide yes)

Commit message: added lables
Connections:
- net SD1_CAL: now reaches R9.2, U1.B13 (SDMMC1_CAL)
- net QSPI0_CAL: now reaches R11.2, U1.M13 (QSPI0_CAL)
- net SD2_CAL: now reaches R10.2, U1.E14 (SDMMC2_CAL)
- net SD0_CAL: now reaches R8.2, U1.R16 (SDMMC0_CAL)
- net MIPI_REXT: now reaches R7.1, U1.V18 (MIPI_REXT)
- no-connect marks 84 -> 86
Other:
- moved on the sheet: C2, R10, R11, R6, R7, R8, R9, TP10, TP11, TP6, TP8, TP9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

Commit message: caps
Parts:
- C35, C38, C41, C61: footprint Capacitor_SMD:C_0201_0603Metric -> PCM_ckl-misc:C_0201_0603Metric_Dense
Changed lines of the file:
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@@
 			)
 		)
-		(property "Footprint" "Capacitor_SMD:C_0201_0603Metric"
+		(property "Footprint" "PCM_ckl-misc:C_0201_0603Metric_Dense"
 			(at 482.6 281.94 0)
 			(hide yes)
@@
 			)
 		)
-		(property "Footprint" "Capacitor_SMD:C_0201_0603Metric"
+		(property "Footprint" "PCM_ckl-misc:C_0201_0603Metric_Dense"
 			(at 505.46 335.28 0)
 			(hide yes)
@@
 			)
 		)
-		(property "Footprint" "Capacitor_SMD:C_0201_0603Metric"
+		(property "Footprint" "PCM_ckl-misc:C_0201_0603Metric_Dense"
 			(at 482.6 285.75 0)
 			(hide yes)
@@
 			)
 		)
-		(property "Footprint" "Capacitor_SMD:C_0201_0603Metric"
+		(property "Footprint" "PCM_ckl-misc:C_0201_0603Metric_Dense"
 			(at 482.6 278.13 0)
 			(hide yes)

Commit message: finished cap placement
Parts:
- C13, C17, C24, C25, C32, C45, C47, C58: footprint Capacitor_SMD:C_0201_0603Metric -> PCM_ckl-misc:C_0201_0603Metric_Dense
Changed lines of the file:
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@@
 			)
 		)
-		(property "Footprint" "Capacitor_SMD:C_0201_0603Metric"
+		(property "Footprint" "PCM_ckl-misc:C_0201_0603Metric_Dense"
 			(at 505.46 259.08 0)
 			(hide yes)
@@
 			)
 		)
-		(property "Footprint" "Capacitor_SMD:C_0201_0603Metric"
+		(property "Footprint" "PCM_ckl-misc:C_0201_0603Metric_Dense"
 			(at 505.46 327.66 0)
 			(hide yes)
@@
 			)
 		)
-		(property "Footprint" "Capacitor_SMD:C_0201_0603Metric"
+		(property "Footprint" "PCM_ckl-misc:C_0201_0603Metric_Dense"
 			(at 482.6 297.18 0)
 			(hide yes)
@@
 			)
 		)
-		(property "Footprint" "Capacitor_SMD:C_0201_0603Metric"
+		(property "Footprint" "PCM_ckl-misc:C_0201_0603Metric_Dense"
 			(at 482.6 266.7 0)
 			(hide yes)
@@
 			)
 		)
-		(property "Footprint" "Capacitor_SMD:C_0201_0603Metric"
+		(property "Footprint" "PCM_ckl-misc:C_0201_0603Metric_Dense"
 			(at 505.46 266.7 0)
 			(hide yes)
@@
 			)
 		)
-		(property "Footprint" "Capacitor_SMD:C_0201_0603Metric"
+		(property "Footprint" "PCM_ckl-misc:C_0201_0603Metric_Dense"
 			(at 505.46 255.27 0)
 			(hide yes)
@@
 			)
 		)
-		(property "Footprint" "Capacitor_SMD:C_0201_0603Metric"
+		(property "Footprint" "PCM_ckl-misc:C_0201_0603Metric_Dense"
 			(at 482.6 274.32 0)
 			(hide yes)
@@
 			)
 		)
-		(property "Footprint" "Capacitor_SMD:C_0201_0603Metric"
+		(property "Footprint" "PCM_ckl-misc:C_0201_0603Metric_Dense"
 			(at 482.6 293.37 0)
 			(hide yes)

Commit message: pwr
Parts:
- C33, C36, C49, C5: footprint Capacitor_SMD:C_0201_0603Metric -> PCM_ckl-misc:C_0201_0603Metric_Dense
Changed lines of the file:
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@@
 			)
 		)
-		(property "Footprint" "Capacitor_SMD:C_0201_0603Metric"
+		(property "Footprint" "PCM_ckl-misc:C_0201_0603Metric_Dense"
 			(at 482.6 300.99 0)
 			(hide yes)
@@
 			)
 		)
-		(property "Footprint" "Capacitor_SMD:C_0201_0603Metric"
+		(property "Footprint" "PCM_ckl-misc:C_0201_0603Metric_Dense"
 			(at 500.38 227.33 0)
 			(hide yes)
@@
 			)
 		)
-		(property "Footprint" "Capacitor_SMD:C_0201_0603Metric"
+		(property "Footprint" "PCM_ckl-misc:C_0201_0603Metric_Dense"
 			(at 528.32 274.32 0)
 			(hide yes)
@@
 			)
 		)
-		(property "Footprint" "Capacitor_SMD:C_0201_0603Metric"
+		(property "Footprint" "PCM_ckl-misc:C_0201_0603Metric_Dense"
 			(at 528.32 278.13 0)
 			(hide yes)
